File: Projects/Camera_System.sch (KiCad schematic (older format))
At the start: 60 parts, among them CON1 AVR-ISP-10, J1 BARREL_JACK, U1 IFX1117ME_V33, U10 RT1105AF160Q, U11 RT1105AF160Q, U12 LCD_1602, U13 RT1105AF160Q, U14 Si501, U15 OV7670-nofifo, U16 ESP8266, U17 SDCARD, U2 LD2980ABM50TR, U3 ATMEGA16A-AU, U4 RT1105AF160Q, U5 RT1105AF160Q, U6 RT1105AF160Q, U7 RT1105AF160Q, U8 CD4014B, U9 PCA9306, Y1 Crystal

Commit message: Layout has been updated
Parts:
- U15: symbol OV7670-nofifo -> OV7670-nofifo-RESCUE-Camera_System
Connections:
- wire segments 271 -> 273
Other:
- moved on the sheet: R1
Changed lines of the file:
@@
 EESchema Schematic File Version 2
+LIBS:Camera_System-rescue
 LIBS:power
 LIBS:device
@@
 	0    -1   -1   0
 $EndComp
-Text Label 3800 6350 0    60   ~ 0
+Text Label 3800 8550 0    60   ~ 0
 CAM_D0
-Text Label 3800 9450 0    60   ~ 0
+Text Label 3800 8650 0    60   ~ 0
 CAM_D1
-Text Label 3800 6550 0    60   ~ 0
+Text Label 3800 8750 0    60   ~ 0
 CAM_D2
-Text Label 3800 6650 0    60   ~ 0
+Text Label 3800 8850 0    60   ~ 0
 CAM_D3
+Text Label 3800 6950 0    60   ~ 0
+CAM_D4
+Text Label 3800 7050 0    60   ~ 0
+CAM_D5
 Text Label 3800 6750 0    60   ~ 0
-CAM_D4
+CAM_D6
 Text Label 3800 6850 0    60   ~ 0
-CAM_D5
-Text Label 3800 6950 0    60   ~ 0
-CAM_D6
-Text Label 3800 7050 0    60   ~ 0
 CAM_D7
 $Comp
 L R R1
 U 1 1 591871FF
-P 4350 7550
-F 0 "R1" V 4250 7550 50  0000 C CNN
-F 1 "0" V 4350 7550 50  0000 C CNN
-F 2 "Resistors_SMD:R_0603_HandSoldering" V 4280 7550 50  0001 C CNN
-F 3 "" H 4350 7550 50  0001 C CNN
-	1    4350 7550
+P 4300 9650
+F 0 "R1" V 4200 9650 50  0000 C CNN
+F 1 "0" V 4300 9650 50  0000 C CNN
+F 2 "Resistors_SMD:R_0603_HandSoldering" V 4230 9650 50  0001 C CNN
+F 3 "" H 4300 9650 50  0001 C CNN
+	1    4300 9650
 	0    1    1    0
 $EndComp
-Text Label 4550 7550 0    60   ~ 0
+Text Label 4500 9650 0    60   ~ 0
 CAM_XCLK
 Text Label 3800 7650 0    60   ~ 0
@@
 Text Label 3800 8250 0    60   ~ 0
 3V3_SDA
-Text Label 3800 8350 0    60   ~ 0
+Text Label 3800 9550 0    60   ~ 0
 WLAN_CHPD
-Text Label 3800 8450 0    60   ~ 0
+Text Label 3800 9250 0    60   ~ 0
 WLAN_RST
-Text Label 3800 8550 0    60   ~ 0
+Text Label 3800 9450 0    60   ~ 0
 WLAN_GPIO0
-Text Label 3800 8650 0    60   ~ 0
+Text Label 3800 9350 0    60   ~ 0
 WLAN_GPIO2
 Text Label 3800 9050 0    60   ~ 0
@@
 Text Label 3800 9150 0    60   ~ 0
 WLAN_TX
-Text Label 3800 9250 0    60   ~ 0
+Text Label 3800 8450 0    60   ~ 0
 CAM_RST
-Text Label 3800 9350 0    60   ~ 0
+Text Label 3800 8350 0    60   ~ 0
 CAM_PWDN
+Text Label 3800 6650 0    60   ~ 0
+CAM_PCLK
+Text Label 3800 6550 0    60   ~ 0
+CAM_HREF
 Text Label 3800 6450 0    60   ~ 0
-CAM_PCLK
-Text Label 3800 9650 0    60   ~ 0
-CAM_HREF
-Text Label 3800 9750 0    60   ~ 0
 CAM_VSINC
 $Comp
@@
 $EndComp
 $Comp
-L OV7670-nofifo U15
+L OV7670-nofifo-RESCUE-Camera_System U15
 U 1 1 59193962
 P 14200 2100
@@
 Text Label 8950 5650 0    60   ~ 0
 CTRL_BTN2
-Text Label 3800 9550 0    60   ~ 0
+Text Label 3800 7550 0    60   ~ 0
 P_S_CLK
 Text Label 10500 5650 0    60   ~ 0
@@
 	3750 7550 4200 7550
 Wire Wire Line
-	4500 7550 4800 7550
-Wire Wire Line
 	3750 7650 4150 7650
 Wire Wire Line
@@
 	1    0    0    -1
 $EndComp
+Wire Wire Line
+	3750 8750 4150 8750
+Wire Wire Line
+	3750 8850 4150 8850
+Wire Wire Line
+	4450 9650 4750 9650
 $EndSCHEMATC

Commit message: Layout first draft finished
Parts:
- added U18, U19: header_male_2.54_2x2, MyLibraries:header_male_2.54_2x2, symbol header_male_2.54_2x2
- added U20: header_male_2.54_2x3, MyLibraries:header_male_2.54_2x3, symbol header_male_2.54_2x3
Connections:
- wire segments 273 -> 287
Other:
- note added: "DEBUG PINS"
- note added: "POWER MANAG."
