File: Projects/CameraSystem/Schematics/Camera_System.sch (KiCad schematic (older format))
At the start: 63 parts, among them CON1 AVR-ISP-10, J1 BARREL_JACK, U1 IFX1117ME_V33, U10 RT1105AF160Q, U11 RT1105AF160Q, U12 LCD_1602, U13 RT1105AF160Q, U14 Si501, U15 OV7670-nofifo, U16 ESP8266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

Commit message: Files were restructured
Other:
- note added: "6.5 < VIN < 15"
- note added: "I_out_max = 1A"
- note removed: "6 < VIN < 15"
- note removed: "I_out = 1.1A"
Changed lines of the file:
@@
 $EndComp
 Text Notes 3250 1200 0    60   ~ 0
-6 < VIN < 15
+6.5 < VIN < 15
 Text Notes 4100 800  0    60   ~ 0
 Order the one with fixed output voltage = 3.3V
 Text Notes 5000 1200 0    60   ~ 0
-I_out = 1.1A
+I_out_max = 1A
 $Comp
 L CP C2
