File: Projects/CameraSystem/Schematics/Memory.sch (KiCad schematic (older format))
At the start: 0 parts

Commit message: feat: first draft of uc schematic created
Parts:
- added C? (x2): 100n, symbol C
- added J?: CONN_02X02, symbol CONN_02X02
- added J?: 1040310811, symbol Micro_SD_Card
- added R?: 10k, symbol R
- added U?: MC74HC125ADTR2G, symbol MC74HC125ADTR2G
Connections:
- new net: R?.2, U?.12 (A4)
- new net GND: C?.1, C?.2, J?.6 (VSS), J?.9 (SHIELD), U?.1 (OE1), U?.10 (OE3), U?.13 (OE4), U?.4 (OE2), U?.7 (GND)
- new net MISO: U?.8 (Y3)
- new net MOSI: U?.2 (A1)
- new net SCK: U?.5 (A2)
- new net SD_CLK_IN: J?.5 (CLK)
- new net SD_CS: C?.1, C?.2, J?.2 (P2), J?.4 (P4), J?.4 (VDD), R?.1, U?.14 (3.3V)
- new net SD_CS_IN: J?.2 (DAT3/CD), U?.11 (Y4)
- new net SD_DATA_IN: J?.3 (CMD), U?.3 (Y1)
- new net SD_DATA_OUT: J?.7 (DAT0), U?.9 (A3)
- new net SD_SCK_IN: U?.6 (Y2)
- new net VDD_3V3: J?.1 (P1), J?.3 (P3)

Commit message: feat: 3.3 regulator housing changed due to temperature
Parts:
- C? (x2): symbol C -> Device:C
- J?: symbol CONN_02X02 -> CameraSystem-rescue:CONN_02X02
- J?: symbol Micro_SD_Card -> CameraSystem-rescue:Micro_SD_Card
- R?: symbol R -> Device:R
- U?: symbol MC74HC125ADTR2G -> cl-integrated_circuits:MC74HC125ADTR2G
Changed lines of the file:
@@
-EESchema Schematic File Version 2
-LIBS:cl-connectors
-LIBS:dk_Addressable-Specialty
-LIBS:dk_Alarms-Buzzers-and-Sirens
-LIBS:dk_Automotive-Relays
-LIBS:dk_Balun
-LIBS:dk_Barrel-Audio-Connectors
-LIBS:dk_Battery-Holders-Clips-Contacts
-LIBS:dk_Clock-Timing-Clock-Generators-PLLs-Frequency-Synthesizers
-LIBS:dk_Clock-Timing-Programmable-Timers-and-Oscillators
-LIBS:dk_Clock-Timing-Real-Time-Clocks
-LIBS:dk_Coaxial-Connectors-RF
-LIBS:dk_Current-Transducers
-LIBS:dk_Data-Acquisition-ADCs-DACs-Special-Purpose
-LIBS:dk_Data-Acquisition-Analog-to-Digital-Converters-ADC
-LIBS:dk_Data-Acquisition-Digital-Potentiometers
-LIBS:dk_Data-Acquisition-Digital-to-Analog-Converters-DAC
-LIBS:dk_Data-Acquisition-Touch-Screen-Controllers
-LIBS:dk_DC-DC-Converters
-LIBS:dk_Digital-Isolators
-LIBS:dk_Diodes-Bridge-Rectifiers
-LIBS:dk_Diodes-Rectifiers-Arrays
-LIBS:dk_Diodes-Rectifiers-Single
-LIBS:dk_Diodes-Zener-Single
-LIBS:dk_Display-Modules-LCD-OLED-Graphic
-LIBS:dk_Display-Modules-LED-Character-and-Numeric
-LIBS:dk_D-Sub-Connectors
-LIBS:dk_Embedded-Microcontrollers
-LIBS:dk_Encoders
-LIBS:dk_Evaluation-Boards-Sensors
-LIBS:dk_Ferrite-Beads-and-Chips
-LIBS:dk_Fixed-Inductors
-LIBS:dk_Fuses
-LIBS:dk_Gas-Sensors
-LIBS:dk_Humidity-Moisture-Sensors
-LIBS:dk_Image-Sensors-Camera
-LIBS:dk_Infrared-UV-Visible-Emitters
-LIBS:dk_Inrush-Current-Limiters-ICL
-LIBS:dk_Interface-Analog-Switches-Multiplexers-Demultiplexers
-LIBS:dk_Interface-Analog-Switches-Special-Purpose
-LIBS:dk_Interface-Controllers
-LIBS:dk_Interface-Drivers-Receivers-Transceivers
-LIBS:dk_Interface-I-O-Expanders
-LIBS:dk_Interface-Modules
-LIBS:dk_Interface-Sensor-and-Detector-Interfaces
-LIBS:dk_Interface-Sensor-Capacitive-Touch
-LIBS:dk_Interface-Specialized
-LIBS:dk_LED-Indication-Discrete
-LIBS:dk_LEDs-Circuit-Board-Indicators-Arrays-Light-Bars-Bar-Graphs
-LIBS:dk_Linear-Amplifiers-Audio
-LIBS:dk_Linear-Amplifiers-Instrumentation-OP-Amps-Buffer-Amps
-LIBS:dk_Linear-Comparators
-LIBS:dk_Logic-Buffers-Drivers-Receivers-Transceivers
-LIBS:dk_Logic-Flip-Flops
-LIBS:dk_Logic-Gates-and-Inverters
-LIBS:dk_Logic-Multivibrators
-LIBS:dk_Logic-Shift-Registers
-LIBS:dk_Logic-Signal-Switches-Multiplexers-Decoders
-LIBS:dk_Logic-Translators-Level-Shifters
-LIBS:dk_Magnetic-Sensors-Compass-Magnetic-Field-Modules
-LIBS:dk_Magnetic-Sensors-Linear-Compass-ICs
-LIBS:dk_Magnetic-Sensors-Switches-Solid-State
-LIBS:dk_Memory
-LIBS:dk_Memory-Connectors-PC-Card-Sockets
-LIBS:dk_Microphones
-LIBS:dk_Modular-Connectors-Jacks
-LIBS:dk_Modular-Connectors-Jacks-With-Magnetics
-LIBS:dk_Motion-Sensors-Accelerometers
-LIBS:dk_Motion-Sensors-IMUs-Inertial-Measurement-Units
-LIBS:dk_Motion-Sensors-Tilt-Switches
-LIBS:dk_Navigation-Switches-Joystick
-LIBS:dk_Optical-Sensors-Ambient-Light-IR-UV-Sensors
-LIBS:dk_Optical-Sensors-Photo-Detectors-Remote-Receiver
-LIBS:dk_Optical-Sensors-Photodiodes
-LIBS:dk_Optical-Sensors-Phototransistors
-LIBS:dk_Optical-Sensors-Reflective-Analog-Output
-LIBS:dk_Optoisolators-Logic-Output
-LIBS:dk_Optoisolators-Transistor-Photovoltaic-Output
-LIBS:dk_Optoisolators-Triac-SCR-Output
-LIBS:dk_Oscillators
-LIBS:dk_PMIC-AC-DC-Converters-Offline-Switchers
-LIBS:dk_PMIC-Battery-Chargers
-LIBS:dk_PMIC-Battery-Management
-LIBS:dk_PMIC-Current-Regulation-Management
-LIBS:dk_PMIC-Full-Half-Bridge-Drivers
-LIBS:dk_PMIC-Gate-Drivers
-LIBS:dk_PMIC-LED-Drivers
-LIBS:dk_PMIC-Motor-Drivers-Controllers
-LIBS:dk_PMIC-OR-Controllers-Ideal-Diodes
-LIBS:dk_PMIC-Power-Distribution-Switches-Load-Drivers
-LIBS:dk_PMIC-Power-Management-Specialized
-LIBS:dk_PMIC-RMS-to-DC-Converters
-LIBS:dk_PMIC-Supervisors
-LIBS:dk_PMIC-Thermal-Management
-LIBS:dk_PMIC-V-F-and-F-V-Converters
-LIBS:dk_PMIC-Voltage-Reference
-LIBS:dk_PMIC-Voltage-Regulators-DC-DC-Switching-Controllers
-LIBS:dk_PMIC-Voltage-Regulators-DC-DC-Switching-Regulators
-LIBS:dk_PMIC-Voltage-Regulators-Linear
-LIBS:dk_PMIC-Voltage-Regulators-Special-Purpose
-LIBS:dk_Power-Relays-Over-2-Amps
-LIBS:dk_Pressure-Sensors-Transducers
-LIBS:dk_Programmable-Oscillators
-LIBS:dk_Pushbutton-Switches
-LIBS:dk_Rectangular-Connectors-Headers-Male-Pins
-LIBS:dk_Reed-Relays
-LIBS:dk_Resistor-Networks-Arrays
-LIBS:dk_RF-Amplifiers
-LIBS:dk_RF-Antennas
-LIBS:dk_RF-Demodulators
-LIBS:dk_RF-Detectors
-LIBS:dk_RF-Evaluation-and-Development-Kits-Boards
-LIBS:dk_RFID-RF-Access-Monitoring-ICs
-LIBS:dk_RF-Receivers
-LIBS:dk_RF-Switches
-LIBS:dk_RF-Transceiver-ICs
-LIBS:dk_RF-Transceiver-Modules
-LIBS:dk_RF-Transmitters
-LIBS:dk_Rotary-Potentiometers-Rheostats
-LIBS:dk_Sensors-Transducers_Accessories
-LIBS:dk_Signal-Relays-Up-to-2-Amps
-LIBS:dk_Slide-Switches
-LIBS:dk_Solid-State-Relays
-LIBS:dk_Specialized-ICs
-LIBS:dk_Specialized-Sensors
-LIBS:dk_Surge-Suppression-ICs
-LIBS:dk_Tactile-Switches
-LIBS:dk_Temperature-Sensors-Analog-and-Digital-Output
-LIBS:dk_Thermal-Cutoffs-Thermal-Fuses
-LIBS:dk_Thyristors-DIACs-SIDACs
-LIBS:dk_Thyristors-SCRs
-LIBS:dk_Thyristors-TRIACs
-LIBS:dk_Toggle-Switches
-LIBS:dk_Transistors-Bipolar-BJT-Arrays
-LIBS:dk_Transistors-Bipolar-BJT-RF
-LIBS:dk_Transistors-Bipolar-BJT-Single
-LIBS:dk_Transistors-Bipolar-BJT-Single-Pre-Biased
-LIBS:dk_Transistors-FETs-MOSFETs-Arrays
-LIBS:dk_Transistors-FETs-MOSFETs-RF
-LIBS:dk_Transistors-FETs-MOSFETs-Single
-LIBS:dk_Transistors-JFETs
-LIBS:dk_Trimmer-Potentiometers
-LIBS:dk_TVS-Diodes
-LIBS:dk_TVS-Mixed-Technology
-LIBS:dk_USB-DVI-HDMI-Connectors
-LIBS:power
-LIBS:device
-LIBS:transistors
-LIBS:conn
-LIBS:linear
-LIBS:regul
-LIBS:74xx
-LIBS:cmos4000
-LIBS:adc-dac
-LIBS:memory
-LIBS:xilinx
-LIBS:microcontrollers
-LIBS:dsp
-LIBS:microchip
-LIBS:analog_switches
-LIBS:motorola
-LIBS:texas
-LIBS:intel
-LIBS:audio
-LIBS:interface
-LIBS:digital-audio
-LIBS:philips
-LIBS:display
-LIBS:cypress
-LIBS:siliconi
-LIBS:opto
-LIBS:atmel
-LIBS:contrib
-LIBS:valves
-LIBS:cl-integrated_circuits
-LIBS:cl-misc
+EESchema Schematic File Version 4
 LIBS:CameraSystem-cache
-EELAYER 25 0
+EELAYER 26 0
 EELAYER END
 $Descr A4 11693 8268
@@
 $EndDescr
 $Comp
-L CONN_02X02 J?
+L CameraSystem-rescue:CONN_02X02 J?
 U 1 1 5BBAA572
 P 2950 1500
+AR Path="/5BBAA572" Ref="J?"  Part="1"
+AR Path="/5BB4DA56/5BBAA572" Ref="J?"  Part="1"
 F 0 "J?" H 2950 1650 50  0000 C CNN
 F 1 "CONN_02X02" H 2950 1350 50  0000 C CNN
@@
 	2700 1450 2650 1450
 Wire Wire Line
-	2650 1450 2650 1550
+	2650 1450 2650 1500
 Wire Wire Line
 	2650 1550 2700 1550
@@
 	3250 1550 3200 1550
 Wire Wire Line
-	3250 1450 3250 1550
+	3250 1450 3250 1500
 Wire Wire Line
 	3250 1450 3200 1450
@@
 VDD_3V3_IN
 $Comp
-L MC74HC125ADTR2G U?
+L cl-integrated_circuits:MC74HC125ADTR2G U?
 U 1 1 5BBAA814
 P 5750 2800
@@
 $EndComp
 $Comp
-L Micro_SD_Card J?
+L CameraSystem-rescue:Micro_SD_Card J?
 U 1 1 5BBAA877
 P 6450 4700
+AR Path="/5BBAA877" Ref="J?"  Part="1"
+AR Path="/5BB4DA56/5BBAA877" Ref="J?"  Part="1"
 F 0 "J?" H 5800 5300 50  0000 C CNN
 F 1 "1040310811" H 7100 5300 50  0000 R CNN
@@
 $EndComp
 $Comp
-L GND #PWR?
+L power:GND #PWR?
 U 1 1 5BBAAC4D
 P 7600 5650
@@
 	7600 5300 7600 5650
 $Comp
-L GND #PWR?
+L power:GND #PWR?
 U 1 1 5BBAAE22
 P 4250 2550
@@
 $EndComp
 $Comp
-L GND #PWR?
+L power:GND #PWR?
 U 1 1 5BBAAE4E
 P 4250 2850
@@
 $EndComp
 $Comp
-L GND #PWR?
+L power:GND #PWR?
 U 1 1 5BBAAE80
 P 4250 3150
@@
 $EndComp
 $Comp
-L GND #PWR?
+L power:GND #PWR?
 U 1 1 5BBAAE94
 P 7500 2650
@@
 $EndComp
 $Comp
-L GND #PWR?
+L power:GND #PWR?
 U 1 1 5BBAAEA8
 P 7500 2950
@@
 SD_SCK_IN
 Wire Wire Line
-	6300 2500 7400 2500
+	6300 2500 6400 2500
 Text Label 7400 2500 0    60   ~ 0
 VDD_3V3_IN
 $Comp
-L R R?
+L Device:R R?
 U 1 1 5BBAB32F
 P 6500 2700
@@
 	6300 2700 6350 2700
 Wire Wire Line
-	6650 2700 7050 2700
+	6650 2700 6850 2700
 Wire Wire Line
 	6850 2700 6850 2500
@@
 Connection ~ 6400 2500
 $Comp
-L C C?
+L Device:C C?
 U 1 1 5BBAB4F4
 P 6400 2150
@@
 	6700 1900 6700 2000
 $Comp
-L GND #PWR?
+L power:GND #PWR?
 U 1 1 5BBAB570
 P 6700 2000
@@
 SD_DATA_OUT
 $Comp
-L C C?
+L Device:C C?
 U 1 1 5BBABB37
 P 4350 5050
@@
 $EndComp
 Wire Wire Line
-	4100 4700 5550 4700
+	4100 4700 4350 4700
 Wire Wire Line
 	4350 4700 4350 4900
 $Comp
-L GND #PWR?
+L power:GND #PWR?
 U 1 1 5BBABC51
 P 4350 5350
@@
 	4600 4900 4600 5350
 $Comp
-L GND #PWR?
+L power:GND #PWR?
 U 1 1 5BBABFC7
 P 4600 5350
@@
 Text Label 4750 4500 0    60   ~ 0
 SD_CS_IN
+Wire Wire Line
+	2650 1500 2650 1550
+Wire Wire Line
+	3250 1500 3250 1550
+Wire Wire Line
+	6850 2500 7400 2500
+Wire Wire Line
+	6400 2500 6850 2500
+Wire Wire Line
+	6850 2700 7050 2700
+Wire Wire Line
+	4350 4700 5550 4700
 $EndSCHEMATC
