File: Projects/CameraSystem/Schematics/Memory.sch (KiCad schematic (older format))
At the start: 8 parts, among them J7 Conn_02x02_Odd_Even, J8 DM3D-SF, U5 MC74HC125ADTR2G

Commit message: replace tvs diodes of camera system
Changed lines of the file:
@@
 Text Label 4700 2700 0    60   ~ 0
 SD_DATA_IN
-Text HLabel 4700 2600 0    60   Input ~ 0
+Text HLabel 4700 2600 0    60   Output ~ 0
 SD_MISO
 Text HLabel 4700 2900 0    60   Input ~ 0
@@
 Wire Wire Line
 	6300 3100 7050 3100
-Text HLabel 7050 3100 2    60   Output ~ 0
+Text HLabel 7050 3100 2    60   Input ~ 0
 SD_MOSI
 Text Label 7050 3000 2    60   ~ 0

Commit message: linux adaptation
Parts:
- U5: symbol cl-integrated_circuits:MC74HC125ADTR2G -> CameraSystem-rescue:MC74HC125ADTR2G-cl-integrated_circuits
Connections:
- net labels added: SD_DATA_IN_BUF, SD_DATA_OUT_BUF
- net labels removed: SD_MISO, SD_MOSI
Changed lines of the file:
@@
 VDD_3V3
 $Comp
-L cl-integrated_circuits:MC74HC125ADTR2G U5
+L CameraSystem-rescue:MC74HC125ADTR2G-cl-integrated_circuits U5
 U 1 1 5BBAA814
 P 5750 2800
+AR Path="/5BBAA814" Ref="U5"  Part="1"
+AR Path="/5BB4DA56/5BBAA814" Ref="U5"  Part="1"
 F 0 "U5" H 5750 2300 60  0000 C CNN
 F 1 "MC74HC125ADTR2G" H 5750 3300 60  0000 C CNN
@@
 L power:GND #PWR0123
 U 1 1 5BBAAE22
-P 4250 2550
-F 0 "#PWR0123" H 4250 2300 50  0001 C CNN
-F 1 "GND" H 4250 2400 50  0000 C CNN
-F 2 "" H 4250 2550 50  0001 C CNN
-F 3 "" H 4250 2550 50  0001 C CNN
-	1    4250 2550
+P 4100 2550
+F 0 "#PWR0123" H 4100 2300 50  0001 C CNN
+F 1 "GND" H 4100 2400 50  0000 C CNN
+F 2 "" H 4100 2550 50  0001 C CNN
+F 3 "" H 4100 2550 50  0001 C CNN
+	1    4100 2550
 	1    0    0    -1
 $EndComp
@@
 L power:GND #PWR0124
 U 1 1 5BBAAE4E
-P 4250 2850
-F 0 "#PWR0124" H 4250 2600 50  0001 C CNN
-F 1 "GND" H 4250 2700 50  0000 C CNN
-F 2 "" H 4250 2850 50  0001 C CNN
-F 3 "" H 4250 2850 50  0001 C CNN
-	1    4250 2850
+P 4100 2850
+F 0 "#PWR0124" H 4100 2600 50  0001 C CNN
+F 1 "GND" H 4100 2700 50  0000 C CNN
+F 2 "" H 4100 2850 50  0001 C CNN
+F 3 "" H 4100 2850 50  0001 C CNN
+	1    4100 2850
 	1    0    0    -1
 $EndComp
@@
 L power:GND #PWR0125
 U 1 1 5BBAAE80
-P 4250 3150
-F 0 "#PWR0125" H 4250 2900 50  0001 C CNN
-F 1 "GND" H 4250 3000 50  0000 C CNN
-F 2 "" H 4250 3150 50  0001 C CNN
-F 3 "" H 4250 3150 50  0001 C CNN
-	1    4250 3150
+P 4100 3150
+F 0 "#PWR0125" H 4100 2900 50  0001 C CNN
+F 1 "GND" H 4100 3000 50  0000 C CNN
+F 2 "" H 4100 3150 50  0001 C CNN
+F 3 "" H 4100 3150 50  0001 C CNN
+	1    4100 3150
 	1    0    0    -1
 $EndComp
@@
 $EndComp
 Wire Wire Line
-	4250 2550 4250 2500
+	4100 2550 4100 2500
 Wire Wire Line
-	4250 2500 5250 2500
+	4100 2500 5250 2500
 Wire Wire Line
-	4250 2850 4250 2800
+	4100 2850 4100 2800
 Wire Wire Line
-	4250 2800 5250 2800
+	4100 2800 5250 2800
 Wire Wire Line
-	4250 3150 4250 3100
+	4100 3150 4100 3100
 Wire Wire Line
-	4250 3100 5250 3100
+	4100 3100 5250 3100
 Wire Wire Line
 	7050 2900 6300 2900
@@
 	5250 2900 4700 2900
 Text Label 4700 2700 0    60   ~ 0
-SD_DATA_IN
+SD_DATA_OUT
 Text HLabel 4700 2600 0    60   Output ~ 0
-SD_MISO
+SD_DATA_OUT_BUF
 Text HLabel 4700 2900 0    60   Input ~ 0
 SD_SCK
@@
 Wire Wire Line
 	6300 3100 7050 3100
-Text HLabel 7050 3100 2    60   Input ~ 0
-SD_MOSI
-Text Label 7050 3000 2    60   ~ 0
-SD_DATA_OUT
+Text HLabel 7050 3000 2    60   Input ~ 0
+SD_DATA_IN_BUF
+Text Label 7050 3100 2    60   ~ 0
+SD_DATA_IN
 $Comp
 L Device:C C19

Commit message: camera was updated
Parts:
- C27: renamed from C19; footprint digikey-footprints:0603 -> Capacitor_SMD:C_0603_1608Metric_Pad1.05x0.95mm_HandSolder
- C28: renamed from C27; footprint digikey-footprints:0603 -> Capacitor_SMD:C_0603_1608Metric_Pad1.05x0.95mm_HandSolder
- C29: renamed from C20; footprint digikey-footprints:0603 -> Capacitor_SMD:C_0603_1608Metric_Pad1.05x0.95mm_HandSolder
- J12: renamed from J7; footprint Pin_Headers:Pin_Header_Straight_2x02_Pitch2.54mm_SMD -> Connector_PinSocket_2.54mm:PinSocket_2x02_P2.54mm_Vertical
- J13: renamed from J8; symbol Connector:Micro_SD_Card_Det -> CameraSystem-rescue:Micro_SD_Card_Det-Connector
- R38: renamed from R12; footprint digikey-footprints:0603 -> Resistor_SMD:R_0603_1608Metric_Pad1.05x0.95mm_HandSolder
- R39: renamed from R25; footprint digikey-footprints:0603 -> Resistor_SMD:R_0603_1608Metric_Pad1.05x0.95mm_HandSolder
- renumbered U5 to U11
Changed lines of the file:
@@
 EESchema Schematic File Version 4
 LIBS:CameraSystem-cache
-EELAYER 26 0
+EELAYER 29 0
 EELAYER END
 $Descr A4 11693 8268
@@
 VDD_3V3
 $Comp
-L CameraSystem-rescue:MC74HC125ADTR2G-cl-integrated_circuits U5
+L CameraSystem-rescue:MC74HC125ADTR2G-cl-integrated_circuits U?
 U 1 1 5BBAA814
 P 5750 2800
-AR Path="/5BBAA814" Ref="U5"  Part="1"
-AR Path="/5BB4DA56/5BBAA814" Ref="U5"  Part="1"
-F 0 "U5" H 5750 2300 60  0000 C CNN
+AR Path="/5BBAA814" Ref="U?"  Part="1"
+AR Path="/5BB4DA56/5BBAA814" Ref="U11"  Part="1"
+F 0 "U11" H 5750 2300 60  0000 C CNN
 F 1 "MC74HC125ADTR2G" H 5750 3300 60  0000 C CNN
 F 2 "custom-footprints:MC74HC125A_TSSOP−14" H 5750 2800 60  0001 C CNN
@@
 $EndComp
 $Comp
-L power:GND #PWR0122
+L power:GND #PWR052
 U 1 1 5BBAAC4D
 P 7600 5650
-F 0 "#PWR0122" H 7600 5400 50  0001 C CNN
+F 0 "#PWR052" H 7600 5400 50  0001 C CNN
 F 1 "GND" H 7600 5500 50  0000 C CNN
 F 2 "" H 7600 5650 50  0001 C CNN
@@
 	7600 5300 7600 5650
 $Comp
-L power:GND #PWR0123
+L power:GND #PWR044
 U 1 1 5BBAAE22
 P 4100 2550
-F 0 "#PWR0123" H 4100 2300 50  0001 C CNN
+F 0 "#PWR044" H 4100 2300 50  0001 C CNN
 F 1 "GND" H 4100 2400 50  0000 C CNN
 F 2 "" H 4100 2550 50  0001 C CNN
@@
 $EndComp
 $Comp
-L power:GND #PWR0124
+L power:GND #PWR045
 U 1 1 5BBAAE4E
 P 4100 2850
-F 0 "#PWR0124" H 4100 2600 50  0001 C CNN
+F 0 "#PWR045" H 4100 2600 50  0001 C CNN
 F 1 "GND" H 4100 2700 50  0000 C CNN
 F 2 "" H 4100 2850 50  0001 C CNN
@@
 $EndComp
 $Comp
-L power:GND #PWR0125
+L power:GND #PWR046
 U 1 1 5BBAAE80
 P 4100 3150
-F 0 "#PWR0125" H 4100 2900 50  0001 C CNN
+F 0 "#PWR046" H 4100 2900 50  0001 C CNN
 F 1 "GND" H 4100 3000 50  0000 C CNN
 F 2 "" H 4100 3150 50  0001 C CNN
@@
 $EndComp
 $Comp
-L power:GND #PWR0126
+L power:GND #PWR050
 U 1 1 5BBAAE94
 P 7000 2600
-F 0 "#PWR0126" H 7000 2350 50  0001 C CNN
+F 0 "#PWR050" H 7000 2350 50  0001 C CNN
 F 1 "GND" H 7000 2450 50  0000 C CNN
 F 2 "" H 7000 2600 50  0001 C CNN
@@
 $EndComp
 $Comp
-L power:GND #PWR0127
+L power:GND #PWR051
 U 1 1 5BBAAEA8
 P 7050 2900
-F 0 "#PWR0127" H 7050 2650 50  0001 C CNN
+F 0 "#PWR051" H 7050 2650 50  0001 C CNN
 F 1 "GND" H 7050 2750 50  0000 C CNN
 F 2 "" H 7050 2900 50  0001 C CNN
@@
 Wire Wire Line
 	5250 2900 4700 2900
-Text Label 4700 2700 0    60   ~ 0
+Text Label 4700 2600 0    60   ~ 0
 SD_DATA_OUT
-Text HLabel 4700 2600 0    60   Output ~ 0
+Text HLabel 4700 2700 0    60   Output ~ 0
 SD_DATA_OUT_BUF
 Text HLabel 4700 2900 0    60   Input ~ 0
@@
 	6300 2500 6400 2500
 $Comp
-L Device:R R25
+L Device:R R39
 U 1 1 5BBAB32F
 P 7300 2550
-F 0 "R25" V 7380 2550 50  0000 C CNN
+F 0 "R39" V 7380 2550 50  0000 C CNN
 F 1 "10k" V 7300 2550 50  0000 C CNN
-F 2 "digikey-footprints:0603" V 7230 2550 50  0001 C CNN
+F 2 "Resistor_SMD:R_0603_1608Metric_Pad1.05x0.95mm_HandSolder" V 7230 2550 50  0001 C CNN
 F 3 "" H 7300 2550 50  0001 C CNN
 	1    7300 2550
@@
 Connection ~ 6400 2500
 $Comp
-L Device:C C20
+L Device:C C29
 U 1 1 5BBAB4F4
 P 6400 2150
-F 0 "C20" H 6425 2250 50  0000 L CNN
+F 0 "C29" H 6425 2250 50  0000 L CNN
 F 1 "100n" H 6425 2050 50  0000 L CNN
-F 2 "digikey-footprints:0603" H 6438 2000 50  0001 C CNN
+F 2 "Capacitor_SMD:C_0603_1608Metric_Pad1.05x0.95mm_HandSolder" H 6438 2000 50  0001 C CNN
 F 3 "" H 6400 2150 50  0001 C CNN
 	1    6400 2150
@@
 	6700 1900 6700 2000
 $Comp
-L power:GND #PWR0128
+L power:GND #PWR049
 U 1 1 5BBAB570
 P 6700 2000
-F 0 "#PWR0128" H 6700 1750 50  0001 C CNN
+F 0 "#PWR049" H 6700 1750 50  0001 C CNN
 F 1 "GND" H 6700 1850 50  0000 C CNN
 F 2 "" H 6700 2000 50  0001 C CNN
@@
 SD_DATA_IN
 $Comp
-L Device:C C19
+L Device:C C27
 U 1 1 5BBABB37
 P 3800 5050
-F 0 "C19" H 3825 5150 50  0000 L CNN
+F 0 "C27" H 3825 5150 50  0000 L CNN
 F 1 "100n" H 3825 4950 50  0000 L CNN
-F 2 "digikey-footprints:0603" H 3838 4900 50  0001 C CNN
+F 2 "Capacitor_SMD:C_0603_1608Metric_Pad1.05x0.95mm_HandSolder" H 3838 4900 50  0001 C CNN
 F 3 "" H 3800 5050 50  0001 C CNN
 	1    3800 5050
@@
 	3800 4700 3800 4900
 $Comp
-L power:GND #PWR0129
+L power:GND #PWR042
 U 1 1 5BBABC51
 P 3800 5350
-F 0 "#PWR0129" H 3800 5100 50  0001 C CNN
+F 0 "#PWR042" H 3800 5100 50  0001 C CNN
 F 1 "GND" H 3800 5200 50  0000 C CNN
 F 2 "" H 3800 5350 50  0001 C CNN
@@
 	4050 4900 4050 5350
 $Comp
-L power:GND #PWR0130
+L power:GND #PWR043
 U 1 1 5BBABFC7
 P 4050 5350
-F 0 "#PWR0130" H 4050 5100 50  0001 C CNN
+F 0 "#PWR043" H 4050 5100 50  0001 C CNN
 F 1 "GND" H 4050 5200 50  0000 C CNN
 F 2 "" H 4050 5350 50  0001 C CNN
@@
 	3800 4700 5550 4700
 $Comp
-L Connector_Generic:Conn_02x02_Odd_Even J7
+L Connector_Generic:Conn_02x02_Odd_Even J12
 U 1 1 5BC2A0E4
 P 2900 1450
-F 0 "J7" H 2950 1667 50  0000 C CNN
+F 0 "J12" H 2950 1667 50  0000 C CNN
 F 1 "Conn_02x02_Odd_Even" H 2950 1576 50  0000 C CNN
-F 2 "Pin_Headers:Pin_Header_Straight_2x02_Pitch2.54mm_SMD" H 2900 1450 50  0001 C CNN
+F 2 "Connector_PinSocket_2.54mm:PinSocket_2x02_P2.54mm_Vertical" H 2900 1450 50  0001 C CNN
 F 3 "~" H 2900 1450 50  0001 C CNN
 	1    2900 1450
@@
 	5250 3000 4700 3000
 $Comp
-L Connector:Micro_SD_Card_Det J8
+L CameraSystem-rescue:Micro_SD_Card_Det-Connector J?
 U 1 1 5BC308F6
 P 6450 4800
-F 0 "J8" H 6400 5617 50  0000 C CNN
+AR Path="/5BC308F6" Ref="J?"  Part="1"
+AR Path="/5BB4DA56/5BC308F6" Ref="J13"  Part="1"
+F 0 "J13" H 6400 5617 50  0000 C CNN
 F 1 "DM3D-SF" H 6400 5526 50  0000 C CNN
 F 2 "custom-footprints:DM3D-SF" H 8500 5500 50  0001 C CNN
@@
 	7250 5300 7600 5300
 $Comp
-L Device:R R12
+L Device:R R38
 U 1 1 5BC30B28
 P 5150 5200
-F 0 "R12" V 5230 5200 50  0000 C CNN
+F 0 "R38" V 5230 5200 50  0000 C CNN
 F 1 "10k" V 5150 5200 50  0000 C CNN
-F 2 "digikey-footprints:0603" V 5080 5200 50  0001 C CNN
+F 2 "Resistor_SMD:R_0603_1608Metric_Pad1.05x0.95mm_HandSolder" V 5080 5200 50  0001 C CNN
 F 3 "" H 5150 5200 50  0001 C CNN
 	1    5150 5200
@@
 $EndComp
 $Comp
-L Device:C C27
+L Device:C C28
 U 1 1 5BC32E9B
 P 5400 5750
-F 0 "C27" H 5425 5850 50  0000 L CNN
+F 0 "C28" H 5425 5850 50  0000 L CNN
 F 1 "100n" H 5425 5650 50  0000 L CNN
-F 2 "digikey-footprints:0603" H 5438 5600 50  0001 C CNN
+F 2 "Capacitor_SMD:C_0603_1608Metric_Pad1.05x0.95mm_HandSolder" H 5438 5600 50  0001 C CNN
 F 3 "" H 5400 5750 50  0001 C CNN
 	1    5400 5750
@@
 $EndComp
 $Comp
-L power:GND #PWR05
+L power:GND #PWR047
 U 1 1 5BC32EF7
 P 5400 6050
-F 0 "#PWR05" H 5400 5800 50  0001 C CNN
+F 0 "#PWR047" H 5400 5800 50  0001 C CNN
 F 1 "GND" H 5400 5900 50  0000 C CNN
 F 2 "" H 5400 6050 50  0001 C CNN
@@
 	5550 5300 5550 5500
 $Comp
-L power:GND #PWR07
+L power:GND #PWR048
 U 1 1 5BC7AC6D
 P 5550 5500
-F 0 "#PWR07" H 5550 5250 50  0001 C CNN
+F 0 "#PWR048" H 5550 5250 50  0001 C CNN
 F 1 "GND" H 5550 5350 50  0000 C CNN
 F 2 "" H 5550 5500 50  0001 C CNN

Commit message: camera was updated
Parts:
- J11: renamed from J13; footprint custom-footprints:DM3D-SF -> Connector_Card:microSD_HC_Hirose_DM3D-SF
- renumbered C27 to C24, C28 to C25, C29 to C26, J12 to J10, R38 to R31, R39 to R32, U11 to U10
Changed lines of the file:
@@
 $Descr A4 11693 8268
 encoding utf-8
-Sheet 9 9
+Sheet 8 9
 Title ""
 Date ""
@@
 P 5750 2800
 AR Path="/5BBAA814" Ref="U?"  Part="1"
-AR Path="/5BB4DA56/5BBAA814" Ref="U11"  Part="1"
-F 0 "U11" H 5750 2300 60  0000 C CNN
+AR Path="/5BB4DA56/5BBAA814" Ref="U10"  Part="1"
+F 0 "U10" H 5750 2300 60  0000 C CNN
 F 1 "MC74HC125ADTR2G" H 5750 3300 60  0000 C CNN
 F 2 "custom-footprints:MC74HC125A_TSSOP−14" H 5750 2800 60  0001 C CNN
@@
 $EndComp
 $Comp
-L power:GND #PWR052
+L power:GND #PWR046
 U 1 1 5BBAAC4D
 P 7600 5650
-F 0 "#PWR052" H 7600 5400 50  0001 C CNN
+F 0 "#PWR046" H 7600 5400 50  0001 C CNN
 F 1 "GND" H 7600 5500 50  0000 C CNN
 F 2 "" H 7600 5650 50  0001 C CNN
@@
 	7600 5300 7600 5650
 $Comp
-L power:GND #PWR044
+L power:GND #PWR038
 U 1 1 5BBAAE22
 P 4100 2550
-F 0 "#PWR044" H 4100 2300 50  0001 C CNN
+F 0 "#PWR038" H 4100 2300 50  0001 C CNN
 F 1 "GND" H 4100 2400 50  0000 C CNN
 F 2 "" H 4100 2550 50  0001 C CNN
@@
 $EndComp
 $Comp
-L power:GND #PWR045
+L power:GND #PWR039
 U 1 1 5BBAAE4E
 P 4100 2850
-F 0 "#PWR045" H 4100 2600 50  0001 C CNN
+F 0 "#PWR039" H 4100 2600 50  0001 C CNN
 F 1 "GND" H 4100 2700 50  0000 C CNN
 F 2 "" H 4100 2850 50  0001 C CNN
@@
 $EndComp
 $Comp
-L power:GND #PWR046
+L power:GND #PWR040
 U 1 1 5BBAAE80
 P 4100 3150
-F 0 "#PWR046" H 4100 2900 50  0001 C CNN
+F 0 "#PWR040" H 4100 2900 50  0001 C CNN
 F 1 "GND" H 4100 3000 50  0000 C CNN
 F 2 "" H 4100 3150 50  0001 C CNN
@@
 $EndComp
 $Comp
-L power:GND #PWR050
+L power:GND #PWR044
 U 1 1 5BBAAE94
 P 7000 2600
-F 0 "#PWR050" H 7000 2350 50  0001 C CNN
+F 0 "#PWR044" H 7000 2350 50  0001 C CNN
 F 1 "GND" H 7000 2450 50  0000 C CNN
 F 2 "" H 7000 2600 50  0001 C CNN
@@
 $EndComp
 $Comp
-L power:GND #PWR051
+L power:GND #PWR045
 U 1 1 5BBAAEA8
 P 7050 2900
-F 0 "#PWR051" H 7050 2650 50  0001 C CNN
+F 0 "#PWR045" H 7050 2650 50  0001 C CNN
 F 1 "GND" H 7050 2750 50  0000 C CNN
 F 2 "" H 7050 2900 50  0001 C CNN
@@
 	6300 2500 6400 2500
 $Comp
-L Device:R R39
+L Device:R R32
 U 1 1 5BBAB32F
 P 7300 2550
-F 0 "R39" V 7380 2550 50  0000 C CNN
+F 0 "R32" V 7380 2550 50  0000 C CNN
 F 1 "10k" V 7300 2550 50  0000 C CNN
 F 2 "Resistor_SMD:R_0603_1608Metric_Pad1.05x0.95mm_HandSolder" V 7230 2550 50  0001 C CNN
@@
 Connection ~ 6400 2500
 $Comp
-L Device:C C29
+L Device:C C26
 U 1 1 5BBAB4F4
 P 6400 2150
-F 0 "C29" H 6425 2250 50  0000 L CNN
+F 0 "C26" H 6425 2250 50  0000 L CNN
 F 1 "100n" H 6425 2050 50  0000 L CNN
 F 2 "Capacitor_SMD:C_0603_1608Metric_Pad1.05x0.95mm_HandSolder" H 6438 2000 50  0001 C CNN
@@
 	6700 1900 6700 2000
 $Comp
-L power:GND #PWR049
+L power:GND #PWR043
 U 1 1 5BBAB570
 P 6700 2000
-F 0 "#PWR049" H 6700 1750 50  0001 C CNN
+F 0 "#PWR043" H 6700 1750 50  0001 C CNN
 F 1 "GND" H 6700 1850 50  0000 C CNN
 F 2 "" H 6700 2000 50  0001 C CNN
@@
 SD_DATA_IN
 $Comp
-L Device:C C27
+L Device:C C24
 U 1 1 5BBABB37
 P 3800 5050
-F 0 "C27" H 3825 5150 50  0000 L CNN
+F 0 "C24" H 3825 5150 50  0000 L CNN
 F 1 "100n" H 3825 4950 50  0000 L CNN
 F 2 "Capacitor_SMD:C_0603_1608Metric_Pad1.05x0.95mm_HandSolder" H 3838 4900 50  0001 C CNN
@@
 	3800 4700 3800 4900
 $Comp
-L power:GND #PWR042
+L power:GND #PWR036
 U 1 1 5BBABC51
 P 3800 5350
-F 0 "#PWR042" H 3800 5100 50  0001 C CNN
+F 0 "#PWR036" H 3800 5100 50  0001 C CNN
 F 1 "GND" H 3800 5200 50  0000 C CNN
 F 2 "" H 3800 5350 50  0001 C CNN
@@
 	4050 4900 4050 5350
 $Comp
-L power:GND #PWR043
+L power:GND #PWR037
 U 1 1 5BBABFC7
 P 4050 5350
-F 0 "#PWR043" H 4050 5100 50  0001 C CNN
+F 0 "#PWR037" H 4050 5100 50  0001 C CNN
 F 1 "GND" H 4050 5200 50  0000 C CNN
 F 2 "" H 4050 5350 50  0001 C CNN
@@
 	3800 4700 5550 4700
 $Comp
-L Connector_Generic:Conn_02x02_Odd_Even J12
+L Connector_Generic:Conn_02x02_Odd_Even J10
 U 1 1 5BC2A0E4
 P 2900 1450
-F 0 "J12" H 2950 1667 50  0000 C CNN
+F 0 "J10" H 2950 1667 50  0000 C CNN
 F 1 "Conn_02x02_Odd_Even" H 2950 1576 50  0000 C CNN
 F 2 "Connector_PinSocket_2.54mm:PinSocket_2x02_P2.54mm_Vertical" H 2900 1450 50  0001 C CNN
@@
 P 6450 4800
 AR Path="/5BC308F6" Ref="J?"  Part="1"
-AR Path="/5BB4DA56/5BC308F6" Ref="J13"  Part="1"
-F 0 "J13" H 6400 5617 50  0000 C CNN
+AR Path="/5BB4DA56/5BC308F6" Ref="J11"  Part="1"
+F 0 "J11" H 6400 5617 50  0000 C CNN
 F 1 "DM3D-SF" H 6400 5526 50  0000 C CNN
-F 2 "custom-footprints:DM3D-SF" H 8500 5500 50  0001 C CNN
+F 2 "Connector_Card:microSD_HC_Hirose_DM3D-SF" H 8500 5500 50  0001 C CNN
 F 3 "https://www.hirose.com/product/en/download_file/key_name/DM3/category/Catalog/doc_file_id/49662/?file_category_id=4&item_id=195&is_series=1" H 6450 4900 50  0001 C CNN
 	1    6450 4800
@@
 	7250 5300 7600 5300
 $Comp
-L Device:R R38
+L Device:R R31
 U 1 1 5BC30B28
 P 5150 5200
-F 0 "R38" V 5230 5200 50  0000 C CNN
+F 0 "R31" V 5230 5200 50  0000 C CNN
 F 1 "10k" V 5150 5200 50  0000 C CNN
 F 2 "Resistor_SMD:R_0603_1608Metric_Pad1.05x0.95mm_HandSolder" V 5080 5200 50  0001 C CNN
@@
 $EndComp
 $Comp
-L Device:C C28
+L Device:C C25
 U 1 1 5BC32E9B
 P 5400 5750
-F 0 "C28" H 5425 5850 50  0000 L CNN
+F 0 "C25" H 5425 5850 50  0000 L CNN
 F 1 "100n" H 5425 5650 50  0000 L CNN
 F 2 "Capacitor_SMD:C_0603_1608Metric_Pad1.05x0.95mm_HandSolder" H 5438 5600 50  0001 C CNN
@@
 $EndComp
 $Comp
-L power:GND #PWR047
+L power:GND #PWR041
 U 1 1 5BC32EF7
 P 5400 6050
-F 0 "#PWR047" H 5400 5800 50  0001 C CNN
+F 0 "#PWR041" H 5400 5800 50  0001 C CNN
 F 1 "GND" H 5400 5900 50  0000 C CNN
 F 2 "" H 5400 6050 50  0001 C CNN
@@
 	5550 5300 5550 5500
 $Comp
-L power:GND #PWR048
+L power:GND #PWR042
 U 1 1 5BC7AC6D
 P 5550 5500
-F 0 "#PWR048" H 5550 5250 50  0001 C CNN
+F 0 "#PWR042" H 5550 5250 50  0001 C CNN
 F 1 "GND" H 5550 5350 50  0000 C CNN
 F 2 "" H 5550 5500 50  0001 C CNN
