File: Projects/CameraSystem/Schematics/Camera.sch (KiCad schematic (older format))
At the start: 0 parts

Commit message: feat: first draft of uc schematic created
Parts:
- added C? (x2): 100n, symbol C
- added J? (x2): CONN_02X02, symbol CONN_02X02
- added Q?: BC846B_215, digikey-footprints:SOT-23-3, symbol BC846B_215
- added R? (x2): 10k, symbol R
- added R?: 4k7, symbol R
- added U?: OV7670, symbol OV7670
- added U?: SIT2001BI-S2-33E-24.000000G, symbol SIT2001BI-S2-33E-24.000000G
Connections:
- net labels added: CAM_CLK, CAM_D0, CAM_D1, CAM_D2, CAM_D3, CAM_D4, CAM_D5, CAM_D6, CAM_D7, CAM_HSYNC, CAM_PCLK, CAM_VSYNC, CAM_XCLK_CTL, GND, SCL_3V3, SDA_3V3, VDD_3V3, VDD_3V3_IN
- wire segments 0 -> 51
- no-connect marks 0 -> 1
Other:
- note added: "Clock can be generated either by uc (10MHz) or by external osc (24MHz)"

Commit message: feat: 3.3 regulator housing changed due to temperature
Parts:
- C? (x2): symbol C -> Device:C
- J? (x2): symbol CONN_02X02 -> CameraSystem-rescue:CONN_02X02
- Q?: symbol BC846B_215 -> CameraSystem-rescue:BC846B_215
- R? (x3): symbol R -> Device:R
- U?: symbol OV7670 -> cl-integrated_circuits:OV7670
- U?: symbol SIT2001BI-S2-33E-24.000000G -> cl-integrated_circuits:SIT2001BI-S2-33E-24.000000G
Changed lines of the file:
@@
-EESchema Schematic File Version 2
-LIBS:cl-connectors
-LIBS:dk_Addressable-Specialty
-LIBS:dk_Alarms-Buzzers-and-Sirens
-LIBS:dk_Automotive-Relays
-LIBS:dk_Balun
-LIBS:dk_Barrel-Audio-Connectors
-LIBS:dk_Battery-Holders-Clips-Contacts
-LIBS:dk_Clock-Timing-Clock-Generators-PLLs-Frequency-Synthesizers
-LIBS:dk_Clock-Timing-Programmable-Timers-and-Oscillators
-LIBS:dk_Clock-Timing-Real-Time-Clocks
-LIBS:dk_Coaxial-Connectors-RF
-LIBS:dk_Current-Transducers
-LIBS:dk_Data-Acquisition-ADCs-DACs-Special-Purpose
-LIBS:dk_Data-Acquisition-Analog-to-Digital-Converters-ADC
-LIBS:dk_Data-Acquisition-Digital-Potentiometers
-LIBS:dk_Data-Acquisition-Digital-to-Analog-Converters-DAC
-LIBS:dk_Data-Acquisition-Touch-Screen-Controllers
-LIBS:dk_DC-DC-Converters
-LIBS:dk_Digital-Isolators
-LIBS:dk_Diodes-Bridge-Rectifiers
-LIBS:dk_Diodes-Rectifiers-Arrays
-LIBS:dk_Diodes-Rectifiers-Single
-LIBS:dk_Diodes-Zener-Single
-LIBS:dk_Display-Modules-LCD-OLED-Graphic
-LIBS:dk_Display-Modules-LED-Character-and-Numeric
-LIBS:dk_D-Sub-Connectors
-LIBS:dk_Embedded-Microcontrollers
-LIBS:dk_Encoders
-LIBS:dk_Evaluation-Boards-Sensors
-LIBS:dk_Ferrite-Beads-and-Chips
-LIBS:dk_Fixed-Inductors
-LIBS:dk_Fuses
-LIBS:dk_Gas-Sensors
-LIBS:dk_Humidity-Moisture-Sensors
-LIBS:dk_Image-Sensors-Camera
-LIBS:dk_Infrared-UV-Visible-Emitters
-LIBS:dk_Inrush-Current-Limiters-ICL
-LIBS:dk_Interface-Analog-Switches-Multiplexers-Demultiplexers
-LIBS:dk_Interface-Analog-Switches-Special-Purpose
-LIBS:dk_Interface-Controllers
-LIBS:dk_Interface-Drivers-Receivers-Transceivers
-LIBS:dk_Interface-I-O-Expanders
-LIBS:dk_Interface-Modules
-LIBS:dk_Interface-Sensor-and-Detector-Interfaces
-LIBS:dk_Interface-Sensor-Capacitive-Touch
-LIBS:dk_Interface-Specialized
-LIBS:dk_LED-Indication-Discrete
-LIBS:dk_LEDs-Circuit-Board-Indicators-Arrays-Light-Bars-Bar-Graphs
-LIBS:dk_Linear-Amplifiers-Audio
-LIBS:dk_Linear-Amplifiers-Instrumentation-OP-Amps-Buffer-Amps
-LIBS:dk_Linear-Comparators
-LIBS:dk_Logic-Buffers-Drivers-Receivers-Transceivers
-LIBS:dk_Logic-Flip-Flops
-LIBS:dk_Logic-Gates-and-Inverters
-LIBS:dk_Logic-Multivibrators
-LIBS:dk_Logic-Shift-Registers
-LIBS:dk_Logic-Signal-Switches-Multiplexers-Decoders
-LIBS:dk_Logic-Translators-Level-Shifters
-LIBS:dk_Magnetic-Sensors-Compass-Magnetic-Field-Modules
-LIBS:dk_Magnetic-Sensors-Linear-Compass-ICs
-LIBS:dk_Magnetic-Sensors-Switches-Solid-State
-LIBS:dk_Memory
-LIBS:dk_Memory-Connectors-PC-Card-Sockets
-LIBS:dk_Microphones
-LIBS:dk_Modular-Connectors-Jacks
-LIBS:dk_Modular-Connectors-Jacks-With-Magnetics
-LIBS:dk_Motion-Sensors-Accelerometers
-LIBS:dk_Motion-Sensors-IMUs-Inertial-Measurement-Units
-LIBS:dk_Motion-Sensors-Tilt-Switches
-LIBS:dk_Navigation-Switches-Joystick
-LIBS:dk_Optical-Sensors-Ambient-Light-IR-UV-Sensors
-LIBS:dk_Optical-Sensors-Photo-Detectors-Remote-Receiver
-LIBS:dk_Optical-Sensors-Photodiodes
-LIBS:dk_Optical-Sensors-Phototransistors
-LIBS:dk_Optical-Sensors-Reflective-Analog-Output
-LIBS:dk_Optoisolators-Logic-Output
-LIBS:dk_Optoisolators-Transistor-Photovoltaic-Output
-LIBS:dk_Optoisolators-Triac-SCR-Output
-LIBS:dk_Oscillators
-LIBS:dk_PMIC-AC-DC-Converters-Offline-Switchers
-LIBS:dk_PMIC-Battery-Chargers
-LIBS:dk_PMIC-Battery-Management
-LIBS:dk_PMIC-Current-Regulation-Management
-LIBS:dk_PMIC-Full-Half-Bridge-Drivers
-LIBS:dk_PMIC-Gate-Drivers
-LIBS:dk_PMIC-LED-Drivers
-LIBS:dk_PMIC-Motor-Drivers-Controllers
-LIBS:dk_PMIC-OR-Controllers-Ideal-Diodes
-LIBS:dk_PMIC-Power-Distribution-Switches-Load-Drivers
-LIBS:dk_PMIC-Power-Management-Specialized
-LIBS:dk_PMIC-RMS-to-DC-Converters
-LIBS:dk_PMIC-Supervisors
-LIBS:dk_PMIC-Thermal-Management
-LIBS:dk_PMIC-V-F-and-F-V-Converters
-LIBS:dk_PMIC-Voltage-Reference
-LIBS:dk_PMIC-Voltage-Regulators-DC-DC-Switching-Controllers
-LIBS:dk_PMIC-Voltage-Regulators-DC-DC-Switching-Regulators
-LIBS:dk_PMIC-Voltage-Regulators-Linear
-LIBS:dk_PMIC-Voltage-Regulators-Special-Purpose
-LIBS:dk_Power-Relays-Over-2-Amps
-LIBS:dk_Pressure-Sensors-Transducers
-LIBS:dk_Programmable-Oscillators
-LIBS:dk_Pushbutton-Switches
-LIBS:dk_Rectangular-Connectors-Headers-Male-Pins
-LIBS:dk_Reed-Relays
-LIBS:dk_Resistor-Networks-Arrays
-LIBS:dk_RF-Amplifiers
-LIBS:dk_RF-Antennas
-LIBS:dk_RF-Demodulators
-LIBS:dk_RF-Detectors
-LIBS:dk_RF-Evaluation-and-Development-Kits-Boards
-LIBS:dk_RFID-RF-Access-Monitoring-ICs
-LIBS:dk_RF-Receivers
-LIBS:dk_RF-Switches
-LIBS:dk_RF-Transceiver-ICs
-LIBS:dk_RF-Transceiver-Modules
-LIBS:dk_RF-Transmitters
-LIBS:dk_Rotary-Potentiometers-Rheostats
-LIBS:dk_Sensors-Transducers_Accessories
-LIBS:dk_Signal-Relays-Up-to-2-Amps
-LIBS:dk_Slide-Switches
-LIBS:dk_Solid-State-Relays
-LIBS:dk_Specialized-ICs
-LIBS:dk_Specialized-Sensors
-LIBS:dk_Surge-Suppression-ICs
-LIBS:dk_Tactile-Switches
-LIBS:dk_Temperature-Sensors-Analog-and-Digital-Output
-LIBS:dk_Thermal-Cutoffs-Thermal-Fuses
-LIBS:dk_Thyristors-DIACs-SIDACs
-LIBS:dk_Thyristors-SCRs
-LIBS:dk_Thyristors-TRIACs
-LIBS:dk_Toggle-Switches
-LIBS:dk_Transistors-Bipolar-BJT-Arrays
-LIBS:dk_Transistors-Bipolar-BJT-RF
-LIBS:dk_Transistors-Bipolar-BJT-Single
-LIBS:dk_Transistors-Bipolar-BJT-Single-Pre-Biased
-LIBS:dk_Transistors-FETs-MOSFETs-Arrays
-LIBS:dk_Transistors-FETs-MOSFETs-RF
-LIBS:dk_Transistors-FETs-MOSFETs-Single
-LIBS:dk_Transistors-JFETs
-LIBS:dk_Trimmer-Potentiometers
-LIBS:dk_TVS-Diodes
-LIBS:dk_TVS-Mixed-Technology
-LIBS:dk_USB-DVI-HDMI-Connectors
-LIBS:power
-LIBS:device
-LIBS:transistors
-LIBS:conn
-LIBS:linear
-LIBS:regul
-LIBS:74xx
-LIBS:cmos4000
-LIBS:adc-dac
-LIBS:memory
-LIBS:xilinx
-LIBS:microcontrollers
-LIBS:dsp
-LIBS:microchip
-LIBS:analog_switches
-LIBS:motorola
-LIBS:texas
-LIBS:intel
-LIBS:audio
-LIBS:interface
-LIBS:digital-audio
-LIBS:philips
-LIBS:display
-LIBS:cypress
-LIBS:siliconi
-LIBS:opto
-LIBS:atmel
-LIBS:contrib
-LIBS:valves
-LIBS:cl-integrated_circuits
-LIBS:cl-misc
+EESchema Schematic File Version 4
 LIBS:CameraSystem-cache
-EELAYER 25 0
+EELAYER 26 0
 EELAYER END
 $Descr A4 11693 8268
@@
 $EndDescr
 $Comp
-L OV7670 U?
+L cl-integrated_circuits:OV7670 U?
 U 1 1 5BBB684E
 P 5350 3050
@@
 VDD_3V3
 $Comp
-L CONN_02X02 J?
+L CameraSystem-rescue:CONN_02X02 J?
 U 1 1 5BBB690A
 P 2700 1550
@@
 VDD_3V3_IN
 $Comp
-L C C?
+L Device:C C?
 U 1 1 5BBB6CC1
 P 4800 2200
@@
 $EndComp
 $Comp
-L GND #PWR?
+L power:GND #PWR?
 U 1 1 5BBB6D0A
 P 4800 2400
@@
 	7150 2700 7150 2750
 $Comp
-L GND #PWR?
+L power:GND #PWR?
 U 1 1 5BBB6FDB
 P 7150 2750
@@
 CAM_HSYNC
 $Comp
-L CONN_02X02 J?
+L CameraSystem-rescue:CONN_02X02 J?
 U 1 1 5BBB9C5D
 P 7750 3000
@@
 CAM_CLK
 $Comp
-L SIT2001BI-S2-33E-24.000000G U?
+L cl-integrated_circuits:SIT2001BI-S2-33E-24.000000G U?
 U 1 1 5BBBA2DE
 P 7700 4050
@@
 $EndComp
 $Comp
-L GND #PWR?
+L power:GND #PWR?
 U 1 1 5BBBA416
 P 7550 4650
@@
 VDD_3V3_IN
 $Comp
-L C C?
+L Device:C C?
 U 1 1 5BBBA5A8
 P 6500 4350
@@
 Connection ~ 6500 4050
 $Comp
-L GND #PWR?
+L power:GND #PWR?
 U 1 1 5BBBA64E
 P 6500 4650
@@
 NoConn ~ 7700 3650
 $Comp
-L R R?
+L Device:R R?
 U 1 1 5BBBA862
 P 8250 4700
@@
 	8250 4850 8250 5050
 $Comp
-L BC846B_215 Q?
+L CameraSystem-rescue:BC846B_215 Q?
 U 1 1 5BBBB096
 P 8350 5250
@@
 $EndComp
 $Comp
-L R R?
+L Device:R R?
 U 1 1 5BBBB16C
 P 8750 5500
@@
 $EndComp
 $Comp
-L GND #PWR?
+L power:GND #PWR?
 U 1 1 5BBBB1AD
 P 8250 5750
@@
 	8250 5450 8250 5750
 $Comp
-L R R?
+L Device:R R?
 U 1 1 5BBBB238
 P 9050 5250

Commit message: feat: add debugging pins
Parts:
- removed J? (x2): CONN_02X02, symbol CameraSystem-rescue:CONN_02X02
- added J? (x2): Conn_02x02_Odd_Even, symbol Connector_Generic:Conn_02x02_Odd_Even
Connections:
- wire segments 51 -> 59
Changed lines of the file:
@@
 Text HLabel 2150 1550 0    60   Input ~ 0
 VDD_3V3
-$Comp
-L CameraSystem-rescue:CONN_02X02 J?
-U 1 1 5BBB690A
-P 2700 1550
-F 0 "J?" H 2700 1700 50  0000 C CNN
-F 1 "CONN_02X02" H 2700 1400 50  0000 C CNN
-F 2 "" H 2700 350 50  0001 C CNN
-F 3 "" H 2700 350 50  0001 C CNN
-	1    2700 1550
-	1    0    0    -1
-$EndComp
 Wire Wire Line
 	2450 1500 2400 1500
 Wire Wire Line
-	2400 1500 2400 1600
+	2400 1500 2400 1550
 Wire Wire Line
 	2400 1600 2450 1600
@@
 	2950 1500 3000 1500
 Wire Wire Line
-	3000 1500 3000 1600
+	3000 1500 3000 1550
 Wire Wire Line
 	3000 1600 2950 1600
@@
 VDD_3V3_IN
 Wire Wire Line
-	3750 2700 4850 2700
+	3750 2700 4550 2700
 Text Label 3750 2700 0    60   ~ 0
 VDD_3V3_IN
@@
 $EndComp
 $Comp
-L power:GND #PWR?
+L power:GND #PWR0131
 U 1 1 5BBB6D0A
 P 4800 2400
-F 0 "#PWR?" H 4800 2150 50  0001 C CNN
+F 0 "#PWR0131" H 4800 2150 50  0001 C CNN
 F 1 "GND" H 4800 2250 50  0000 C CNN
 F 2 "" H 4800 2400 50  0001 C CNN
@@
 	7150 2700 7150 2750
 $Comp
-L power:GND #PWR?
+L power:GND #PWR0132
 U 1 1 5BBB6FDB
 P 7150 2750
-F 0 "#PWR?" H 7150 2500 50  0001 C CNN
+F 0 "#PWR0132" H 7150 2500 50  0001 C CNN
 F 1 "GND" H 7150 2600 50  0000 C CNN
 F 2 "" H 7150 2750 50  0001 C CNN
@@
 Text HLabel 6400 2900 2    60   Output ~ 0
 CAM_HSYNC
-$Comp
-L CameraSystem-rescue:CONN_02X02 J?
-U 1 1 5BBB9C5D
-P 7750 3000
-F 0 "J?" H 7750 3150 50  0000 C CNN
-F 1 "CONN_02X02" H 7750 2850 50  0000 C CNN
-F 2 "" H 7750 1800 50  0001 C CNN
-F 3 "" H 7750 1800 50  0001 C CNN
-	1    7750 3000
-	1    0    0    -1
-$EndComp
 Wire Wire Line
 	7500 2950 7400 2950
 Wire Wire Line
-	7400 2950 7400 3050
+	7400 2950 7400 3000
 Wire Wire Line
 	7400 3050 7500 3050
@@
 $EndComp
 $Comp
-L power:GND #PWR?
+L power:GND #PWR0133
 U 1 1 5BBBA416
 P 7550 4650
-F 0 "#PWR?" H 7550 4400 50  0001 C CNN
+F 0 "#PWR0133" H 7550 4400 50  0001 C CNN
 F 1 "GND" H 7550 4500 50  0000 C CNN
 F 2 "" H 7550 4650 50  0001 C CNN
@@
 	7550 4500 7550 4650
 Wire Wire Line
-	6200 4050 7100 4050
+	6200 4050 6500 4050
 Text Label 6200 4050 0    60   ~ 0
 VDD_3V3_IN
@@
 Connection ~ 6500 4050
 $Comp
-L power:GND #PWR?
+L power:GND #PWR0134
 U 1 1 5BBBA64E
 P 6500 4650
-F 0 "#PWR?" H 6500 4400 50  0001 C CNN
+F 0 "#PWR0134" H 6500 4400 50  0001 C CNN
 F 1 "GND" H 6500 4500 50  0000 C CNN
 F 2 "" H 6500 4650 50  0001 C CNN
@@
 $EndComp
 Wire Wire Line
-	8250 4850 8250 5050
+	8250 4850 8250 4950
 $Comp
 L CameraSystem-rescue:BC846B_215 Q?
 U 1 1 5BBBB096
 P 8350 5250
+AR Path="/5BBBB096" Ref="Q?"  Part="1"
+AR Path="/5BB4DA63/5BBBB096" Ref="Q?"  Part="1"
 F 0 "Q?" H 8224 5416 60  0000 L CNN
 F 1 "BC846B_215" V 8556 5250 60  0000 C CNN
@@
 $EndComp
 $Comp
-L power:GND #PWR?
+L power:GND #PWR0135
 U 1 1 5BBBB1AD
 P 8250 5750
-F 0 "#PWR?" H 8250 5500 50  0001 C CNN
+F 0 "#PWR0135" H 8250 5500 50  0001 C CNN
 F 1 "GND" H 8250 5600 50  0000 C CNN
 F 2 "" H 8250 5750 50  0001 C CNN
@@
 $EndComp
 Wire Wire Line
-	8250 5450 8250 5750
+	8250 5450 8250 5700
 $Comp
 L Device:R R?
@@
 $EndComp
 Wire Wire Line
-	8550 5250 8900 5250
+	8550 5250 8750 5250
 Wire Wire Line
 	8750 5250 8750 5350
@@
 Text Notes 7600 2650 0    60   ~ 0
 Clock can be generated either by uc (10MHz) or by external osc (24MHz)
+Wire Wire Line
+	2400 1550 2400 1600
+Wire Wire Line
+	3000 1550 3000 1600
+Wire Wire Line
+	4550 2700 4850 2700
+Wire Wire Line
+	7400 3000 7400 3050
+Wire Wire Line
+	6500 4050 7100 4050
+Wire Wire Line
+	8750 5250 8900 5250
+Wire Wire Line
+	8250 5700 8250 5750
+Wire Wire Line
+	8250 4950 8250 5050
+$Comp
+L Connector_Generic:Conn_02x02_Odd_Even J?
+U 1 1 5BC287BF
+P 2650 1500
+F 0 "J?" H 2700 1717 50  0000 C CNN
+F 1 "Conn_02x02_Odd_Even" H 2700 1626 50  0000 C CNN
+F 2 "" H 2650 1500 50  0001 C CNN
+F 3 "~" H 2650 1500 50  0001 C CNN
+	1    2650 1500
+	1    0    0    -1
+$EndComp
+$Comp
+L Connector_Generic:Conn_02x02_Odd_Even J?
+U 1 1 5BC289B3
+P 7700 2950
+F 0 "J?" H 7750 3167 50  0000 C CNN
+F 1 "Conn_02x02_Odd_Even" H 7750 3076 50  0000 C CNN
+F 2 "" H 7700 2950 50  0001 C CNN
+F 3 "~" H 7700 2950 50  0001 C CNN
+	1    7700 2950
+	1    0    0    -1
+$EndComp
 $EndSCHEMATC

Commit message: feat: DRC run
Parts:
- C21, C22: renamed from C?; footprint (none) -> Capacitor_SMD:C_0603_1608Metric_Pad1.05x0.95mm_HandSolder
- R26, R27, R28: renamed from R?; footprint (none) -> Resistor_SMD:R_0603_1608Metric_Pad1.05x0.95mm_HandSolder
- gave numbers to parts that had none: 5
Changed lines of the file:
@@
 $EndDescr
 $Comp
-L cl-integrated_circuits:OV7670 U?
+L cl-integrated_circuits:OV7670 U6
 U 1 1 5BBB684E
 P 5350 3050
-F 0 "U?" H 5350 2550 60  0000 C CNN
+F 0 "U6" H 5350 2550 60  0000 C CNN
 F 1 "OV7670" H 5350 3550 60  0000 C CNN
 F 2 "" H 5350 3050 60  0001 C CNN
@@
 VDD_3V3_IN
 $Comp
-L Device:C C?
+L Device:C C21
 U 1 1 5BBB6CC1
 P 4800 2200
-F 0 "C?" H 4825 2300 50  0000 L CNN
+F 0 "C21" H 4825 2300 50  0000 L CNN
 F 1 "100n" H 4825 2100 50  0000 L CNN
-F 2 "" H 4838 2050 50  0001 C CNN
+F 2 "Capacitor_SMD:C_0603_1608Metric_Pad1.05x0.95mm_HandSolder" H 4838 2050 50  0001 C CNN
 F 3 "" H 4800 2200 50  0001 C CNN
 	1    4800 2200
@@
 CAM_CLK
 $Comp
-L cl-integrated_circuits:SIT2001BI-S2-33E-24.000000G U?
+L cl-integrated_circuits:SIT2001BI-S2-33E-24.000000G U7
 U 1 1 5BBBA2DE
 P 7700 4050
-F 0 "U?" H 7700 3700 60  0000 C CNN
+F 0 "U7" H 7700 3700 60  0000 C CNN
 F 1 "SIT2001BI-S2-33E-24.000000G" H 7700 4550 60  0000 C CNN
 F 2 "" H 7700 4050 60  0001 C CNN
@@
 VDD_3V3_IN
 $Comp
-L Device:C C?
+L Device:C C22
 U 1 1 5BBBA5A8
 P 6500 4350
-F 0 "C?" H 6525 4450 50  0000 L CNN
+F 0 "C22" H 6525 4450 50  0000 L CNN
 F 1 "100n" H 6525 4250 50  0000 L CNN
-F 2 "" H 6538 4200 50  0001 C CNN
+F 2 "Capacitor_SMD:C_0603_1608Metric_Pad1.05x0.95mm_HandSolder" H 6538 4200 50  0001 C CNN
 F 3 "" H 6500 4350 50  0001 C CNN
 	1    6500 4350
@@
 NoConn ~ 7700 3650
 $Comp
-L Device:R R?
+L Device:R R26
 U 1 1 5BBBA862
 P 8250 4700
-F 0 "R?" V 8330 4700 50  0000 C CNN
+F 0 "R26" V 8330 4700 50  0000 C CNN
 F 1 "10k" V 8250 4700 50  0000 C CNN
-F 2 "" V 8180 4700 50  0001 C CNN
+F 2 "Resistor_SMD:R_0603_1608Metric_Pad1.05x0.95mm_HandSolder" V 8180 4700 50  0001 C CNN
 F 3 "" H 8250 4700 50  0001 C CNN
 	1    8250 4700
@@
 P 8350 5250
 AR Path="/5BBBB096" Ref="Q?"  Part="1"
-AR Path="/5BB4DA63/5BBBB096" Ref="Q?"  Part="1"
-F 0 "Q?" H 8224 5416 60  0000 L CNN
+AR Path="/5BB4DA63/5BBBB096" Ref="Q2"  Part="1"
+F 0 "Q2" H 8224 5416 60  0000 L CNN
 F 1 "BC846B_215" V 8556 5250 60  0000 C CNN
 F 2 "digikey-footprints:SOT-23-3" H 8550 5450 60  0001 L CNN
@@
 $EndComp
 $Comp
-L Device:R R?
+L Device:R R27
 U 1 1 5BBBB16C
 P 8750 5500
-F 0 "R?" V 8830 5500 50  0000 C CNN
+F 0 "R27" V 8830 5500 50  0000 C CNN
 F 1 "10k" V 8750 5500 50  0000 C CNN
-F 2 "" V 8680 5500 50  0001 C CNN
+F 2 "Resistor_SMD:R_0603_1608Metric_Pad1.05x0.95mm_HandSolder" V 8680 5500 50  0001 C CNN
 F 3 "" H 8750 5500 50  0001 C CNN
 	1    8750 5500
@@
 	8250 5450 8250 5700
 $Comp
-L Device:R R?
+L Device:R R28
 U 1 1 5BBBB238
 P 9050 5250
-F 0 "R?" V 9130 5250 50  0000 C CNN
+F 0 "R28" V 9130 5250 50  0000 C CNN
 F 1 "4k7" V 9050 5250 50  0000 C CNN
-F 2 "" V 8980 5250 50  0001 C CNN
+F 2 "Resistor_SMD:R_0603_1608Metric_Pad1.05x0.95mm_HandSolder" V 8980 5250 50  0001 C CNN
 F 3 "" H 9050 5250 50  0001 C CNN
 	1    9050 5250
@@
 	8250 4950 8250 5050
 $Comp
-L Connector_Generic:Conn_02x02_Odd_Even J?
+L Connector_Generic:Conn_02x02_Odd_Even J9
 U 1 1 5BC287BF
 P 2650 1500
-F 0 "J?" H 2700 1717 50  0000 C CNN
+F 0 "J9" H 2700 1717 50  0000 C CNN
 F 1 "Conn_02x02_Odd_Even" H 2700 1626 50  0000 C CNN
 F 2 "" H 2650 1500 50  0001 C CNN
@@
 $EndComp
 $Comp
-L Connector_Generic:Conn_02x02_Odd_Even J?
+L Connector_Generic:Conn_02x02_Odd_Even J10
 U 1 1 5BC289B3
 P 7700 2950
-F 0 "J?" H 7750 3167 50  0000 C CNN
+F 0 "J10" H 7750 3167 50  0000 C CNN
 F 1 "Conn_02x02_Odd_Even" H 7750 3076 50  0000 C CNN
 F 2 "" H 7700 2950 50  0001 C CNN
