File: Projects/CameraSystem/Schematics/Microcontroller.sch (KiCad schematic (older format))
At the start: 0 parts

Commit message: feat:add led datasheets and microcontroler
Parts:
- added C? (x2): C, symbol C
- added D?: BZX84C3V3LT1G, SOT23-3, symbol D_Zener
- added R?: 10k, symbol R
- added S?: GPTS203211B, digikey-footprints:PushButton_12x12mm_THT_GPTS203211B, symbol GPTS203211B
- added U?: ATMEGA16A-AU, TQFP44, symbol ATMEGA16A-AU
- added Y?: Crystal, symbol Crystal
Connections:
- net labels added: GND, SPI_RST, SPI_RX, SPI_TX, UC_RST, VDD_3V3
- wire segments 0 -> 26
Changed lines of the file:
@@
 $Descr A4 11693 8268
 encoding utf-8
-Sheet 1 6
+Sheet 3 6
 Title ""
 Date ""
@@
 Comment4 ""
 $EndDescr
+Text HLabel 2350 900  0    60   Input ~ 0
+VDD_3V3
+Text HLabel 2350 1700 0    60   Input ~ 0
+SPI_RST
+Text HLabel 6650 4500 2    60   Output ~ 0
+SPI_TX
+Text HLabel 6650 4400 2    60   Input ~ 0
+SPI_RX
+$Comp
+L ATMEGA16A-AU U?
+U 1 1 5BB89FDE
+P 5250 3400
+F 0 "U?" H 4300 5280 50  0000 L BNN
+F 1 "ATMEGA16A-AU" H 5800 1450 50  0000 L BNN
+F 2 "TQFP44" H 5250 3400 50  0001 C CIN
+F 3 "" H 5250 3400 50  0001 C CNN
+	1    5250 3400
+	1    0    0    -1
+$EndComp
+Wire Wire Line
+	6350 4500 6650 4500
+Wire Wire Line
+	6350 4400 6650 4400
+Wire Wire Line
+	2350 1700 4150 1700
+Wire Wire Line
+	2350 900  5350 900
+Wire Wire Line
+	5350 900  5350 1400
+Wire Wire Line
+	5150 1400 5150 900
+Connection ~ 5150 900
+Wire Wire Line
+	5050 1400 5050 900
+Connection ~ 5050 900
+Wire Wire Line
+	4950 1400 4950 900
+Connection ~ 4950 900
+$Comp
+L GND #PWR?
+U 1 1 5BB8A17E
+P 5150 5550
+F 0 "#PWR?" H 5150 5300 50  0001 C CNN
+F 1 "GND" H 5150 5400 50  0000 C CNN
+F 2 "" H 5150 5550 50  0001 C CNN
+F 3 "" H 5150 5550 50  0001 C CNN
+	1    5150 5550
+	1    0    0    -1
+$EndComp
+Wire Wire Line
+	4950 5400 4950 5500
+Wire Wire Line
+	4950 5500 5350 5500
+Wire Wire Line
+	5350 5500 5350 5400
+Wire Wire Line
+	5150 5400 5150 5550
+Connection ~ 5150 5500
+Wire Wire Line
+	5050 5400 5050 5500
+Connection ~ 5050 5500
+$Comp
+L R R?
+U 1 1 5BB8AD84
+P 2700 1300
+F 0 "R?" V 2780 1300 50  0000 C CNN
+F 1 "10k" V 2700 1300 50  0000 C CNN
+F 2 "" V 2630 1300 50  0001 C CNN
+F 3 "" H 2700 1300 50  0001 C CNN
+	1    2700 1300
+	1    0    0    -1
+$EndComp
+Wire Wire Line
+	2700 900  2700 1150
+Connection ~ 2700 900
+Wire Wire Line
+	2700 1450 2700 1850
+Connection ~ 2700 1700
+$Comp
+L D_Zener D?
+U 1 1 5BB8ADE9
+P 3000 1300
+F 0 "D?" H 3000 1400 50  0000 C CNN
+F 1 "BZX84C3V3LT1G" H 3000 1200 50  0000 C CNN
+F 2 "SOT23-3" H 3000 1500 50  0000 C CNN
+F 3 "" H 3000 1300 50  0001 C CNN
+	1    3000 1300
+	0    1    1    0
+$EndComp
+Wire Wire Line
+	3000 1150 3000 900
+Connection ~ 3000 900
+Wire Wire Line
+	3000 1450 3000 1700
+Connection ~ 3000 1700
+$Comp
+L GPTS203211B S?
+U 1 1 5BB8AF7E
+P 2700 2050
+F 0 "S?" H 2550 2200 50  0000 C CNN
+F 1 "GPTS203211B" H 2700 1950 50  0000 C CNN
+F 2 "digikey-footprints:PushButton_12x12mm_THT_GPTS203211B" H 2900 2250 50  0001 L CNN
+F 3 "http://switches-connectors-custom.cwind.com/Asset/GPTS203211BR2.pdf" H 2900 2350 60  0001 L CNN
+F 4 "CW181-ND" H 2900 2450 60  0001 L CNN "Digi-Key_PN"
+F 5 "GPTS203211B" H 2900 2550 60  0001 L CNN "MPN"
+F 6 "Switches" H 2900 2650 60  0001 L CNN "Category"
+F 7 "Pushbutton Switches" H 2900 2750 60  0001 L CNN "Family"
+F 8 "http://switches-connectors-custom.cwind.com/Asset/GPTS203211BR2.pdf" H 2900 2850 60  0001 L CNN "DK_Datasheet_Link"
+F 9 "/product-detail/en/cw-industries/GPTS203211B/CW181-ND/3190590" H 2900 2950 60  0001 L CNN "DK_Detail_Page"
+F 10 "SWITCH PUSHBUTTON SPST 1A 30V" H 2900 3050 60  0001 L CNN "Description"
+F 11 "CW Industries" H 2900 3150 60  0001 L CNN "Manufacturer"
+F 12 "Active" H 2900 3250 60  0001 L CNN "Status"
+	1    2700 2050
+	0    -1   -1   0
+$EndComp
+Wire Wire Line
+	2700 2250 2700 3100
+$Comp
+L GND #PWR?
+U 1 1 5BB8B0A7
+P 2700 3100
+F 0 "#PWR?" H 2700 2850 50  0001 C CNN
+F 1 "GND" H 2700 2950 50  0000 C CNN
+F 2 "" H 2700 3100 50  0001 C CNN
+F 3 "" H 2700 3100 50  0001 C CNN
+	1    2700 3100
+	1    0    0    -1
+$EndComp
+Text Label 3050 1700 0    60   ~ 0
+UC_RST
+$Comp
+L C C?
+U 1 1 5BB8B458
+P 3750 2850
+F 0 "C?" H 3775 2950 50  0000 L CNN
+F 1 "C" H 3775 2750 50  0000 L CNN
+F 2 "" H 3788 2700 50  0001 C CNN
+F 3 "" H 3750 2850 50  0001 C CNN
+	1    3750 2850
+	1    0    0    -1
+$EndComp
+$Comp
+L C C?
+U 1 1 5BB8B606
+P 3100 2850
+F 0 "C?" H 3125 2950 50  0000 L CNN
+F 1 "C" H 3125 2750 50  0000 L CNN
+F 2 "" H 3138 2700 50  0001 C CNN
+F 3 "" H 3100 2850 50  0001 C CNN
+	1    3100 2850
+	1    0    0    -1
+$EndComp
+$Comp
+L Crystal Y?
+U 1 1 5BB8B63E
+P 3450 2600
+F 0 "Y?" H 3450 2750 50  0000 C CNN
+F 1 "Crystal" H 3450 2450 50  0000 C CNN
+F 2 "" H 3450 2600 50  0001 C CNN
+F 3 "" H 3450 2600 50  0001 C CNN
+	1    3450 2600
+	1    0    0    -1
+$EndComp
+$Comp
+L GND #PWR?
+U 1 1 5BB8B73D
+P 3100 3100
+F 0 "#PWR?" H 3100 2850 50  0001 C CNN
+F 1 "GND" H 3100 2950 50  0000 C CNN
+F 2 "" H 3100 3100 50  0001 C CNN
+F 3 "" H 3100 3100 50  0001 C CNN
+	1    3100 3100
+	1    0    0    -1
+$EndComp
+$Comp
+L GND #PWR?
+U 1 1 5BB8B77C
+P 3750 3100
+F 0 "#PWR?" H 3750 2850 50  0001 C CNN
+F 1 "GND" H 3750 2950 50  0000 C CNN
+F 2 "" H 3750 3100 50  0001 C CNN
+F 3 "" H 3750 3100 50  0001 C CNN
+	1    3750 3100
+	1    0    0    -1
+$EndComp
+Wire Wire Line
+	3100 3100 3100 3000
+Wire Wire Line
+	3100 2700 3100 2100
+Wire Wire Line
+	3100 2100 4150 2100
+Wire Wire Line
+	4150 2500 3750 2500
+Wire Wire Line
+	3750 2500 3750 2700
+Wire Wire Line
+	3750 3000 3750 3100
+Wire Wire Line
+	3300 2600 3100 2600
+Connection ~ 3100 2600
+Wire Wire Line
+	3600 2600 3750 2600
+Connection ~ 3750 2600
 $EndSCHEMATC

Commit message: feat: add i2c ic, add additional datasheets and simulations
Parts:
- removed S?: GPTS203211B, digikey-footprints:PushButton_12x12mm_THT_GPTS203211B, symbol GPTS203211B
- added C? (x4): 100n, symbol C
- added FB?: BLM18PG121SN1D, digikey-footprints:0603, symbol BLM18PG121SN1D
- added J?: CONN_02X03, symbol CONN_02X03
- added R? (x4): 330, symbol R
- added R?: 1M, symbol R
- added S?: KS-01Q-01, digikey-footprints:PushButton_Round_D12mm_THT_KS-01Q-01, symbol KS-01Q-01
- C? (x2): value C -> 27p
- Y?: value Crystal -> ABLS2-10.000MHZ-D4Y-T; footprint (none) -> F
Connections:
- net labels added: MISO, MOSI, SCK, SCL_3V3, SDA_3V3, WIFI_EN, WIFI_RST
- wire segments 26 -> 67

Commit message: feat: first draft of uc schematic created
Parts:
- added D?: APG1608SYKC/T, symbol LED
- added R?: 560, symbol R
- added R? (x2): 2K2, symbol R
Connections:
- net labels added: CS
- wire segments 67 -> 78
Changed lines of the file:
@@
 $Descr A4 11693 8268
 encoding utf-8
-Sheet 3 7
+Sheet 3 8
 Title ""
 Date ""
@@
 	1    0    0    -1
 $EndComp
-Wire Wire Line
-	6350 4500 6650 4500
-Wire Wire Line
-	6350 4400 6650 4400
-Wire Wire Line
-	2000 1700 4150 1700
-Wire Wire Line
-	2000 800  5150 800
-Wire Wire Line
-	5350 800  5350 1400
-Wire Wire Line
-	5150 800  5150 1400
-Wire Wire Line
-	5050 1400 5050 800
-Connection ~ 5050 800
-Wire Wire Line
-	4950 1400 4950 800
-Connection ~ 4950 800
-Wire Wire Line
-	4950 5400 4950 5500
-Wire Wire Line
-	4950 5500 5350 5500
-Wire Wire Line
-	5350 5500 5350 5400
-Wire Wire Line
-	5150 5400 5150 5550
-Connection ~ 5150 5500
-Wire Wire Line
-	5050 5400 5050 5500
-Connection ~ 5050 5500
-Wire Wire Line
-	2350 800  2350 1050
-Connection ~ 2350 800
-Wire Wire Line
-	2350 1350 2350 1900
-Connection ~ 2350 1700
-Wire Wire Line
-	3000 1050 3000 800
-Connection ~ 3000 800
-Wire Wire Line
-	3000 1350 3000 1700
-Connection ~ 3000 1700
-Wire Wire Line
-	2950 3500 2950 3400
-Wire Wire Line
-	2950 2100 2950 3100
-Wire Wire Line
-	2950 2100 4150 2100
-Wire Wire Line
-	3450 2500 4150 2500
-Wire Wire Line
-	3600 2500 3600 3100
-Wire Wire Line
-	3600 3400 3600 3500
-Wire Wire Line
-	3150 3000 2950 3000
-Connection ~ 2950 3000
-Wire Wire Line
-	3450 3000 3600 3000
-Connection ~ 3600 3000
-Wire Wire Line
-	4050 900  4050 800
-Connection ~ 4050 800
-Wire Wire Line
-	4050 1200 4050 1250
-Wire Wire Line
-	2250 2450 2250 2400
-Wire Wire Line
-	2250 2400 2450 2400
-Wire Wire Line
-	2450 2400 2450 2450
-Wire Wire Line
-	2250 2850 2250 2900
-Wire Wire Line
-	2250 2900 2450 2900
-Wire Wire Line
-	2450 2900 2450 2850
-Wire Wire Line
-	2350 2200 2350 2400
-Connection ~ 2350 2400
-Wire Wire Line
-	2350 2900 2350 3100
-Connection ~ 2350 2900
-Wire Wire Line
-	1550 4950 1700 4950
-Wire Wire Line
-	1700 4850 1600 4850
-Wire Wire Line
-	1600 4850 1600 4750
-Wire Wire Line
-	1600 4750 1550 4750
-Wire Wire Line
-	1250 4750 950  4750
-Wire Wire Line
-	1250 4950 950  4950
-Wire Wire Line
-	1700 5050 1600 5050
-Wire Wire Line
-	1600 5050 1600 5150
-Wire Wire Line
-	1600 5150 950  5150
-Wire Wire Line
-	2200 4950 2450 4950
-Wire Wire Line
-	2200 4850 2350 4850
-Wire Wire Line
-	2350 4850 2350 4750
-Wire Wire Line
-	2350 4750 2850 4750
-Wire Wire Line
-	2750 4950 2850 4950
-Wire Wire Line
-	2200 5050 2350 5050
-Wire Wire Line
-	2350 5050 2350 5150
-Wire Wire Line
-	4650 1250 4650 1200
-Wire Wire Line
-	4650 900  4650 800
-Connection ~ 4650 800
-Wire Wire Line
-	4350 1250 4350 1200
-Wire Wire Line
-	4350 900  4350 800
-Connection ~ 4350 800
 $Comp
 L C C?
@@
 	1    0    0    -1
 $EndComp
-Wire Wire Line
-	5600 1300 5600 1250
-Wire Wire Line
-	5600 950  5600 800
-Wire Wire Line
-	5350 800  5850 800
 $Comp
 L BLM18PG121SN1D FB?
@@
 	1    0    0    -1
 $EndComp
-Connection ~ 5600 800
-Wire Wire Line
-	6250 800  6700 800
 Text Label 6700 800  0    60   ~ 0
 VDD_3V3
-Wire Wire Line
-	6350 3100 6950 3100
-Wire Wire Line
-	6350 3200 6950 3200
-Wire Wire Line
-	6350 3300 6950 3300
 Text HLabel 6950 3100 2    60   Output ~ 0
 MOSI
 Text HLabel 6950 3200 2    60   Input ~ 0
 MISO
-Text HLabel 6950 3300 2    60   Output ~ 0
+Text HLabel 8750 3300 2    60   Output ~ 0
 SCK
 $Comp
@@
 	0    1    1    0
 $EndComp
+Text HLabel 6900 2600 2    60   Output ~ 0
+WIFI_EN
+Text HLabel 6900 2700 2    60   Output ~ 0
+WIFI_RST
+Text HLabel 7750 3500 2    60   Output ~ 0
+SCL_3V3
+Text HLabel 7750 3600 2    60   BiDi ~ 0
+SDA_3V3
+$Comp
+L LED D?
+U 1 1 5BBA7F65
+P 8400 4000
+F 0 "D?" H 8400 4100 50  0000 C CNN
+F 1 "APG1608SYKC/T" H 8400 3900 50  0000 C CNN
+F 2 "" H 8400 4000 50  0001 C CNN
+F 3 "" H 8400 4000 50  0001 C CNN
+	1    8400 4000
+	0    -1   -1   0
+$EndComp
+$Comp
+L R R?
+U 1 1 5BBA823A
+P 8400 3650
+F 0 "R?" V 8480 3650 50  0000 C CNN
+F 1 "560" V 8400 3650 50  0000 C CNN
+F 2 "" V 8330 3650 50  0001 C CNN
+F 3 "" H 8400 3650 50  0001 C CNN
+	1    8400 3650
+	-1   0    0    1
+$EndComp
+$Comp
+L GND #PWR?
+U 1 1 5BBA86F6
+P 8400 4300
+F 0 "#PWR?" H 8400 4050 50  0001 C CNN
+F 1 "GND" H 8400 4150 50  0000 C CNN
+F 2 "" H 8400 4300 50  0001 C CNN
+F 3 "" H 8400 4300 50  0001 C CNN
+	1    8400 4300
+	1    0    0    -1
+$EndComp
+Text HLabel 6950 3000 2    60   Output ~ 0
+CS
+Wire Wire Line
+	6350 4500 6650 4500
+Wire Wire Line
+	6350 4400 6650 4400
+Wire Wire Line
+	2000 1700 4150 1700
+Wire Wire Line
+	2000 800  5150 800
+Wire Wire Line
+	5350 800  5350 1400
+Wire Wire Line
+	5150 800  5150 1400
+Wire Wire Line
+	5050 1400 5050 800
+Connection ~ 5050 800
+Wire Wire Line
+	4950 1400 4950 800
+Connection ~ 4950 800
+Wire Wire Line
+	4950 5400 4950 5500
+Wire Wire Line
+	4950 5500 5350 5500
+Wire Wire Line
+	5350 5500 5350 5400
+Wire Wire Line
+	5150 5400 5150 5550
+Connection ~ 5150 5500
+Wire Wire Line
+	5050 5400 5050 5500
+Connection ~ 5050 5500
+Wire Wire Line
+	2350 800  2350 1050
+Connection ~ 2350 800
+Wire Wire Line
+	2350 1350 2350 1900
+Connection ~ 2350 1700
+Wire Wire Line
+	3000 1050 3000 800
+Connection ~ 3000 800
+Wire Wire Line
+	3000 1350 3000 1700
+Connection ~ 3000 1700
+Wire Wire Line
+	2950 3500 2950 3400
+Wire Wire Line
+	2950 2100 2950 3100
+Wire Wire Line
+	2950 2100 4150 2100
+Wire Wire Line
+	3450 2500 4150 2500
+Wire Wire Line
+	3600 2500 3600 3100
+Wire Wire Line
+	3600 3400 3600 3500
+Wire Wire Line
+	3150 3000 2950 3000
+Connection ~ 2950 3000
+Wire Wire Line
+	3450 3000 3600 3000
+Connection ~ 3600 3000
+Wire Wire Line
+	4050 900  4050 800
+Connection ~ 4050 800
+Wire Wire Line
+	4050 1200 4050 1250
+Wire Wire Line
+	2250 2450 2250 2400
+Wire Wire Line
+	2250 2400 2450 2400
+Wire Wire Line
+	2450 2400 2450 2450
+Wire Wire Line
+	2250 2850 2250 2900
+Wire Wire Line
+	2250 2900 2450 2900
+Wire Wire Line
+	2450 2900 2450 2850
+Wire Wire Line
+	2350 2200 2350 2400
+Connection ~ 2350 2400
+Wire Wire Line
+	2350 2900 2350 3100
+Connection ~ 2350 2900
+Wire Wire Line
+	1550 4950 1700 4950
+Wire Wire Line
+	1700 4850 1600 4850
+Wire Wire Line
+	1600 4850 1600 4750
+Wire Wire Line
+	1600 4750 1550 4750
+Wire Wire Line
+	1250 4750 950  4750
+Wire Wire Line
+	1250 4950 950  4950
+Wire Wire Line
+	1700 5050 1600 5050
+Wire Wire Line
+	1600 5050 1600 5150
+Wire Wire Line
+	1600 5150 950  5150
+Wire Wire Line
+	2200 4950 2450 4950
+Wire Wire Line
+	2200 4850 2350 4850
+Wire Wire Line
+	2350 4850 2350 4750
+Wire Wire Line
+	2350 4750 2850 4750
+Wire Wire Line
+	2750 4950 2850 4950
+Wire Wire Line
+	2200 5050 2350 5050
+Wire Wire Line
+	2350 5050 2350 5150
+Wire Wire Line
+	4650 1250 4650 1200
+Wire Wire Line
+	4650 900  4650 800
+Connection ~ 4650 800
+Wire Wire Line
+	4350 1250 4350 1200
+Wire Wire Line
+	4350 900  4350 800
+Connection ~ 4350 800
+Wire Wire Line
+	5600 1300 5600 1250
+Wire Wire Line
+	5600 950  5600 800
+Wire Wire Line
+	5350 800  5850 800
+Connection ~ 5600 800
+Wire Wire Line
+	6250 800  6700 800
+Wire Wire Line
+	6350 3100 6950 3100
+Wire Wire Line
+	6350 3200 6950 3200
+Wire Wire Line
+	6350 3300 8750 3300
 Connection ~ 3600 2500
 Wire Wire Line
@@
 Wire Wire Line
 	6350 2600 6900 2600
-Text HLabel 6900 2600 2    60   Output ~ 0
-WIFI_EN
 Wire Wire Line
 	6350 2700 6900 2700
-Text HLabel 6900 2700 2    60   Output ~ 0
-WIFI_RST
-Wire Wire Line
-	6350 3500 6950 3500
-Wire Wire Line
-	6350 3600 6950 3600
-Text HLabel 6950 3500 2    60   Output ~ 0
-SCL_3V3
-Text HLabel 6950 3600 2    60   BiDi ~ 0
-SDA_3V3
+Wire Wire Line
+	6350 3500 7750 3500
+Wire Wire Line
+	6350 3600 7750 3600
+Connection ~ 8400 3300
+Wire Wire Line
+	8400 3800 8400 3850
+Wire Wire Line
+	8400 4150 8400 4300
+Wire Wire Line
+	6350 3000 6950 3000
+Wire Wire Line
+	8400 3300 8400 3500
+$Comp
+L R R?
+U 1 1 5BBB9240
+P 7450 2950
+F 0 "R?" V 7530 2950 50  0000 C CNN
+F 1 "2K2" V 7450 2950 50  0000 C CNN
+F 2 "" V 7380 2950 50  0001 C CNN
+F 3 "" H 7450 2950 50  0001 C CNN
+	1    7450 2950
+	-1   0    0    1
+$EndComp
+$Comp
+L R R?
+U 1 1 5BBB92F1
+P 7650 2950
+F 0 "R?" V 7730 2950 50  0000 C CNN
+F 1 "2K2" V 7650 2950 50  0000 C CNN
+F 2 "" V 7580 2950 50  0001 C CNN
+F 3 "" H 7650 2950 50  0001 C CNN
+	1    7650 2950
+	-1   0    0    1
+$EndComp
+Wire Wire Line
+	7450 3100 7450 3500
+Connection ~ 7450 3500
+Wire Wire Line
+	7650 3100 7650 3600
+Connection ~ 7650 3600
+Wire Wire Line
+	7450 2800 7450 2550
+Wire Wire Line
+	7450 2550 7650 2550
+Wire Wire Line
+	7650 2550 7650 2800
+Wire Wire Line
+	7550 2550 7550 2400
+Wire Wire Line
+	7550 2400 7600 2400
+Connection ~ 7550 2550
+Text Label 7600 2400 0    60   ~ 0
+VDD_3V3
 $EndSCHEMATC

Commit message: feat: add keypad schematic
Parts:
- added C?: 100n, symbol C
Connections:
- net labels added: CAM_CLK, CAM_D0, CAM_D1, CAM_D2, CAM_D3, CAM_D4, CAM_D5, CAM_D6, CAM_D7, CAM_HSYNC, CAM_PCLK, CAM_VSYNC, CAM_XCLK_CTL
- wire segments 78 -> 118
Other:
- moved on the sheet: S?

Commit message: feat: 3.3 regulator housing changed due to temperature
Parts:
- C? (x7): symbol C -> Device:C
- D?: symbol D_Zener -> Device:D_Zener
- D?: symbol LED -> Device:LED
- FB?: symbol BLM18PG121SN1D -> CameraSystem-rescue:BLM18PG121SN1D
- J?: symbol CONN_02X03 -> CameraSystem-rescue:CONN_02X03
- R? (x9): symbol R -> Device:R
- S?: symbol KS-01Q-01 -> CameraSystem-rescue:KS-01Q-01
- U?: symbol ATMEGA16A-AU -> CameraSystem-rescue:ATMEGA16A-AU
- Y?: symbol Crystal -> Device:Crystal
Connections:
- net labels added: QT_CHN, QT_RST
- wire segments 118 -> 120

Commit message: feat: add debugging pins
Parts:
- removed J?: CONN_02X03, symbol CameraSystem-rescue:CONN_02X03
- added C?: 100n, symbol Device:C
- added J? (x2): Conn_01x02, symbol Connector_Generic:Conn_01x02
- added J?: Conn_01x03, symbol Connector_Generic:Conn_01x03
- added J?: Conn_02x03_Odd_Even, symbol Connector_Generic:Conn_02x03_Odd_Even
- added R? (x7): 10k, symbol Device:R
Connections:
- wire segments 120 -> 150
Other:
- note added: "For debugging purposes"
- note added: "NA"

Commit message: feat: DRC run
Parts:
- C10, C11, C12, C13, C14, C15, C16, C17: renamed from C?; footprint (none) -> Capacitor_SMD:C_0603_1608Metric_Pad1.05x0.95mm_HandSolder
- R10, R11, R12, R13, R14, R15, R16, R17, R18, R19, R20, R21, R6, R7, R8, R9: renamed from R?; footprint (none) -> Resistor_SMD:R_0603_1608Metric_Pad1.05x0.95mm_HandSolder
- gave numbers to parts that had none: 10

Commit message: feat: add new motor module to the schematic
Parts:
- removed R13, R14, R15, R17, R18: 10k, Resistor_SMD:R_0603_1608Metric_Pad1.05x0.95mm_HandSolder, symbol Device:R
Connections:
- net labels added: M_DIR, M_EN, M_PWM, SENSOR1, SENSOR2
- wire segments 150 -> 140
Changed lines of the file:
@@
 $Descr A4 11693 8268
 encoding utf-8
-Sheet 3 8
+Sheet 3 9
 Title ""
 Date ""
@@
 Text Notes 9400 3600 0    50   ~ 0
 For debugging purposes
-Wire Wire Line
-	6350 5100 6650 5100
-Wire Wire Line
-	6650 5100 6650 5200
-$Comp
-L Device:R R15
-U 1 1 5BC21924
-P 6650 5350
-F 0 "R15" V 6730 5350 50  0000 C CNN
-F 1 "10k" V 6650 5350 50  0000 C CNN
-F 2 "Resistor_SMD:R_0603_1608Metric_Pad1.05x0.95mm_HandSolder" V 6580 5350 50  0001 C CNN
-F 3 "" H 6650 5350 50  0001 C CNN
-	1    6650 5350
-	-1   0    0    1
-$EndComp
-$Comp
-L power:GND #PWR05
-U 1 1 5BC21A51
-P 6650 5550
-F 0 "#PWR05" H 6650 5300 50  0001 C CNN
-F 1 "GND" H 6650 5400 50  0000 C CNN
-F 2 "" H 6650 5550 50  0001 C CNN
-F 3 "" H 6650 5550 50  0001 C CNN
-	1    6650 5550
-	1    0    0    -1
-$EndComp
-Wire Wire Line
-	6650 5500 6650 5550
 Text Notes 6700 5350 0    50   ~ 0
 NA
@@
 	1    1900 4950
 	1    0    0    -1
-$EndComp
-$Comp
-L Device:R R14
-U 1 1 5BC2A60A
-P 6600 4200
-F 0 "R14" V 6680 4200 50  0000 C CNN
-F 1 "10k" V 6600 4200 50  0000 C CNN
-F 2 "Resistor_SMD:R_0603_1608Metric_Pad1.05x0.95mm_HandSolder" V 6530 4200 50  0001 C CNN
-F 3 "" H 6600 4200 50  0001 C CNN
-	1    6600 4200
-	0    1    1    0
-$EndComp
-$Comp
-L Device:R R18
-U 1 1 5BC2A764
-P 6900 4100
-F 0 "R18" V 6980 4100 50  0000 C CNN
-F 1 "10k" V 6900 4100 50  0000 C CNN
-F 2 "Resistor_SMD:R_0603_1608Metric_Pad1.05x0.95mm_HandSolder" V 6830 4100 50  0001 C CNN
-F 3 "" H 6900 4100 50  0001 C CNN
-	1    6900 4100
-	0    1    1    0
-$EndComp
-$Comp
-L Device:R R13
-U 1 1 5BC2A815
-P 6600 4000
-F 0 "R13" V 6680 4000 50  0000 C CNN
-F 1 "10k" V 6600 4000 50  0000 C CNN
-F 2 "Resistor_SMD:R_0603_1608Metric_Pad1.05x0.95mm_HandSolder" V 6530 4000 50  0001 C CNN
-F 3 "" H 6600 4000 50  0001 C CNN
-	1    6600 4000
-	0    1    1    0
-$EndComp
-$Comp
-L Device:R R17
-U 1 1 5BC2A86F
-P 6900 3900
-F 0 "R17" V 6980 3900 50  0000 C CNN
-F 1 "10k" V 6900 3900 50  0000 C CNN
-F 2 "Resistor_SMD:R_0603_1608Metric_Pad1.05x0.95mm_HandSolder" V 6830 3900 50  0001 C CNN
-F 3 "" H 6900 3900 50  0001 C CNN
-	1    6900 3900
-	0    1    1    0
 $EndComp
 $Comp
@@
 	0    1    1    0
 $EndComp
-Text Notes 7250 4300 0    50   ~ 0
-NA
 Text Notes 6350 3000 0    50   ~ 0
 NA
 Wire Wire Line
-	6350 3900 6750 3900
-Wire Wire Line
-	7600 3900 7600 4000
-Wire Wire Line
-	7050 3900 7600 3900
-Wire Wire Line
-	6350 4200 6450 4200
-Connection ~ 7600 4200
-Wire Wire Line
-	7600 4200 7600 4250
-Wire Wire Line
-	6750 4200 7600 4200
-Wire Wire Line
-	6450 4000 6350 4000
-Wire Wire Line
-	6350 4100 6750 4100
-Wire Wire Line
-	7050 4100 7600 4100
-Connection ~ 7600 4100
-Wire Wire Line
-	7600 4100 7600 4200
-Wire Wire Line
-	6750 4000 7600 4000
-Connection ~ 7600 4000
-Wire Wire Line
-	7600 4000 7600 4100
-Wire Wire Line
 	6350 2900 6450 2900
 Wire Wire Line
@@
 Wire Wire Line
 	6750 2900 7250 2900
-$Comp
-L power:GND #PWR07
-U 1 1 5BC56C7A
-P 7600 4250
-F 0 "#PWR07" H 7600 4000 50  0001 C CNN
-F 1 "GND" H 7600 4100 50  0000 C CNN
-F 2 "" H 7600 4250 50  0001 C CNN
-F 3 "" H 7600 4250 50  0001 C CNN
-	1    7600 4250
-	1    0    0    -1
-$EndComp
 $Comp
 L power:GND #PWR06
@@
 Connection ~ 7250 2900
 Wire Notes Line
-	6400 4300 6400 3850
-Wire Notes Line
-	6400 3850 7150 3850
-Wire Notes Line
-	7150 3850 7150 4300
-Wire Notes Line
-	7150 4300 6400 4300
-Wire Notes Line
 	6450 2750 6450 2950
 Wire Notes Line
@@
 Wire Wire Line
 	3950 3300 3950 3500
+Text HLabel 6650 5100 2    60   Output ~ 0
+M_PWM
+Wire Wire Line
+	6350 5100 6650 5100
+Text HLabel 6950 3900 2    60   Output ~ 0
+M_DIR
+Wire Wire Line
+	6350 3900 6950 3900
+Wire Wire Line
+	6350 4000 6950 4000
+Text HLabel 6950 4000 2    60   Output ~ 0
+M_EN
+Text HLabel 6950 4100 2    60   Input ~ 0
+SENSOR1
+Text HLabel 6950 4200 2    60   Input ~ 0
+SENSOR2
+Wire Wire Line
+	6350 4200 6950 4200
+Wire Wire Line
+	6350 4100 6950 4100
 $EndSCHEMATC
