File: Projects/CameraSystem/Schematics/Microcontroller.sch (KiCad schematic (older format))
At the start: 24 parts, among them J2 Conn_02x03_Odd_Even, J3 Conn_01x02, J4 Conn_01x03, J5 Conn_01x02, SW1 SW_Push, U3 ATMEGA16A-AU, Y2 ABLS2-10.000MHZ-D4Y-T

Commit message: camera layout updated
Parts:
- removed J4: Conn_01x03, Connector_PinSocket_2.54mm:PinSocket_1x03_P2.54mm_Vertical, symbol Connector_Generic:Conn_01x03
Connections:
- net labels removed: SPI_RX, SPI_TX
- wire segments 124 -> 121
Changed lines of the file:
@@
 SDA_3V3
-$Comp
-L Connector_Generic:Conn_01x03 J4
-U 1 1 5BBF43CB
-P 10050 4300
-F 0 "J4" H 10130 4342 50  0000 L CNN
-F 1 "Conn_01x03" H 10130 4251 50  0000 L CNN
-F 2 "Connector_PinSocket_2.54mm:PinSocket_1x03_P2.54mm_Vertical" H 10050 4300 50  0001 C CNN
-F 3 "~" H 10050 4300 50  0001 C CNN
-	1    10050 4300
-	1    0    0    -1
-$EndComp
-Wire Wire Line
-	9400 4200 9850 4200
-Wire Wire Line
-	9400 4300 9850 4300
-Wire Wire Line
-	9850 4400 9400 4400
-Text Label 9400 4200 0    50   ~ 0
-MOSI
-Text Label 9400 4300 0    50   ~ 0
-MISO
-Text Label 9400 4400 0    50   ~ 0
-SCK
 $Comp
 L Connector_Generic:Conn_01x02 J5
@@
 	9850 4800 9400 4800
 Text Label 9400 4700 0    50   ~ 0
-SPI_RX
+UC_SPI_RX
 Text Label 9400 4800 0    50   ~ 0
-SPI_TX
+UC_SPI_TX
 Text Notes 9400 3600 0    50   ~ 0
 For debugging purposes
