File: Projects/CameraSystem/Schematics/WIFI.sch (KiCad schematic (older format))
At the start: 0 parts

Commit message: feat: add i2c ic, add additional datasheets and simulations
Parts:
- added C?: 100n, symbol C
- added Q?: BC846B_215, digikey-footprints:SOT-23-3, symbol BC846B_215
- added R?: 4K7, symbol R
- added R? (x2): 10k, symbol R
- added U?: ESP8266, symbol ESP8266
Connections:
- net labels added: GND, VDD_3V3, WIFI_EN, WIFI_RST, WIFI_RX, WIFI_TX
- wire segments 0 -> 18
Changed lines of the file:
@@
 $Descr A4 11693 8268
 encoding utf-8
-Sheet 3 6
+Sheet 4 7
 Title ""
 Date ""
@@
 Comment4 ""
 $EndDescr
+Text HLabel 5700 3500 0    60   Input ~ 0
+VDD_3V3
+Text HLabel 5700 3200 0    60   Output ~ 0
+WIFI_TX
+Text HLabel 7200 3500 2    60   Input ~ 0
+WIFI_RX
+Text HLabel 4050 3700 0    60   Input ~ 0
+WIFI_RST
+Text HLabel 5700 3300 0    60   Input ~ 0
+WIFI_EN
+$Comp
+L ESP8266 U?
+U 1 1 5BB97A97
+P 6500 3350
+F 0 "U?" H 6500 3050 60  0000 C CNN
+F 1 "ESP8266" H 6500 3650 60  0000 C CNN
+F 2 "" H 6500 3350 60  0001 C CNN
+F 3 "" H 6500 3350 60  0001 C CNN
+	1    6500 3350
+	1    0    0    -1
+$EndComp
+$Comp
+L C C?
+U 1 1 5BB97B07
+P 5850 3800
+F 0 "C?" H 5875 3900 50  0000 L CNN
+F 1 "100n" H 5875 3700 50  0000 L CNN
+F 2 "" H 5888 3650 50  0001 C CNN
+F 3 "" H 5850 3800 50  0001 C CNN
+	1    5850 3800
+	1    0    0    -1
+$EndComp
+$Comp
+L GND #PWR?
+U 1 1 5BB97B4E
+P 5850 4350
+F 0 "#PWR?" H 5850 4100 50  0001 C CNN
+F 1 "GND" H 5850 4200 50  0000 C CNN
+F 2 "" H 5850 4350 50  0001 C CNN
+F 3 "" H 5850 4350 50  0001 C CNN
+	1    5850 4350
+	1    0    0    -1
+$EndComp
+Wire Wire Line
+	5700 3500 6000 3500
+Wire Wire Line
+	5850 3650 5850 3500
+Connection ~ 5850 3500
+Wire Wire Line
+	5850 4350 5850 3950
+$Comp
+L GND #PWR?
+U 1 1 5BB97B87
+P 7750 3300
+F 0 "#PWR?" H 7750 3050 50  0001 C CNN
+F 1 "GND" H 7750 3150 50  0000 C CNN
+F 2 "" H 7750 3300 50  0001 C CNN
+F 3 "" H 7750 3300 50  0001 C CNN
+	1    7750 3300
+	1    0    0    -1
+$EndComp
+Wire Wire Line
+	7000 3200 7750 3200
+Wire Wire Line
+	7750 3200 7750 3300
+Wire Wire Line
+	7000 3500 7200 3500
+Wire Wire Line
+	6000 3200 5700 3200
+Wire Wire Line
+	6000 3300 5700 3300
+$Comp
+L R R?
+U 1 1 5BB97CCF
+P 4300 3700
+F 0 "R?" V 4380 3700 50  0000 C CNN
+F 1 "4K7" V 4300 3700 50  0000 C CNN
+F 2 "" V 4230 3700 50  0001 C CNN
+F 3 "" H 4300 3700 50  0001 C CNN
+	1    4300 3700
+	0    1    1    0
+$EndComp
+Wire Wire Line
+	4050 3700 4150 3700
+$Comp
+L R R?
+U 1 1 5BB97D2C
+P 4600 4000
+F 0 "R?" V 4680 4000 50  0000 C CNN
+F 1 "10k" V 4600 4000 50  0000 C CNN
+F 2 "" V 4530 4000 50  0001 C CNN
+F 3 "" H 4600 4000 50  0001 C CNN
+	1    4600 4000
+	-1   0    0    1
+$EndComp
+Wire Wire Line
+	6000 3400 5000 3400
+Wire Wire Line
+	5000 3250 5000 3500
+$Comp
+L R R?
+U 1 1 5BB97D8F
+P 5000 3100
+F 0 "R?" V 5080 3100 50  0000 C CNN
+F 1 "10k" V 5000 3100 50  0000 C CNN
+F 2 "" V 4930 3100 50  0001 C CNN
+F 3 "" H 5000 3100 50  0001 C CNN
+	1    5000 3100
+	-1   0    0    1
+$EndComp
+Wire Wire Line
+	5000 2950 5000 2750
+Wire Wire Line
+	5000 2750 5100 2750
+Text Label 5100 2750 0    60   ~ 0
+VDD_3V3
+Connection ~ 5000 3400
+Wire Wire Line
+	4450 3700 4700 3700
+Wire Wire Line
+	4600 3700 4600 3850
+Wire Wire Line
+	4600 4150 4600 4250
+Wire Wire Line
+	4600 4250 5000 4250
+Wire Wire Line
+	5000 3900 5000 4350
+$Comp
+L GND #PWR?
+U 1 1 5BB97FB0
+P 5000 4350
+F 0 "#PWR?" H 5000 4100 50  0001 C CNN
+F 1 "GND" H 5000 4200 50  0000 C CNN
+F 2 "" H 5000 4350 50  0001 C CNN
+F 3 "" H 5000 4350 50  0001 C CNN
+	1    5000 4350
+	1    0    0    -1
+$EndComp
+Connection ~ 5000 4250
+Connection ~ 4600 3700
+$Comp
+L BC846B_215 Q?
+U 1 1 5BB98225
+P 4900 3700
+F 0 "Q?" H 4774 3866 60  0000 L CNN
+F 1 "BC846B_215" V 5106 3700 60  0000 C CNN
+F 2 "digikey-footprints:SOT-23-3" H 5100 3900 60  0001 L CNN
+F 3 "https://assets.nexperia.com/documents/data-sheet/BC846_SER.pdf" H 5100 4000 60  0001 L CNN
+F 4 "1727-2920-1-ND" H 5100 4100 60  0001 L CNN "Digi-Key_PN"
+F 5 "BC846B,215" H 5100 4200 60  0001 L CNN "MPN"
+F 6 "Discrete Semiconductor Products" H 5100 4300 60  0001 L CNN "Category"
+F 7 "Transistors - Bipolar (BJT) - Single" H 5100 4400 60  0001 L CNN "Family"
+F 8 "https://assets.nexperia.com/documents/data-sheet/BC846_SER.pdf" H 5100 4500 60  0001 L CNN "DK_Datasheet_Link"
+F 9 "/product-detail/en/nexperia-usa-inc/BC846B,215/1727-2920-1-ND/763459" H 5100 4600 60  0001 L CNN "DK_Detail_Page"
+F 10 "TRANS NPN 65V 0.1A SOT23" H 5100 4700 60  0001 L CNN "Description"
+F 11 "Nexperia USA Inc." H 5100 4800 60  0001 L CNN "Manufacturer"
+F 12 "Active" H 5100 4900 60  0001 L CNN "Status"
+	1    4900 3700
+	1    0    0    -1
+$EndComp
 $EndSCHEMATC

Commit message: feat: first draft of uc schematic created
Parts:
- added J?: CONN_02X02, symbol CONN_02X02
Connections:
- net labels added: VDD_3V3_IN
- wire segments 18 -> 26
Changed lines of the file:
@@
 $Descr A4 11693 8268
 encoding utf-8
-Sheet 4 7
+Sheet 4 8
 Title ""
 Date ""
@@
 Comment4 ""
 $EndDescr
-Text HLabel 5700 3500 0    60   Input ~ 0
-VDD_3V3
 Text HLabel 5700 3200 0    60   Output ~ 0
 WIFI_TX
@@
 $EndComp
 Wire Wire Line
-	5700 3500 6000 3500
+	5350 3500 6000 3500
 Wire Wire Line
 	5850 3650 5850 3500
@@
 	5000 2750 5100 2750
 Text Label 5100 2750 0    60   ~ 0
-VDD_3V3
+VDD_3V3_IN
 Connection ~ 5000 3400
 Wire Wire Line
@@
 	1    0    0    -1
 $EndComp
+Text HLabel 3400 2150 0    60   Input ~ 0
+VDD_3V3
+Wire Wire Line
+	3400 2150 3650 2150
+Wire Wire Line
+	4250 2150 4600 2150
+Text Label 4600 2150 0    60   ~ 0
+VDD_3V3_IN
+Text Label 5350 3500 0    60   ~ 0
+VDD_3V3_IN
+$Comp
+L CONN_02X02 J?
+U 1 1 5BBA9829
+P 3950 2150
+F 0 "J?" H 3950 2300 50  0000 C CNN
+F 1 "CONN_02X02" H 3950 2000 50  0000 C CNN
+F 2 "" H 3950 950 50  0001 C CNN
+F 3 "" H 3950 950 50  0001 C CNN
+	1    3950 2150
+	1    0    0    -1
+$EndComp
+Wire Wire Line
+	3700 2100 3650 2100
+Wire Wire Line
+	3650 2100 3650 2200
+Wire Wire Line
+	3650 2200 3700 2200
+Connection ~ 3650 2150
+Wire Wire Line
+	4250 2200 4200 2200
+Wire Wire Line
+	4250 2100 4250 2200
+Wire Wire Line
+	4200 2100 4250 2100
+Connection ~ 4250 2150
 $EndSCHEMATC

Commit message: feat: 3.3 regulator housing changed due to temperature
Parts:
- C?: symbol C -> Device:C
- J?: symbol CONN_02X02 -> CameraSystem-rescue:CONN_02X02
- Q?: symbol BC846B_215 -> CameraSystem-rescue:BC846B_215
- R? (x3): symbol R -> Device:R
- U?: symbol ESP8266 -> cl-integrated_circuits:ESP8266
Connections:
- wire segments 26 -> 32
Changed lines of the file:
@@
-EESchema Schematic File Version 2
-LIBS:cl-connectors
-LIBS:dk_Addressable-Specialty
-LIBS:dk_Alarms-Buzzers-and-Sirens
-LIBS:dk_Automotive-Relays
-LIBS:dk_Balun
-LIBS:dk_Barrel-Audio-Connectors
-LIBS:dk_Battery-Holders-Clips-Contacts
-LIBS:dk_Clock-Timing-Clock-Generators-PLLs-Frequency-Synthesizers
-LIBS:dk_Clock-Timing-Programmable-Timers-and-Oscillators
-LIBS:dk_Clock-Timing-Real-Time-Clocks
-LIBS:dk_Coaxial-Connectors-RF
-LIBS:dk_Current-Transducers
-LIBS:dk_Data-Acquisition-ADCs-DACs-Special-Purpose
-LIBS:dk_Data-Acquisition-Analog-to-Digital-Converters-ADC
-LIBS:dk_Data-Acquisition-Digital-Potentiometers
-LIBS:dk_Data-Acquisition-Digital-to-Analog-Converters-DAC
-LIBS:dk_Data-Acquisition-Touch-Screen-Controllers
-LIBS:dk_DC-DC-Converters
-LIBS:dk_Digital-Isolators
-LIBS:dk_Diodes-Bridge-Rectifiers
-LIBS:dk_Diodes-Rectifiers-Arrays
-LIBS:dk_Diodes-Rectifiers-Single
-LIBS:dk_Diodes-Zener-Single
-LIBS:dk_Display-Modules-LCD-OLED-Graphic
-LIBS:dk_Display-Modules-LED-Character-and-Numeric
-LIBS:dk_D-Sub-Connectors
-LIBS:dk_Embedded-Microcontrollers
-LIBS:dk_Encoders
-LIBS:dk_Evaluation-Boards-Sensors
-LIBS:dk_Ferrite-Beads-and-Chips
-LIBS:dk_Fixed-Inductors
-LIBS:dk_Fuses
-LIBS:dk_Gas-Sensors
-LIBS:dk_Humidity-Moisture-Sensors
-LIBS:dk_Image-Sensors-Camera
-LIBS:dk_Infrared-UV-Visible-Emitters
-LIBS:dk_Inrush-Current-Limiters-ICL
-LIBS:dk_Interface-Analog-Switches-Multiplexers-Demultiplexers
-LIBS:dk_Interface-Analog-Switches-Special-Purpose
-LIBS:dk_Interface-Controllers
-LIBS:dk_Interface-Drivers-Receivers-Transceivers
-LIBS:dk_Interface-I-O-Expanders
-LIBS:dk_Interface-Modules
-LIBS:dk_Interface-Sensor-and-Detector-Interfaces
-LIBS:dk_Interface-Sensor-Capacitive-Touch
-LIBS:dk_Interface-Specialized
-LIBS:dk_LED-Indication-Discrete
-LIBS:dk_LEDs-Circuit-Board-Indicators-Arrays-Light-Bars-Bar-Graphs
-LIBS:dk_Linear-Amplifiers-Audio
-LIBS:dk_Linear-Amplifiers-Instrumentation-OP-Amps-Buffer-Amps
-LIBS:dk_Linear-Comparators
-LIBS:dk_Logic-Buffers-Drivers-Receivers-Transceivers
-LIBS:dk_Logic-Flip-Flops
-LIBS:dk_Logic-Gates-and-Inverters
-LIBS:dk_Logic-Multivibrators
-LIBS:dk_Logic-Shift-Registers
-LIBS:dk_Logic-Signal-Switches-Multiplexers-Decoders
-LIBS:dk_Logic-Translators-Level-Shifters
-LIBS:dk_Magnetic-Sensors-Compass-Magnetic-Field-Modules
-LIBS:dk_Magnetic-Sensors-Linear-Compass-ICs
-LIBS:dk_Magnetic-Sensors-Switches-Solid-State
-LIBS:dk_Memory
-LIBS:dk_Memory-Connectors-PC-Card-Sockets
-LIBS:dk_Microphones
-LIBS:dk_Modular-Connectors-Jacks
-LIBS:dk_Modular-Connectors-Jacks-With-Magnetics
-LIBS:dk_Motion-Sensors-Accelerometers
-LIBS:dk_Motion-Sensors-IMUs-Inertial-Measurement-Units
-LIBS:dk_Motion-Sensors-Tilt-Switches
-LIBS:dk_Navigation-Switches-Joystick
-LIBS:dk_Optical-Sensors-Ambient-Light-IR-UV-Sensors
-LIBS:dk_Optical-Sensors-Photo-Detectors-Remote-Receiver
-LIBS:dk_Optical-Sensors-Photodiodes
-LIBS:dk_Optical-Sensors-Phototransistors
-LIBS:dk_Optical-Sensors-Reflective-Analog-Output
-LIBS:dk_Optoisolators-Logic-Output
-LIBS:dk_Optoisolators-Transistor-Photovoltaic-Output
-LIBS:dk_Optoisolators-Triac-SCR-Output
-LIBS:dk_Oscillators
-LIBS:dk_PMIC-AC-DC-Converters-Offline-Switchers
-LIBS:dk_PMIC-Battery-Chargers
-LIBS:dk_PMIC-Battery-Management
-LIBS:dk_PMIC-Current-Regulation-Management
-LIBS:dk_PMIC-Full-Half-Bridge-Drivers
-LIBS:dk_PMIC-Gate-Drivers
-LIBS:dk_PMIC-LED-Drivers
-LIBS:dk_PMIC-Motor-Drivers-Controllers
-LIBS:dk_PMIC-OR-Controllers-Ideal-Diodes
-LIBS:dk_PMIC-Power-Distribution-Switches-Load-Drivers
-LIBS:dk_PMIC-Power-Management-Specialized
-LIBS:dk_PMIC-RMS-to-DC-Converters
-LIBS:dk_PMIC-Supervisors
-LIBS:dk_PMIC-Thermal-Management
-LIBS:dk_PMIC-V-F-and-F-V-Converters
-LIBS:dk_PMIC-Voltage-Reference
-LIBS:dk_PMIC-Voltage-Regulators-DC-DC-Switching-Controllers
-LIBS:dk_PMIC-Voltage-Regulators-DC-DC-Switching-Regulators
-LIBS:dk_PMIC-Voltage-Regulators-Linear
-LIBS:dk_PMIC-Voltage-Regulators-Special-Purpose
-LIBS:dk_Power-Relays-Over-2-Amps
-LIBS:dk_Pressure-Sensors-Transducers
-LIBS:dk_Programmable-Oscillators
-LIBS:dk_Pushbutton-Switches
-LIBS:dk_Rectangular-Connectors-Headers-Male-Pins
-LIBS:dk_Reed-Relays
-LIBS:dk_Resistor-Networks-Arrays
-LIBS:dk_RF-Amplifiers
-LIBS:dk_RF-Antennas
-LIBS:dk_RF-Demodulators
-LIBS:dk_RF-Detectors
-LIBS:dk_RF-Evaluation-and-Development-Kits-Boards
-LIBS:dk_RFID-RF-Access-Monitoring-ICs
-LIBS:dk_RF-Receivers
-LIBS:dk_RF-Switches
-LIBS:dk_RF-Transceiver-ICs
-LIBS:dk_RF-Transceiver-Modules
-LIBS:dk_RF-Transmitters
-LIBS:dk_Rotary-Potentiometers-Rheostats
-LIBS:dk_Sensors-Transducers_Accessories
-LIBS:dk_Signal-Relays-Up-to-2-Amps
-LIBS:dk_Slide-Switches
-LIBS:dk_Solid-State-Relays
-LIBS:dk_Specialized-ICs
-LIBS:dk_Specialized-Sensors
-LIBS:dk_Surge-Suppression-ICs
-LIBS:dk_Tactile-Switches
-LIBS:dk_Temperature-Sensors-Analog-and-Digital-Output
-LIBS:dk_Thermal-Cutoffs-Thermal-Fuses
-LIBS:dk_Thyristors-DIACs-SIDACs
-LIBS:dk_Thyristors-SCRs
-LIBS:dk_Thyristors-TRIACs
-LIBS:dk_Toggle-Switches
-LIBS:dk_Transistors-Bipolar-BJT-Arrays
-LIBS:dk_Transistors-Bipolar-BJT-RF
-LIBS:dk_Transistors-Bipolar-BJT-Single
-LIBS:dk_Transistors-Bipolar-BJT-Single-Pre-Biased
-LIBS:dk_Transistors-FETs-MOSFETs-Arrays
-LIBS:dk_Transistors-FETs-MOSFETs-RF
-LIBS:dk_Transistors-FETs-MOSFETs-Single
-LIBS:dk_Transistors-JFETs
-LIBS:dk_Trimmer-Potentiometers
-LIBS:dk_TVS-Diodes
-LIBS:dk_TVS-Mixed-Technology
-LIBS:dk_USB-DVI-HDMI-Connectors
-LIBS:power
-LIBS:device
-LIBS:transistors
-LIBS:conn
-LIBS:linear
-LIBS:regul
-LIBS:74xx
-LIBS:cmos4000
-LIBS:adc-dac
-LIBS:memory
-LIBS:xilinx
-LIBS:microcontrollers
-LIBS:dsp
-LIBS:microchip
-LIBS:analog_switches
-LIBS:motorola
-LIBS:texas
-LIBS:intel
-LIBS:audio
-LIBS:interface
-LIBS:digital-audio
-LIBS:philips
-LIBS:display
-LIBS:cypress
-LIBS:siliconi
-LIBS:opto
-LIBS:atmel
-LIBS:contrib
-LIBS:valves
-LIBS:cl-integrated_circuits
-LIBS:cl-misc
+EESchema Schematic File Version 4
 LIBS:CameraSystem-cache
-EELAYER 25 0
+EELAYER 26 0
 EELAYER END
 $Descr A4 11693 8268
@@
 WIFI_EN
 $Comp
-L ESP8266 U?
+L cl-integrated_circuits:ESP8266 U?
 U 1 1 5BB97A97
 P 6500 3350
@@
 $EndComp
 $Comp
-L C C?
+L Device:C C?
 U 1 1 5BB97B07
 P 5850 3800
@@
 $EndComp
 $Comp
-L GND #PWR?
+L power:GND #PWR?
 U 1 1 5BB97B4E
 P 5850 4350
@@
 $EndComp
 Wire Wire Line
-	5350 3500 6000 3500
+	5350 3500 5850 3500
 Wire Wire Line
 	5850 3650 5850 3500
@@
 	5850 4350 5850 3950
 $Comp
-L GND #PWR?
+L power:GND #PWR?
 U 1 1 5BB97B87
 P 7750 3300
@@
 	6000 3300 5700 3300
 $Comp
-L R R?
+L Device:R R?
 U 1 1 5BB97CCF
 P 4300 3700
@@
 	4050 3700 4150 3700
 $Comp
-L R R?
+L Device:R R?
 U 1 1 5BB97D2C
 P 4600 4000
@@
 	6000 3400 5000 3400
 Wire Wire Line
-	5000 3250 5000 3500
-$Comp
-L R R?
+	5000 3250 5000 3400
+$Comp
+L Device:R R?
 U 1 1 5BB97D8F
 P 5000 3100
@@
 Connection ~ 5000 3400
 Wire Wire Line
-	4450 3700 4700 3700
+	4450 3700 4600 3700
 Wire Wire Line
 	4600 3700 4600 3850
@@
 	4600 4250 5000 4250
 Wire Wire Line
-	5000 3900 5000 4350
-$Comp
-L GND #PWR?
+	5000 3900 5000 4250
+$Comp
+L power:GND #PWR?
 U 1 1 5BB97FB0
 P 5000 4350
@@
 Connection ~ 4600 3700
 $Comp
-L BC846B_215 Q?
+L CameraSystem-rescue:BC846B_215 Q?
 U 1 1 5BB98225
 P 4900 3700
+AR Path="/5BB98225" Ref="Q?"  Part="1"
+AR Path="/5BB4D9C1/5BB98225" Ref="Q?"  Part="1"
 F 0 "Q?" H 4774 3866 60  0000 L CNN
 F 1 "BC846B_215" V 5106 3700 60  0000 C CNN
@@
 VDD_3V3_IN
 $Comp
-L CONN_02X02 J?
+L CameraSystem-rescue:CONN_02X02 J?
 U 1 1 5BBA9829
 P 3950 2150
+AR Path="/5BBA9829" Ref="J?"  Part="1"
+AR Path="/5BB4D9C1/5BBA9829" Ref="J?"  Part="1"
 F 0 "J?" H 3950 2300 50  0000 C CNN
 F 1 "CONN_02X02" H 3950 2000 50  0000 C CNN
@@
 	3700 2100 3650 2100
 Wire Wire Line
-	3650 2100 3650 2200
+	3650 2100 3650 2150
 Wire Wire Line
 	3650 2200 3700 2200
@@
 	4250 2200 4200 2200
 Wire Wire Line
-	4250 2100 4250 2200
+	4250 2100 4250 2150
 Wire Wire Line
 	4200 2100 4250 2100
 Connection ~ 4250 2150
+Wire Wire Line
+	5850 3500 6000 3500
+Wire Wire Line
+	5000 3400 5000 3500
+Wire Wire Line
+	5000 4250 5000 4350
+Wire Wire Line
+	4600 3700 4700 3700
+Wire Wire Line
+	3650 2150 3650 2200
+Wire Wire Line
+	4250 2150 4250 2200
 $EndSCHEMATC

Commit message: feat: add debugging pins
Parts:
- removed J?: CONN_02X02, symbol CameraSystem-rescue:CONN_02X02
- added J?: Conn_02x02_Odd_Even, symbol Connector_Generic:Conn_02x02_Odd_Even
Changed lines of the file:
@@
 $EndComp
 $Comp
-L power:GND #PWR?
+L power:GND #PWR0119
 U 1 1 5BB97B4E
 P 5850 4350
-F 0 "#PWR?" H 5850 4100 50  0001 C CNN
+F 0 "#PWR0119" H 5850 4100 50  0001 C CNN
 F 1 "GND" H 5850 4200 50  0000 C CNN
 F 2 "" H 5850 4350 50  0001 C CNN
@@
 	5850 4350 5850 3950
 $Comp
-L power:GND #PWR?
+L power:GND #PWR0120
 U 1 1 5BB97B87
 P 7750 3300
-F 0 "#PWR?" H 7750 3050 50  0001 C CNN
+F 0 "#PWR0120" H 7750 3050 50  0001 C CNN
 F 1 "GND" H 7750 3150 50  0000 C CNN
 F 2 "" H 7750 3300 50  0001 C CNN
@@
 	5000 3900 5000 4250
 $Comp
-L power:GND #PWR?
+L power:GND #PWR0121
 U 1 1 5BB97FB0
 P 5000 4350
-F 0 "#PWR?" H 5000 4100 50  0001 C CNN
+F 0 "#PWR0121" H 5000 4100 50  0001 C CNN
 F 1 "GND" H 5000 4200 50  0000 C CNN
 F 2 "" H 5000 4350 50  0001 C CNN
@@
 Text Label 5350 3500 0    60   ~ 0
 VDD_3V3_IN
-$Comp
-L CameraSystem-rescue:CONN_02X02 J?
-U 1 1 5BBA9829
-P 3950 2150
-AR Path="/5BBA9829" Ref="J?"  Part="1"
-AR Path="/5BB4D9C1/5BBA9829" Ref="J?"  Part="1"
-F 0 "J?" H 3950 2300 50  0000 C CNN
-F 1 "CONN_02X02" H 3950 2000 50  0000 C CNN
-F 2 "" H 3950 950 50  0001 C CNN
-F 3 "" H 3950 950 50  0001 C CNN
-	1    3950 2150
-	1    0    0    -1
-$EndComp
 Wire Wire Line
 	3700 2100 3650 2100
@@
 Wire Wire Line
 	4250 2150 4250 2200
+$Comp
+L Connector_Generic:Conn_02x02_Odd_Even J?
+U 1 1 5BC6841F
+P 3900 2100
+F 0 "J?" H 3950 2317 50  0000 C CNN
+F 1 "Conn_02x02_Odd_Even" H 3950 2226 50  0000 C CNN
+F 2 "" H 3900 2100 50  0001 C CNN
+F 3 "~" H 3900 2100 50  0001 C CNN
+	1    3900 2100
+	1    0    0    -1
+$EndComp
 $EndSCHEMATC

Commit message: feat: DRC run
Parts:
- C18: renamed from C?; footprint (none) -> Capacitor_SMD:C_0603_1608Metric_Pad1.05x0.95mm_HandSolder
- R22, R23, R24: renamed from R?; footprint (none) -> Resistor_SMD:R_0603_1608Metric_Pad1.05x0.95mm_HandSolder
- gave numbers to parts that had none: 3
Connections:
- no-connect marks 0 -> 2
Changed lines of the file:
@@
 WIFI_EN
 $Comp
-L cl-integrated_circuits:ESP8266 U?
+L cl-integrated_circuits:ESP8266 U4
 U 1 1 5BB97A97
 P 6500 3350
-F 0 "U?" H 6500 3050 60  0000 C CNN
+F 0 "U4" H 6500 3050 60  0000 C CNN
 F 1 "ESP8266" H 6500 3650 60  0000 C CNN
 F 2 "" H 6500 3350 60  0001 C CNN
@@
 $EndComp
 $Comp
-L Device:C C?
+L Device:C C18
 U 1 1 5BB97B07
 P 5850 3800
-F 0 "C?" H 5875 3900 50  0000 L CNN
+F 0 "C18" H 5875 3900 50  0000 L CNN
 F 1 "100n" H 5875 3700 50  0000 L CNN
-F 2 "" H 5888 3650 50  0001 C CNN
+F 2 "Capacitor_SMD:C_0603_1608Metric_Pad1.05x0.95mm_HandSolder" H 5888 3650 50  0001 C CNN
 F 3 "" H 5850 3800 50  0001 C CNN
 	1    5850 3800
@@
 	6000 3300 5700 3300
 $Comp
-L Device:R R?
+L Device:R R22
 U 1 1 5BB97CCF
 P 4300 3700
-F 0 "R?" V 4380 3700 50  0000 C CNN
+F 0 "R22" V 4380 3700 50  0000 C CNN
 F 1 "4K7" V 4300 3700 50  0000 C CNN
-F 2 "" V 4230 3700 50  0001 C CNN
+F 2 "Resistor_SMD:R_0603_1608Metric_Pad1.05x0.95mm_HandSolder" V 4230 3700 50  0001 C CNN
 F 3 "" H 4300 3700 50  0001 C CNN
 	1    4300 3700
@@
 	4050 3700 4150 3700
 $Comp
-L Device:R R?
+L Device:R R23
 U 1 1 5BB97D2C
 P 4600 4000
-F 0 "R?" V 4680 4000 50  0000 C CNN
+F 0 "R23" V 4680 4000 50  0000 C CNN
 F 1 "10k" V 4600 4000 50  0000 C CNN
-F 2 "" V 4530 4000 50  0001 C CNN
+F 2 "Resistor_SMD:R_0603_1608Metric_Pad1.05x0.95mm_HandSolder" V 4530 4000 50  0001 C CNN
 F 3 "" H 4600 4000 50  0001 C CNN
 	1    4600 4000
@@
 	5000 3250 5000 3400
 $Comp
-L Device:R R?
+L Device:R R24
 U 1 1 5BB97D8F
 P 5000 3100
-F 0 "R?" V 5080 3100 50  0000 C CNN
+F 0 "R24" V 5080 3100 50  0000 C CNN
 F 1 "10k" V 5000 3100 50  0000 C CNN
-F 2 "" V 4930 3100 50  0001 C CNN
+F 2 "Resistor_SMD:R_0603_1608Metric_Pad1.05x0.95mm_HandSolder" V 4930 3100 50  0001 C CNN
 F 3 "" H 5000 3100 50  0001 C CNN
 	1    5000 3100
@@
 P 4900 3700
 AR Path="/5BB98225" Ref="Q?"  Part="1"
-AR Path="/5BB4D9C1/5BB98225" Ref="Q?"  Part="1"
-F 0 "Q?" H 4774 3866 60  0000 L CNN
+AR Path="/5BB4D9C1/5BB98225" Ref="Q1"  Part="1"
+F 0 "Q1" H 4774 3866 60  0000 L CNN
 F 1 "BC846B_215" V 5106 3700 60  0000 C CNN
 F 2 "digikey-footprints:SOT-23-3" H 5100 3900 60  0001 L CNN
@@
 	4250 2150 4250 2200
 $Comp
-L Connector_Generic:Conn_02x02_Odd_Even J?
+L Connector_Generic:Conn_02x02_Odd_Even J6
 U 1 1 5BC6841F
 P 3900 2100
-F 0 "J?" H 3950 2317 50  0000 C CNN
+F 0 "J6" H 3950 2317 50  0000 C CNN
 F 1 "Conn_02x02_Odd_Even" H 3950 2226 50  0000 C CNN
 F 2 "" H 3900 2100 50  0001 C CNN
@@
 	1    0    0    -1
 $EndComp
+NoConn ~ 7000 3400
+NoConn ~ 7000 3300
 $EndSCHEMATC
