File: Projects/CameraSystem/Schematics/WIFI.sch (KiCad schematic (older format))
At the start: 7 parts, among them J6 Conn_02x02_Odd_Even, Q1 BC846B_215, U4 ESP8266

Commit message: feat: symbol assignment updated
Parts:
- C18: footprint Capacitor_SMD:C_0603_1608Metric_Pad1.05x0.95mm_HandSolder -> digikey-footprints:0603
- R22, R23, R24: footprint Resistor_SMD:R_0603_1608Metric_Pad1.05x0.95mm_HandSolder -> digikey-footprints:0603
Changed lines of the file:
@@
 F 0 "C18" H 5875 3900 50  0000 L CNN
 F 1 "100n" H 5875 3700 50  0000 L CNN
-F 2 "Capacitor_SMD:C_0603_1608Metric_Pad1.05x0.95mm_HandSolder" H 5888 3650 50  0001 C CNN
+F 2 "digikey-footprints:0603" H 5888 3650 50  0001 C CNN
 F 3 "" H 5850 3800 50  0001 C CNN
 	1    5850 3800
@@
 F 0 "R22" V 4380 3700 50  0000 C CNN
 F 1 "4K7" V 4300 3700 50  0000 C CNN
-F 2 "Resistor_SMD:R_0603_1608Metric_Pad1.05x0.95mm_HandSolder" V 4230 3700 50  0001 C CNN
+F 2 "digikey-footprints:0603" V 4230 3700 50  0001 C CNN
 F 3 "" H 4300 3700 50  0001 C CNN
 	1    4300 3700
@@
 F 0 "R23" V 4680 4000 50  0000 C CNN
 F 1 "10k" V 4600 4000 50  0000 C CNN
-F 2 "Resistor_SMD:R_0603_1608Metric_Pad1.05x0.95mm_HandSolder" V 4530 4000 50  0001 C CNN
+F 2 "digikey-footprints:0603" V 4530 4000 50  0001 C CNN
 F 3 "" H 4600 4000 50  0001 C CNN
 	1    4600 4000
@@
 F 0 "R24" V 5080 3100 50  0000 C CNN
 F 1 "10k" V 5000 3100 50  0000 C CNN
-F 2 "Resistor_SMD:R_0603_1608Metric_Pad1.05x0.95mm_HandSolder" V 4930 3100 50  0001 C CNN
+F 2 "digikey-footprints:0603" V 4930 3100 50  0001 C CNN
 F 3 "" H 5000 3100 50  0001 C CNN
 	1    5000 3100

Commit message: feat: assign footprints
Parts:
- J6: footprint (none) -> Pin_Headers:Pin_Header_Straight_2x02_Pitch2.54mm_SMD
- U4: footprint (none) -> Pin_Headers:Pin_Header_Straight_2x08_Pitch2.54mm
Changed lines of the file:
@@
 F 0 "U4" H 6500 3050 60  0000 C CNN
 F 1 "ESP8266" H 6500 3650 60  0000 C CNN
-F 2 "" H 6500 3350 60  0001 C CNN
+F 2 "Pin_Headers:Pin_Header_Straight_2x08_Pitch2.54mm" H 6500 3350 60  0001 C CNN
 F 3 "" H 6500 3350 60  0001 C CNN
 	1    6500 3350
@@
 F 0 "J6" H 3950 2317 50  0000 C CNN
 F 1 "Conn_02x02_Odd_Even" H 3950 2226 50  0000 C CNN
-F 2 "" H 3900 2100 50  0001 C CNN
+F 2 "Pin_Headers:Pin_Header_Straight_2x02_Pitch2.54mm_SMD" H 3900 2100 50  0001 C CNN
 F 3 "~" H 3900 2100 50  0001 C CNN
 	1    3900 2100

Commit message: feat: start layout
Parts:
- U4: footprint Pin_Headers:Pin_Header_Straight_2x08_Pitch2.54mm -> Pin_Headers:Pin_Header_Straight_2x04_Pitch2.54mm
Changed lines of the file:
@@
 F 0 "U4" H 6500 3050 60  0000 C CNN
 F 1 "ESP8266" H 6500 3650 60  0000 C CNN
-F 2 "Pin_Headers:Pin_Header_Straight_2x08_Pitch2.54mm" H 6500 3350 60  0001 C CNN
+F 2 "Pin_Headers:Pin_Header_Straight_2x04_Pitch2.54mm" H 6500 3350 60  0001 C CNN
 F 3 "" H 6500 3350 60  0001 C CNN
 	1    6500 3350
