File: Projects/CameraSystem/Schematics/Keypad.sch (KiCad schematic (older format))
At the start: 0 parts

Commit message: feat: first draft of uc schematic created
Other:
- note removed: "- LEDs are designed to draw approx 2.5mA (Lower power consumption)\n- Jumpers in the modules prevent overloading during Serial Programming"
Changed lines of the file:
@@
 Comment4 ""
 $EndDescr
-$Sheet
-S 950  1350 900  1500
-U 5BB4C1AE
-F0 "Input_Interface" 60
-F1 "Input_Interface.sch" 60
-F2 "VDD_5V0" O R 1850 1500 60
-F3 "VDD_3V3" O R 1850 1800 60
-F4 "SPI_RST" O R 1850 2100 60
-F5 "SPI_TX" O R 1850 2400 60
-F6 "SPI_RX" I R 1850 2700 60
-$EndSheet
-$Sheet
-S 3550 1650 1100 5300
-U 5BB4D99F
-F0 "Microcontroller" 60
-F1 "Microcontroller.sch" 60
-F2 "VDD_3V3" I L 3550 1800 60
-F3 "SPI_RST" I L 3550 2100 60
-F4 "SPI_TX" O L 3550 2700 60
-F5 "SPI_RX" I L 3550 2400 60
-F6 "MOSI" O R 4650 2400 60
-F7 "MISO" I R 4650 2700 60
-F8 "SCK" O R 4650 3000 60
-F9 "WIFI_EN" O L 3550 3000 60
-F10 "WIFI_RST" O L 3550 3300 60
-F11 "SCL_3V3" O R 4650 2100 60
-F12 "SDA_3V3" B R 4650 1800 60
-F13 "CS" O R 4650 3300 60
-$EndSheet
-$Sheet
-S 950  3500 900  1400
-U 5BB4D9C1
-F0 "Wifi" 60
-F1 "Wifi.sch" 60
-F2 "VDD_3V3" I R 1850 3700 60
-F3 "WIFI_TX" O R 1850 4200 60
-F4 "WIFI_RX" I R 1850 3950 60
-F5 "WIFI_RST" I R 1850 4700 60
-F6 "WIFI_EN" I R 1850 4450 60
-$EndSheet
-$Sheet
-S 6050 2550 1150 1450
-U 5BB4DA56
-F0 "Memory" 60
-F1 "Memory.sch" 60
-F2 "VDD_3V3" I L 6050 2700 60
-F3 "MOSI" I L 6050 2950 60
-F4 "SCK" I L 6050 3550 60
-F5 "SD_CS" I L 6050 3850 60
-F6 "MISO" O L 6050 3250 60
-$EndSheet
-$Sheet
-S 9550 4200 1150 2050
-U 5BB4DA63
-F0 "Camera" 60
-F1 "Camera.sch" 60
-$EndSheet
-Text Notes 7700 1250 0    60   ~ 0
-- LEDs are designed to draw approx 2.5mA (Lower power consumption)\n- Jumpers in the modules prevent overloading during Serial Programming
-Wire Wire Line
-	1850 1800 2050 1800
-Wire Wire Line
-	2050 1800 2300 1800
-Wire Wire Line
-	2300 1800 3550 1800
-Wire Wire Line
-	1850 2100 3550 2100
-Wire Wire Line
-	1850 2400 2300 2400
-Wire Wire Line
-	2300 2400 3550 2400
-Wire Wire Line
-	1850 2700 2550 2700
-Wire Wire Line
-	2550 2700 3550 2700
-Wire Wire Line
-	1850 3700 2050 3700
-Wire Wire Line
-	2050 3700 2050 1800
-Connection ~ 2050 1800
-Wire Wire Line
-	1850 3950 2300 3950
-Wire Wire Line
-	2300 3950 2300 2400
-Connection ~ 2300 2400
-Wire Wire Line
-	1850 4200 2550 4200
-Wire Wire Line
-	2550 4200 2550 2700
-Connection ~ 2550 2700
-Wire Wire Line
-	1850 4450 2850 4450
-Wire Wire Line
-	2850 4450 2850 3000
-Wire Wire Line
-	2850 3000 3550 3000
-Wire Wire Line
-	1850 4700 3150 4700
-Wire Wire Line
-	3150 4700 3150 3300
-Wire Wire Line
-	3150 3300 3550 3300
-Wire Wire Line
-	2300 1800 2300 1500
-Wire Wire Line
-	2300 1500 5850 1500
-Wire Wire Line
-	5850 1500 6050 1500
-Connection ~ 2300 1800
-Wire Wire Line
-	1850 1500 2050 1500
-Wire Wire Line
-	2050 1500 2050 1200
-Wire Wire Line
-	2050 1200 6050 1200
-Wire Wire Line
-	4650 1800 6050 1800
-Wire Wire Line
-	4650 2100 6050 2100
-$Sheet
-S 6050 1050 1150 1200
-U 5BB9CC6E
-F0 "Display" 60
-F1 "Display.sch" 60
-F2 "VDD_5V0" I L 6050 1200 60
-F3 "VDD_3V3" I L 6050 1500 60
-F4 "SDA_3V3" B L 6050 1800 60
-F5 "SCL_3V3" I L 6050 2100 60
-$EndSheet
-Wire Wire Line
-	5850 1500 5850 2700
-Wire Wire Line
-	5850 2700 6050 2700
-Connection ~ 5850 1500
-Wire Wire Line
-	4650 2400 5650 2400
-Wire Wire Line
-	5650 2400 5650 2950
-Wire Wire Line
-	4650 2700 5450 2700
-Wire Wire Line
-	5450 2700 5450 3250
-Wire Wire Line
-	4650 3000 5300 3000
-Wire Wire Line
-	5300 3000 5300 3550
-Wire Wire Line
-	5650 2950 6050 2950
-Wire Wire Line
-	5450 3250 6050 3250
-Wire Wire Line
-	5300 3550 6050 3550
-Wire Wire Line
-	4650 3300 5100 3300
-Wire Wire Line
-	5100 3300 5100 3850
-Wire Wire Line
-	5100 3850 6050 3850
-$Sheet
-S 950  5400 900  1500
-U 5BBB389E
-F0 "Keypad" 60
-F1 "Keypad.sch" 60
-$EndSheet
 $EndSCHEMATC

Commit message: feat: add keypad schematic
Parts:
- added C?: 100n, symbol C
- added K? (x7): TouchPad, symbol TouchPad
- added Q? (x2): BC846B_215, digikey-footprints:SOT-23-3, symbol BC846B_215
- added R? (x9): 4K7, symbol R
- added R? (x4): 10K, symbol R
- added U?: AT42QT1070-SSUR, symbol AT42QT1070-SSUR
Connections:
- net labels added: GND, QT_CHN, QT_RST, SCL_3V3, SDA_3V3, VDD_3V3, _QT_CHN_IN, _QT_RST_IN
- wire segments 0 -> 59

Commit message: feat: 3.3 regulator housing changed due to temperature
Parts:
- C?: symbol C -> Device:C
- K? (x7): symbol TouchPad -> cl-misc:TouchPad
- Q? (x2): symbol BC846B_215 -> CameraSystem-rescue:BC846B_215
- R? (x13): symbol R -> Device:R
- U?: symbol AT42QT1070-SSUR -> cl-integrated_circuits:AT42QT1070-SSUR
Connections:
- wire segments 59 -> 64

Commit message: feat: DRC run
Parts:
- C26: renamed from C?; footprint (none) -> Capacitor_SMD:C_0603_1608Metric_Pad1.05x0.95mm_HandSolder
- R31, R32, R33, R34, R35, R36, R37, R38, R39, R40, R41, R42, R43: renamed from R?; footprint (none) -> Resistor_SMD:R_0603_1608Metric_Pad1.05x0.95mm_HandSolder
- gave numbers to parts that had none: 10
Changed lines of the file:
@@
 VDD_3V3
 $Comp
-L cl-integrated_circuits:AT42QT1070-SSUR U?
+L cl-integrated_circuits:AT42QT1070-SSUR U10
 U 1 1 5BBEA4BE
 P 5100 3500
-F 0 "U?" H 5100 3000 60  0000 C CNN
+F 0 "U10" H 5100 3000 60  0000 C CNN
 F 1 "AT42QT1070-SSUR" H 5100 4000 60  0000 C CNN
 F 2 "" H 5100 3500 60  0001 C CNN
@@
 $EndComp
 $Comp
-L cl-misc:TouchPad K?
+L cl-misc:TouchPad K3
 U 1 1 5BBEA57E
 P 7800 2750
-F 0 "K?" H 7800 2550 60  0000 C CNN
+F 0 "K3" H 7800 2550 60  0000 C CNN
 F 1 "TouchPad" H 7800 2950 60  0000 C CNN
 F 2 "" H 7850 2750 60  0001 C CNN
@@
 $EndComp
 $Comp
-L Device:R R?
+L Device:R R38
 U 1 1 5BBEA671
 P 6050 3300
-F 0 "R?" V 6130 3300 50  0000 C CNN
+F 0 "R38" V 6130 3300 50  0000 C CNN
 F 1 "4K7" V 6050 3300 50  0000 C CNN
-F 2 "" V 5980 3300 50  0001 C CNN
+F 2 "Resistor_SMD:R_0603_1608Metric_Pad1.05x0.95mm_HandSolder" V 5980 3300 50  0001 C CNN
 F 3 "" H 6050 3300 50  0001 C CNN
 	1    6050 3300
@@
 $EndComp
 $Comp
-L Device:R R?
+L Device:R R41
 U 1 1 5BBEA704
 P 6400 3400
-F 0 "R?" V 6480 3400 50  0000 C CNN
+F 0 "R41" V 6480 3400 50  0000 C CNN
 F 1 "4K7" V 6400 3400 50  0000 C CNN
-F 2 "" V 6330 3400 50  0001 C CNN
+F 2 "Resistor_SMD:R_0603_1608Metric_Pad1.05x0.95mm_HandSolder" V 6330 3400 50  0001 C CNN
 F 3 "" H 6400 3400 50  0001 C CNN
 	1    6400 3400
@@
 $EndComp
 $Comp
-L Device:R R?
+L Device:R R39
 U 1 1 5BBEA734
 P 6050 3500
-F 0 "R?" V 6130 3500 50  0000 C CNN
+F 0 "R39" V 6130 3500 50  0000 C CNN
 F 1 "4K7" V 6050 3500 50  0000 C CNN
-F 2 "" V 5980 3500 50  0001 C CNN
+F 2 "Resistor_SMD:R_0603_1608Metric_Pad1.05x0.95mm_HandSolder" V 5980 3500 50  0001 C CNN
 F 3 "" H 6050 3500 50  0001 C CNN
 	1    6050 3500
@@
 $EndComp
 $Comp
-L Device:R R?
+L Device:R R42
 U 1 1 5BBEA762
 P 6400 3600
-F 0 "R?" V 6480 3600 50  0000 C CNN
+F 0 "R42" V 6480 3600 50  0000 C CNN
 F 1 "4K7" V 6400 3600 50  0000 C CNN
-F 2 "" V 6330 3600 50  0001 C CNN
+F 2 "Resistor_SMD:R_0603_1608Metric_Pad1.05x0.95mm_HandSolder" V 6330 3600 50  0001 C CNN
 F 3 "" H 6400 3600 50  0001 C CNN
 	1    6400 3600
@@
 $EndComp
 $Comp
-L Device:R R?
+L Device:R R40
 U 1 1 5BBEA798
 P 6050 3700
-F 0 "R?" V 6130 3700 50  0000 C CNN
+F 0 "R40" V 6130 3700 50  0000 C CNN
 F 1 "4K7" V 6050 3700 50  0000 C CNN
-F 2 "" V 5980 3700 50  0001 C CNN
+F 2 "Resistor_SMD:R_0603_1608Metric_Pad1.05x0.95mm_HandSolder" V 5980 3700 50  0001 C CNN
 F 3 "" H 6050 3700 50  0001 C CNN
 	1    6050 3700
@@
 $EndComp
 $Comp
-L Device:R R?
+L Device:R R43
 U 1 1 5BBEA7D0
 P 6400 3800
-F 0 "R?" V 6480 3800 50  0000 C CNN
+F 0 "R43" V 6480 3800 50  0000 C CNN
 F 1 "4K7" V 6400 3800 50  0000 C CNN
-F 2 "" V 6330 3800 50  0001 C CNN
+F 2 "Resistor_SMD:R_0603_1608Metric_Pad1.05x0.95mm_HandSolder" V 6330 3800 50  0001 C CNN
 F 3 "" H 6400 3800 50  0001 C CNN
 	1    6400 3800
@@
 $EndComp
 $Comp
-L Device:R R?
+L Device:R R34
 U 1 1 5BBEA834
 P 3850 3800
-F 0 "R?" V 3930 3800 50  0000 C CNN
+F 0 "R34" V 3930 3800 50  0000 C CNN
 F 1 "4K7" V 3850 3800 50  0000 C CNN
-F 2 "" V 3780 3800 50  0001 C CNN
+F 2 "Resistor_SMD:R_0603_1608Metric_Pad1.05x0.95mm_HandSolder" V 3780 3800 50  0001 C CNN
 F 3 "" H 3850 3800 50  0001 C CNN
 	1    3850 3800
@@
 	5750 3800 6250 3800
 $Comp
-L cl-misc:TouchPad K?
+L cl-misc:TouchPad K5
 U 1 1 5BBEAA5F
 P 7800 3850
-F 0 "K?" H 7800 3650 60  0000 C CNN
+F 0 "K5" H 7800 3650 60  0000 C CNN
 F 1 "TouchPad" H 7800 4050 60  0000 C CNN
 F 2 "" H 7850 3850 60  0001 C CNN
@@
 $EndComp
 $Comp
-L cl-misc:TouchPad K?
+L cl-misc:TouchPad K4
 U 1 1 5BBEAAB3
 P 7800 3300
-F 0 "K?" H 7800 3100 60  0000 C CNN
+F 0 "K4" H 7800 3100 60  0000 C CNN
 F 1 "TouchPad" H 7800 3500 60  0000 C CNN
 F 2 "" H 7850 3300 60  0001 C CNN
@@
 $EndComp
 $Comp
-L cl-misc:TouchPad K?
+L cl-misc:TouchPad K2
 U 1 1 5BBEAAF6
 P 7800 2250
-F 0 "K?" H 7800 2050 60  0000 C CNN
+F 0 "K2" H 7800 2050 60  0000 C CNN
 F 1 "TouchPad" H 7800 2450 60  0000 C CNN
 F 2 "" H 7850 2250 60  0001 C CNN
@@
 $EndComp
 $Comp
-L cl-misc:TouchPad K?
+L cl-misc:TouchPad K6
 U 1 1 5BBEAD74
 P 7800 4400
-F 0 "K?" H 7800 4200 60  0000 C CNN
+F 0 "K6" H 7800 4200 60  0000 C CNN
 F 1 "TouchPad" H 7800 4600 60  0000 C CNN
 F 2 "" H 7850 4400 60  0001 C CNN
@@
 $EndComp
 $Comp
-L cl-misc:TouchPad K?
+L cl-misc:TouchPad K7
 U 1 1 5BBEADBD
 P 7800 4950
-F 0 "K?" H 7800 4750 60  0000 C CNN
+F 0 "K7" H 7800 4750 60  0000 C CNN
 F 1 "TouchPad" H 7800 5150 60  0000 C CNN
 F 2 "" H 7850 4950 60  0001 C CNN
@@
 $EndComp
 $Comp
-L cl-misc:TouchPad K?
+L cl-misc:TouchPad K1
 U 1 1 5BBEAF3D
 P 2800 3800
-F 0 "K?" H 2800 3600 60  0000 C CNN
+F 0 "K1" H 2800 3600 60  0000 C CNN
 F 1 "TouchPad" H 2800 4000 60  0000 C CNN
 F 2 "" H 2850 3800 60  0001 C CNN
@@
 	3950 3200 3950 2500
 $Comp
-L Device:C C?
+L Device:C C26
 U 1 1 5BBEB7A8
 P 4200 2700
-F 0 "C?" H 4225 2800 50  0000 L CNN
+F 0 "C26" H 4225 2800 50  0000 L CNN
 F 1 "100n" H 4225 2600 50  0000 L CNN
-F 2 "" H 4238 2550 50  0001 C CNN
+F 2 "Capacitor_SMD:C_0603_1608Metric_Pad1.05x0.95mm_HandSolder" H 4238 2550 50  0001 C CNN
 F 3 "" H 4200 2700 50  0001 C CNN
 	1    4200 2700
@@
 P 2450 6100
 AR Path="/5BBED1E8" Ref="Q?"  Part="1"
-AR Path="/5BBB389E/5BBED1E8" Ref="Q?"  Part="1"
-F 0 "Q?" H 2324 6266 60  0000 L CNN
+AR Path="/5BBB389E/5BBED1E8" Ref="Q3"  Part="1"
+F 0 "Q3" H 2324 6266 60  0000 L CNN
 F 1 "BC846B_215" V 2656 6100 60  0000 C CNN
 F 2 "digikey-footprints:SOT-23-3" H 2650 6300 60  0001 L CNN
@@
 $EndComp
 $Comp
-L Device:R R?
+L Device:R R33
 U 1 1 5BBED49D
 P 2550 5400
-F 0 "R?" V 2630 5400 50  0000 C CNN
+F 0 "R33" V 2630 5400 50  0000 C CNN
 F 1 "10K" V 2550 5400 50  0000 C CNN
-F 2 "" V 2480 5400 50  0001 C CNN
+F 2 "Resistor_SMD:R_0603_1608Metric_Pad1.05x0.95mm_HandSolder" V 2480 5400 50  0001 C CNN
 F 3 "" H 2550 5400 50  0001 C CNN
 	1    2550 5400
@@
 	2050 6100 2050 6300
 $Comp
-L Device:R R?
+L Device:R R32
 U 1 1 5BBED791
 P 2050 6450
-F 0 "R?" V 2130 6450 50  0000 C CNN
+F 0 "R32" V 2130 6450 50  0000 C CNN
 F 1 "10K" V 2050 6450 50  0000 C CNN
-F 2 "" V 1980 6450 50  0001 C CNN
+F 2 "Resistor_SMD:R_0603_1608Metric_Pad1.05x0.95mm_HandSolder" V 1980 6450 50  0001 C CNN
 F 3 "" H 2050 6450 50  0001 C CNN
 	1    2050 6450
@@
 $EndComp
 $Comp
-L Device:R R?
+L Device:R R31
 U 1 1 5BBED993
 P 1700 6100
-F 0 "R?" V 1780 6100 50  0000 C CNN
+F 0 "R31" V 1780 6100 50  0000 C CNN
 F 1 "4K7" V 1700 6100 50  0000 C CNN
-F 2 "" V 1630 6100 50  0001 C CNN
+F 2 "Resistor_SMD:R_0603_1608Metric_Pad1.05x0.95mm_HandSolder" V 1630 6100 50  0001 C CNN
 F 3 "" H 1700 6100 50  0001 C CNN
 	1    1700 6100
@@
 P 5250 6100
 AR Path="/5BBEE372" Ref="Q?"  Part="1"
-AR Path="/5BBB389E/5BBEE372" Ref="Q?"  Part="1"
-F 0 "Q?" H 5124 6266 60  0000 L CNN
+AR Path="/5BBB389E/5BBEE372" Ref="Q4"  Part="1"
+F 0 "Q4" H 5124 6266 60  0000 L CNN
 F 1 "BC846B_215" V 5456 6100 60  0000 C CNN
 F 2 "digikey-footprints:SOT-23-3" H 5450 6300 60  0001 L CNN
@@
 $EndComp
 $Comp
-L Device:R R?
+L Device:R R37
 U 1 1 5BBEE378
 P 5350 5400
-F 0 "R?" V 5430 5400 50  0000 C CNN
+F 0 "R37" V 5430 5400 50  0000 C CNN
 F 1 "10K" V 5350 5400 50  0000 C CNN
-F 2 "" V 5280 5400 50  0001 C CNN
+F 2 "Resistor_SMD:R_0603_1608Metric_Pad1.05x0.95mm_HandSolder" V 5280 5400 50  0001 C CNN
 F 3 "" H 5350 5400 50  0001 C CNN
 	1    5350 5400
@@
 	4850 6100 4850 6300
 $Comp
-L Device:R R?
+L Device:R R36
 U 1 1 5BBEE381
 P 4850 6450
-F 0 "R?" V 4930 6450 50  0000 C CNN
+F 0 "R36" V 4930 6450 50  0000 C CNN
 F 1 "10K" V 4850 6450 50  0000 C CNN
-F 2 "" V 4780 6450 50  0001 C CNN
+F 2 "Resistor_SMD:R_0603_1608Metric_Pad1.05x0.95mm_HandSolder" V 4780 6450 50  0001 C CNN
 F 3 "" H 4850 6450 50  0001 C CNN
 	1    4850 6450
@@
 $EndComp
 $Comp
-L Device:R R?
+L Device:R R35
 U 1 1 5BBEE395
 P 4500 6100
-F 0 "R?" V 4580 6100 50  0000 C CNN
+F 0 "R35" V 4580 6100 50  0000 C CNN
 F 1 "4K7" V 4500 6100 50  0000 C CNN
-F 2 "" V 4430 6100 50  0001 C CNN
+F 2 "Resistor_SMD:R_0603_1608Metric_Pad1.05x0.95mm_HandSolder" V 4430 6100 50  0001 C CNN
 F 3 "" H 4500 6100 50  0001 C CNN
 	1    4500 6100

Commit message: feat: add interface to Q Pad
Parts:
- added J? (x2): Conn_01x06, symbol Connector_Generic:Conn_01x06
Connections:
- net labels added: QP_GND, QT_CHN_CON, QT_RST_CON, SCL_3V3_CON, SDA_3V3_CON, VDD_3V3_CON
- wire segments 64 -> 84
Changed lines of the file:
@@
 Comment4 ""
 $EndDescr
-Text HLabel 3650 3200 0    60   Input ~ 0
-VDD_3V3
 $Comp
 L cl-integrated_circuits:AT42QT1070-SSUR U10
@@
 	5850 2850 6150 2850
 Wire Wire Line
-	6150 2850 6150 2950
-$Comp
-L power:GND #PWR0141
-U 1 1 5BBEB5AC
-P 6150 2950
-F 0 "#PWR0141" H 6150 2700 50  0001 C CNN
-F 1 "GND" H 6150 2800 50  0000 C CNN
-F 2 "" H 6150 2950 50  0001 C CNN
-F 3 "" H 6150 2950 50  0001 C CNN
-	1    6150 2950
-	1    0    0    -1
-$EndComp
-Wire Wire Line
 	3650 3200 3950 3200
 Wire Wire Line
@@
 $EndComp
 Connection ~ 3950 3200
-$Comp
-L power:GND #PWR0142
-U 1 1 5BBEBA45
-P 4200 2900
-F 0 "#PWR0142" H 4200 2650 50  0001 C CNN
-F 1 "GND" H 4200 2750 50  0000 C CNN
-F 2 "" H 4200 2900 50  0001 C CNN
-F 3 "" H 4200 2900 50  0001 C CNN
-	1    4200 2900
-	1    0    0    -1
-$EndComp
-Wire Wire Line
-	4200 2900 4200 2850
 Wire Wire Line
 	4200 2550 4200 2500
@@
 	4450 3300 4350 3300
 Wire Wire Line
-	4350 3300 4350 4100
-$Comp
-L power:GND #PWR0143
-U 1 1 5BBEBE54
-P 4350 4100
-F 0 "#PWR0143" H 4350 3850 50  0001 C CNN
-F 1 "GND" H 4350 3950 50  0000 C CNN
-F 2 "" H 4350 4100 50  0001 C CNN
-F 3 "" H 4350 4100 50  0001 C CNN
-	1    4350 4100
-	1    0    0    -1
-$EndComp
-Wire Wire Line
 	4450 3700 3650 3700
 Wire Wire Line
 	4450 3400 3650 3400
-Text HLabel 3650 3400 0    60   BiDi ~ 0
-SDA_3V3
-Text HLabel 3650 3700 0    60   Input ~ 0
-SCL_3V3
 Wire Wire Line
 	4450 3500 3650 3500
@@
 	-1   0    0    1
 $EndComp
-$Comp
-L power:GND #PWR0144
-U 1 1 5BBED885
-P 2050 6750
-F 0 "#PWR0144" H 2050 6500 50  0001 C CNN
-F 1 "GND" H 2050 6600 50  0000 C CNN
-F 2 "" H 2050 6750 50  0001 C CNN
-F 3 "" H 2050 6750 50  0001 C CNN
-	1    2050 6750
-	1    0    0    -1
-$EndComp
 Wire Wire Line
 	2050 6600 2050 6750
 Wire Wire Line
 	2550 6300 2550 6750
-$Comp
-L power:GND #PWR0145
-U 1 1 5BBED94F
-P 2550 6750
-F 0 "#PWR0145" H 2550 6500 50  0001 C CNN
-F 1 "GND" H 2550 6600 50  0000 C CNN
-F 2 "" H 2550 6750 50  0001 C CNN
-F 3 "" H 2550 6750 50  0001 C CNN
-	1    2550 6750
-	1    0    0    -1
-$EndComp
 $Comp
 L Device:R R31
@@
 Text Label 3150 5700 0    60   ~ 0
 _QT_RST_IN
-Text HLabel 1350 6100 0    60   Input ~ 0
-QT_RST
 $Comp
 L CameraSystem-rescue:BC846B_215 Q?
@@
 	-1   0    0    1
 $EndComp
-$Comp
-L power:GND #PWR0146
-U 1 1 5BBEE387
-P 4850 6750
-F 0 "#PWR0146" H 4850 6500 50  0001 C CNN
-F 1 "GND" H 4850 6600 50  0000 C CNN
-F 2 "" H 4850 6750 50  0001 C CNN
-F 3 "" H 4850 6750 50  0001 C CNN
-	1    4850 6750
-	1    0    0    -1
-$EndComp
 Wire Wire Line
 	4850 6600 4850 6750
 Wire Wire Line
 	5350 6300 5350 6750
-$Comp
-L power:GND #PWR0147
-U 1 1 5BBEE38F
-P 5350 6750
-F 0 "#PWR0147" H 5350 6500 50  0001 C CNN
-F 1 "GND" H 5350 6600 50  0000 C CNN
-F 2 "" H 5350 6750 50  0001 C CNN
-F 3 "" H 5350 6750 50  0001 C CNN
-	1    5350 6750
-	1    0    0    -1
-$EndComp
 $Comp
 L Device:R R35
@@
 	5350 5700 5950 5700
 Connection ~ 5350 5700
-Text HLabel 4150 6100 0    60   Input ~ 0
-QT_CHN
 Text Label 5950 5700 0    60   ~ 0
 _QT_CHN_IN
@@
 Wire Wire Line
 	5350 5700 5350 5550
+$Comp
+L Connector_Generic:Conn_01x06 J?
+U 1 1 5BBF5B08
+P 1750 3500
+F 0 "J?" H 1830 3492 50  0000 L CNN
+F 1 "Conn_01x06" H 1830 3401 50  0000 L CNN
+F 2 "" H 1750 3500 50  0001 C CNN
+F 3 "~" H 1750 3500 50  0001 C CNN
+	1    1750 3500
+	1    0    0    -1
+$EndComp
+Text HLabel 1450 3800 0    60   Input ~ 0
+QT_RST_CON
+Text HLabel 1450 3700 0    60   Input ~ 0
+QT_CHN_CON
+Text HLabel 1450 3600 0    60   Input ~ 0
+SCL_3V3_CON
+Text HLabel 1450 3400 0    60   BiDi ~ 0
+SDA_3V3_CON
+Text HLabel 1450 3300 0    60   Input ~ 0
+VDD_3V3_CON
+Wire Wire Line
+	1450 3300 1550 3300
+Wire Wire Line
+	1450 3400 1550 3400
+Wire Wire Line
+	1450 3600 1550 3600
+Wire Wire Line
+	1450 3700 1550 3700
+Wire Wire Line
+	1450 3800 1550 3800
+Wire Wire Line
+	2050 6750 2550 6750
+Connection ~ 2550 6750
+Wire Wire Line
+	2550 6850 2650 6850
+Wire Wire Line
+	2550 6750 2550 6850
+Text Label 2650 6850 0    60   ~ 0
+QP_GND
+Wire Wire Line
+	4850 6750 5350 6750
+Wire Wire Line
+	5350 6750 5350 6850
+Wire Wire Line
+	5350 6850 5450 6850
+Connection ~ 5350 6750
+Text Label 5450 6850 0    60   ~ 0
+QP_GND
+Wire Wire Line
+	4350 4200 4450 4200
+Wire Wire Line
+	4350 3300 4350 4200
+Wire Wire Line
+	4200 3000 4300 3000
+Wire Wire Line
+	4200 2850 4200 3000
+Text Label 4300 3000 0    60   ~ 0
+QP_GND
+Text Label 4450 4200 0    60   ~ 0
+QP_GND
+Text Label 6150 2850 0    60   ~ 0
+QP_GND
+Text Label 1350 6100 2    60   ~ 0
+QT_RST
+Text Label 4150 6100 2    60   ~ 0
+QT_CHN
+Text Label 3650 3200 2    60   ~ 0
+VDD_3V3
+Text Label 3650 3400 2    60   ~ 0
+SDA_3V3
+Text Label 3650 3700 2    60   ~ 0
+SCL_3V3
+$Comp
+L Connector_Generic:Conn_01x06 J?
+U 1 1 5BC19F1B
+P 1750 4450
+F 0 "J?" H 1830 4442 50  0000 L CNN
+F 1 "Conn_01x06" H 1830 4351 50  0000 L CNN
+F 2 "" H 1750 4450 50  0001 C CNN
+F 3 "~" H 1750 4450 50  0001 C CNN
+	1    1750 4450
+	1    0    0    -1
+$EndComp
+Wire Wire Line
+	1450 4250 1550 4250
+Wire Wire Line
+	1450 4350 1550 4350
+Wire Wire Line
+	1450 4450 1550 4450
+Wire Wire Line
+	1450 4550 1550 4550
+Wire Wire Line
+	1450 4650 1550 4650
+Wire Wire Line
+	1450 4750 1550 4750
+Text Label 1450 4250 2    60   ~ 0
+VDD_3V3
+Text Label 1450 4350 2    60   ~ 0
+SDA_3V3
+Text Label 1450 4450 2    60   ~ 0
+QP_GND
+Text Label 1450 4550 2    60   ~ 0
+SCL_3V3
+Text Label 1450 4650 2    60   ~ 0
+QT_CHN
+Text Label 1450 4750 2    60   ~ 0
+QT_RST
+Wire Wire Line
+	650  3500 650  3650
+Wire Wire Line
+	650  3500 1550 3500
+$Comp
+L power:GND #PWR?
+U 1 1 5BC1F64F
+P 650 3650
+F 0 "#PWR?" H 650 3400 50  0001 C CNN
+F 1 "GND" H 655 3477 50  0000 C CNN
+F 2 "" H 650 3650 50  0001 C CNN
+F 3 "" H 650 3650 50  0001 C CNN
+	1    650  3650
+	1    0    0    -1
+$EndComp
 $EndSCHEMATC

Commit message: feat: schematic updated
Parts:
- gave numbers to parts that had none: 2
Changed lines of the file:
@@
 	5350 5700 5350 5550
 $Comp
-L Connector_Generic:Conn_01x06 J?
+L Connector_Generic:Conn_01x06 J11
 U 1 1 5BBF5B08
 P 1750 3500
-F 0 "J?" H 1830 3492 50  0000 L CNN
+F 0 "J11" H 1830 3492 50  0000 L CNN
 F 1 "Conn_01x06" H 1830 3401 50  0000 L CNN
 F 2 "" H 1750 3500 50  0001 C CNN
@@
 SCL_3V3
 $Comp
-L Connector_Generic:Conn_01x06 J?
+L Connector_Generic:Conn_01x06 J12
 U 1 1 5BC19F1B
 P 1750 4450
-F 0 "J?" H 1830 4442 50  0000 L CNN
+F 0 "J12" H 1830 4442 50  0000 L CNN
 F 1 "Conn_01x06" H 1830 4351 50  0000 L CNN
 F 2 "" H 1750 4450 50  0001 C CNN
@@
 	650  3500 1550 3500
 $Comp
-L power:GND #PWR?
+L power:GND #PWR0141
 U 1 1 5BC1F64F
 P 650 3650
-F 0 "#PWR?" H 650 3400 50  0001 C CNN
+F 0 "#PWR0141" H 650 3400 50  0001 C CNN
 F 1 "GND" H 655 3477 50  0000 C CNN
 F 2 "" H 650 3650 50  0001 C CNN
