File: Projects/CameraSystem/Schematics/Display.sch (KiCad schematic (older format))
At the start: 6 parts

Commit message: feat: add i2c ic, add additional datasheets and simulations
Parts:
- removed C?: 100n, symbol C
- removed Q?: BC846B_215, digikey-footprints:SOT-23-3, symbol BC846B_215
- removed R?: 4K7, symbol R
- removed R? (x2): 10k, symbol R
- removed U?: ESP8266, symbol ESP8266
- added C? (x3): 100n, symbol C
- added R?: 1K74, symbol R
- added R? (x2): 0, symbol R
- added R?: 1K47, symbol R
- added U?: LCD_2x16_w_i2c, symbol LCD_2x16_w_i2c
- added U?: PCA9306D_118, digikey-footprints:SOIC-8_W3.9mm, symbol PCA9306D_118
Connections:
- net labels added: SCL_3V3, SCL_5V0, SDA_3V3, SDA_5V0, VDD_5V0
- net labels removed: WIFI_EN, WIFI_RST, WIFI_RX, WIFI_TX
- wire segments 18 -> 30

Commit message: feat: first draft of uc schematic created
Parts:
- R? (x2): value 0 -> 100k
Other:
- note added: "NA"
Changed lines of the file:
@@
 $Descr A4 11693 8268
 encoding utf-8
-Sheet 7 7
+Sheet 7 8
 Title ""
 Date ""
@@
 P 4800 4350
 F 0 "R?" V 4880 4350 50  0000 C CNN
-F 1 "0" V 4800 4350 50  0000 C CNN
+F 1 "100k" V 4800 4350 50  0000 C CNN
 F 2 "" V 4730 4350 50  0001 C CNN
 F 3 "" H 4800 4350 50  0001 C CNN
@@
 P 5000 4350
 F 0 "R?" V 5080 4350 50  0000 C CNN
-F 1 "0" V 5000 4350 50  0000 C CNN
+F 1 "100k" V 5000 4350 50  0000 C CNN
 F 2 "" V 4930 4350 50  0001 C CNN
 F 3 "" H 5000 4350 50  0001 C CNN
@@
 	4800 4500 4800 4850
 Connection ~ 4800 4850
+Text Notes 4650 4250 0    60   ~ 0
+NA
+Text Notes 4850 4250 0    60   ~ 0
+NA
 $EndSCHEMATC

Commit message: feat: 3.3 regulator housing changed due to temperature
Parts:
- removed R? (x2): 100k, symbol R
- C? (x3): symbol C -> Device:C
- R?: symbol R -> Device:R
- R?: value 1K47 -> 1K74; symbol R -> Device:R
- U?: symbol LCD_2x16_w_i2c -> cl-integrated_circuits:LCD_2x16_w_i2c
- U?: symbol PCA9306D_118 -> CameraSystem-rescue:PCA9306D_118
Connections:
- wire segments 30 -> 34
Other:
- note removed: "NA"

Commit message: feat: DRC run
Parts:
- C23, C24, C25: renamed from C?; footprint (none) -> Capacitor_SMD:C_0603_1608Metric_Pad1.05x0.95mm_HandSolder
- R29, R30: renamed from R?; footprint (none) -> Resistor_SMD:R_0603_1608Metric_Pad1.05x0.95mm_HandSolder
- gave numbers to parts that had none: 2
Changed lines of the file:
@@
 SCL_3V3
 $Comp
-L cl-integrated_circuits:LCD_2x16_w_i2c U?
+L cl-integrated_circuits:LCD_2x16_w_i2c U9
 U 1 1 5BB9D5E3
 P 6350 2300
-F 0 "U?" H 6350 1950 60  0000 C CNN
+F 0 "U9" H 6350 1950 60  0000 C CNN
 F 1 "LCD_2x16_w_i2c" H 6350 2650 60  0000 C CNN
 F 2 "" H 6350 2300 60  0001 C CNN
@@
 $EndComp
 $Comp
-L Device:C C?
+L Device:C C23
 U 1 1 5BB9D673
 P 4300 2400
-F 0 "C?" H 4325 2500 50  0000 L CNN
+F 0 "C23" H 4325 2500 50  0000 L CNN
 F 1 "100n" H 4325 2300 50  0000 L CNN
-F 2 "" H 4338 2250 50  0001 C CNN
+F 2 "Capacitor_SMD:C_0603_1608Metric_Pad1.05x0.95mm_HandSolder" H 4338 2250 50  0001 C CNN
 F 3 "" H 4300 2400 50  0001 C CNN
 	1    4300 2400
@@
 P 6100 4850
 AR Path="/5BB9DA52" Ref="U?"  Part="1"
-AR Path="/5BB9CC6E/5BB9DA52" Ref="U?"  Part="1"
-F 0 "U?" H 5900 5300 60  0000 C CNN
+AR Path="/5BB9CC6E/5BB9DA52" Ref="U8"  Part="1"
+F 0 "U8" H 5900 5300 60  0000 C CNN
 F 1 "PCA9306D_118" H 6350 5400 60  0000 R CNN
 F 2 "digikey-footprints:SOIC-8_W3.9mm" H 6300 5050 60  0001 L CNN
@@
 Connection ~ 6200 4150
 $Comp
-L Device:C C?
+L Device:C C25
 U 1 1 5BB9DC5C
 P 6500 4500
-F 0 "C?" H 6525 4600 50  0000 L CNN
+F 0 "C25" H 6525 4600 50  0000 L CNN
 F 1 "100n" H 6525 4400 50  0000 L CNN
-F 2 "" H 6538 4350 50  0001 C CNN
+F 2 "Capacitor_SMD:C_0603_1608Metric_Pad1.05x0.95mm_HandSolder" H 6538 4350 50  0001 C CNN
 F 3 "" H 6500 4500 50  0001 C CNN
 	1    6500 4500
@@
 	6100 3350 6100 4350
 $Comp
-L Device:C C?
+L Device:C C24
 U 1 1 5BB9DEB0
 P 6500 3550
-F 0 "C?" H 6525 3650 50  0000 L CNN
+F 0 "C24" H 6525 3650 50  0000 L CNN
 F 1 "100n" H 6525 3450 50  0000 L CNN
-F 2 "" H 6538 3400 50  0001 C CNN
+F 2 "Capacitor_SMD:C_0603_1608Metric_Pad1.05x0.95mm_HandSolder" H 6538 3400 50  0001 C CNN
 F 3 "" H 6500 3550 50  0001 C CNN
 	1    6500 3550
@@
 	6100 5150 6100 5300
 $Comp
-L Device:R R?
+L Device:R R29
 U 1 1 5BB9E244
 P 5200 4350
-F 0 "R?" V 5280 4350 50  0000 C CNN
+F 0 "R29" V 5280 4350 50  0000 C CNN
 F 1 "1K74" V 5200 4350 50  0000 C CNN
-F 2 "" V 5130 4350 50  0001 C CNN
+F 2 "Resistor_SMD:R_0603_1608Metric_Pad1.05x0.95mm_HandSolder" V 5130 4350 50  0001 C CNN
 F 3 "" H 5200 4350 50  0001 C CNN
 	1    5200 4350
@@
 SCL_5V0
 $Comp
-L Device:R R?
+L Device:R R30
 U 1 1 5BB9E8B2
 P 5400 4350
-F 0 "R?" V 5480 4350 50  0000 C CNN
+F 0 "R30" V 5480 4350 50  0000 C CNN
 F 1 "1K74" V 5400 4350 50  0000 C CNN
-F 2 "" V 5330 4350 50  0001 C CNN
+F 2 "Resistor_SMD:R_0603_1608Metric_Pad1.05x0.95mm_HandSolder" V 5330 4350 50  0001 C CNN
 F 3 "" H 5400 4350 50  0001 C CNN
 	1    5400 4350

Commit message: feat: symbol assignment updated
Parts:
- C23, C24, C25: footprint Capacitor_SMD:C_0603_1608Metric_Pad1.05x0.95mm_HandSolder -> digikey-footprints:0603
- R29, R30: footprint Resistor_SMD:R_0603_1608Metric_Pad1.05x0.95mm_HandSolder -> digikey-footprints:0603
Changed lines of the file:
@@
 F 0 "C23" H 4325 2500 50  0000 L CNN
 F 1 "100n" H 4325 2300 50  0000 L CNN
-F 2 "Capacitor_SMD:C_0603_1608Metric_Pad1.05x0.95mm_HandSolder" H 4338 2250 50  0001 C CNN
+F 2 "digikey-footprints:0603" H 4338 2250 50  0001 C CNN
 F 3 "" H 4300 2400 50  0001 C CNN
 	1    4300 2400
@@
 F 0 "C25" H 6525 4600 50  0000 L CNN
 F 1 "100n" H 6525 4400 50  0000 L CNN
-F 2 "Capacitor_SMD:C_0603_1608Metric_Pad1.05x0.95mm_HandSolder" H 6538 4350 50  0001 C CNN
+F 2 "digikey-footprints:0603" H 6538 4350 50  0001 C CNN
 F 3 "" H 6500 4500 50  0001 C CNN
 	1    6500 4500
@@
 F 0 "C24" H 6525 3650 50  0000 L CNN
 F 1 "100n" H 6525 3450 50  0000 L CNN
-F 2 "Capacitor_SMD:C_0603_1608Metric_Pad1.05x0.95mm_HandSolder" H 6538 3400 50  0001 C CNN
+F 2 "digikey-footprints:0603" H 6538 3400 50  0001 C CNN
 F 3 "" H 6500 3550 50  0001 C CNN
 	1    6500 3550
@@
 F 0 "R29" V 5280 4350 50  0000 C CNN
 F 1 "1K74" V 5200 4350 50  0000 C CNN
-F 2 "Resistor_SMD:R_0603_1608Metric_Pad1.05x0.95mm_HandSolder" V 5130 4350 50  0001 C CNN
+F 2 "digikey-footprints:0603" V 5130 4350 50  0001 C CNN
 F 3 "" H 5200 4350 50  0001 C CNN
 	1    5200 4350
@@
 F 0 "R30" V 5480 4350 50  0000 C CNN
 F 1 "1K74" V 5400 4350 50  0000 C CNN
-F 2 "Resistor_SMD:R_0603_1608Metric_Pad1.05x0.95mm_HandSolder" V 5330 4350 50  0001 C CNN
+F 2 "digikey-footprints:0603" V 5330 4350 50  0001 C CNN
 F 3 "" H 5400 4350 50  0001 C CNN
 	1    5400 4350
