File: Projects/CameraSystem/Schematics/CameraSystem.kicad_pcb (KiCad board)
At the start: 2 copper layers, 1 part, among them J1 USB_B_MICRO_SMD

Commit message: feat: set up layout
Parts:
- added C1: 1u, Capacitors_SMD:C_0603_HandSoldering, F.Cu at (141.1, 106.7)
- added C2: 1u, Capacitors_SMD:C_0603_HandSoldering, F.Cu at (150.9, 104.6)
- added U1: CH340, custom-footprints:SO16, F.Cu at (156.2, 92.6)
- added U2: AZ1117CH-3_3TRG1, digikey-footprints:SOT-223, F.Cu at (141.5, 101.0)
- J1: value USB_B_MICRO_SMD -> 10118192-0001LF; footprint MyLibraries:USB_B_MICRO_SMD -> digikey-footprints:USB_Micro_B_Female_10118192
- moved J1 22.3 mm to (126.2, 104.4), turned to 270 degrees
Connections:
- J1 pad 1: (no net) -> /Input_Interface/VDD_5V0
- J1 pad 5: (no net) -> GND

Commit message: feat: start layout
Parts:
- added C10: 100n, digikey-footprints:0603, F.Cu at (215.7, 152.2)
- added C11: 27p, digikey-footprints:0603, F.Cu at (206.8, 155.2)
- added C12: 27p, digikey-footprints:0603, F.Cu at (204.2, 155.2)
- added C13: 100n, digikey-footprints:0603, F.Cu at (213.2, 152.2)
- added C14: 100n, digikey-footprints:0603, F.Cu at (201.7, 155.2)
- added C15: 100n, digikey-footprints:0603, F.Cu at (216.2, 149.3)
- added C16: 100n, digikey-footprints:0603, F.Cu at (218.7, 149.3)
- added C17: 100n, digikey-footprints:0603, F.Cu at (199.1, 155.2)
- added C18: 100n, digikey-footprints:0603, F.Cu at (240.8, 94.4)
- added C19: 100n, digikey-footprints:0603, F.Cu at (234.6, 126.0)
- added C20: 100n, digikey-footprints:0603, F.Cu at (222.9, 130.3)
- added C21: 100n, digikey-footprints:0603, F.Cu at (173.0, 92.2)
- added C22: 100n, digikey-footprints:0603, F.Cu at (149.3, 94.4)
- added C23: 100n, digikey-footprints:0603, F.Cu at (245.3, 147.7)
- added C24: 100n, digikey-footprints:0603, F.Cu at (245.3, 149.2)
- added C25: 100n, digikey-footprints:0603, F.Cu at (239.9, 155.2)
- added C26: 100n, digikey-footprints:0603, F.Cu at (150.4, 149.7)
- added C27: 100n, digikey-footprints:0603, F.Cu at (226.9, 126.0)
- added C3: 22p, digikey-footprints:0603, F.Cu at (264.5, 123.8)
- added C4: 22p, digikey-footprints:0603, F.Cu at (280.6, 115.1)
- added C5: 100n, digikey-footprints:0603, F.Cu at (30.2, 53.1)
- added C6: 100n, digikey-footprints:0603, F.Cu at (264.5, 122.4)
- added C7: 100n, digikey-footprints:0603, F.Cu at (261.9, 123.8)
- added C8: EEE1VA470WP, custom-footprints:PANASONIC_AL_SMD_D_D8, F.Cu at (257.2, 122.1)
- added C9: EEE1VA470WP, custom-footprints:PANASONIC_AL_SMD_D_D8, F.Cu at (281.7, 125.7)
- added D1: TPD2E001DRLR, digikey-footprints:SOT-553, F.Cu at (29.0, 56.1)
- added D2: APG1608CGKC/T, custom-footprints:LED_APG1608, F.Cu at (269.5, 123.7)
- added D3: APG1608SYKC/T, custom-footprints:LED_APG1608, F.Cu at (272.7, 120.8)
- added D4: APG1608SURKC/T, custom-footprints:LED_APG1608, F.Cu at (269.3, 122.3)
- added D5: BZX84C3V3LT1G, custom-footprints:SOT−23_(TO−236), F.Cu at (213.4, 150.0)
- added D6: APG1608SYKC/T, custom-footprints:LED_APG1608, F.Cu at (218.2, 152.0)
- added F1: MF-MSMF075/24, custom-footprints:PTC_MF-MSMF, F.Cu at (29.6, 47.8)
- added FB1: BLM18PG121SN1D, digikey-footprints:0603, F.Cu at (213.2, 154.1)
- added J10: Conn_02x02_Odd_Even, Pin_Headers:Pin_Header_Straight_2x02_Pitch2.54mm_SMD, F.Cu at (181.1, 64.0)
- added J11: Conn_01x06, Pin_Headers:Pin_Header_Straight_1x06_Pitch2.54mm, F.Cu at (161.2, 110.5)
- added J12: Conn_01x06, Pin_Headers:Pin_Header_Straight_1x06_Pitch2.54mm, F.Cu at (159.4, 175.6)
- added J13: Conn_02x02_Odd_Even, Pin_Headers:Pin_Header_Straight_2x02_Pitch2.54mm_SMD, F.Cu at (247.1, 133.2)
- added J14: Conn_02x05_Odd_Even, Pin_Headers:Pin_Header_Straight_2x05_Pitch2.54mm, F.Cu at (284.5, 143.4)
- added J2: Conn_02x03_Odd_Even, Pin_Headers:Pin_Header_Straight_2x03_Pitch2.54mm, F.Cu at (217.7, 172.0)
- added J3: Conn_01x02, Pin_Headers:Pin_Header_Straight_1x02_Pitch2.54mm, F.Cu at (246.1, 168.7)
- added J4: Conn_01x03, Pin_Headers:Pin_Header_Straight_1x03_Pitch2.54mm, F.Cu at (224.8, 137.8)
- added J5: Conn_01x02, Pin_Headers:Pin_Header_Straight_1x02_Pitch2.54mm, F.Cu at (228.5, 137.8)
- added J6: Conn_02x02_Odd_Even, Pin_Headers:Pin_Header_Straight_2x02_Pitch2.54mm_SMD, F.Cu at (229.1, 77.7)
- added J7: Conn_02x02_Odd_Even, Pin_Headers:Pin_Header_Straight_2x02_Pitch2.54mm_SMD, F.Cu at (244.3, 116.0)
- added J8: DM3D-SF, custom-footprints:DM3D-SF, F.Cu at (32.1, 80.6)
- added J9: Conn_02x02_Odd_Even, Pin_Headers:Pin_Header_Straight_2x02_Pitch2.54mm_SMD, F.Cu at (148.7, 66.8)
- added K1: TouchPad, custom-footprints:QPad_Round_D10, F.Cu at (156.9, 151.0)
- added K2: TouchPad, custom-footprints:QPad_Round_D10, F.Cu at (184.2, 141.0)
- added K3: TouchPad, custom-footprints:QPad_Round_D10, F.Cu at (166.9, 151.0)
- added K4: TouchPad, custom-footprints:QPad_Round_D10, F.Cu at (164.2, 141.0)
- added K5: TouchPad, custom-footprints:QPad_Round_D10, F.Cu at (154.2, 141.0)
- added K6: TouchPad, custom-footprints:QPad_Round_D10, F.Cu at (146.9, 157.3)
- added K7: TouchPad, custom-footprints:QPad_Round_D10, F.Cu at (174.2, 141.0)
- added Q1: BC846B_215, digikey-footprints:SOT-23-3, F.Cu at (265.3, 86.9)
- added Q2: BC846B_215, digikey-footprints:SOT-23-3, F.Cu at (173.6, 89.5)
- added Q3: BC846B_215, digikey-footprints:SOT-23-3, F.Cu at (157.4, 158.0)
- added Q4: BC846B_215, digikey-footprints:SOT-23-3, F.Cu at (153.7, 158.0)
- added R1: 1k, digikey-footprints:0603, F.Cu at (267.6, 121.1)
- added R10: 330, digikey-footprints:0603, F.Cu at (230.5, 142.9)
- added R11: 1M, digikey-footprints:0603, F.Cu at (214.4, 155.6)
- added R12: 10k, digikey-footprints:0603, F.Cu at (237.1, 126.0)
- added R16: 10k, digikey-footprints:0603, F.Cu at (211.9, 155.6)
- added R19: 2K2, digikey-footprints:0603, F.Cu at (209.3, 155.6)
- added R2: 1k, digikey-footprints:0603, F.Cu at (261.9, 125.3)
- added R20: 2K2, digikey-footprints:0603, F.Cu at (215.7, 153.7)
- added R21: 560, digikey-footprints:0603, F.Cu at (218.3, 150.8)
- added R22: 4K7, digikey-footprints:0603, F.Cu at (238.2, 94.4)
- added R23: 10k, digikey-footprints:0603, F.Cu at (235.7, 94.4)
- added R24: 10k, digikey-footprints:0603, F.Cu at (233.1, 94.4)
- added R25: 10k, digikey-footprints:0603, F.Cu at (229.5, 126.0)
- added R26: 10k, digikey-footprints:0603, F.Cu at (176.7, 92.0)
- added R27: 10k, digikey-footprints:0603, F.Cu at (179.9, 88.2)
- added R28: 4k7, digikey-footprints:0603, F.Cu at (143.1, 130.0)
- added R29: 1K74, digikey-footprints:0603, F.Cu at (247.9, 147.7)
- added R3: 560, digikey-footprints:0603, F.Cu at (264.5, 125.3)
- added R30: 1K74, digikey-footprints:0603, F.Cu at (245.3, 150.6)
- added R31: 4K7, digikey-footprints:0603, F.Cu at (150.4, 151.1)
- added R32: 10K, digikey-footprints:0603, F.Cu at (145.7, 163.1)
- added R33: 10K, digikey-footprints:0603, F.Cu at (148.2, 163.1)
- added R34: 4K7, digikey-footprints:0603, F.Cu at (150.8, 163.1)
- added R35: 4K7, digikey-footprints:0603, F.Cu at (153.3, 160.7)
- added R36: 10K, digikey-footprints:0603, F.Cu at (155.9, 160.7)
- added R37: 10K, digikey-footprints:0603, F.Cu at (153.3, 162.1)
- added R38: 4K7, digikey-footprints:0603, F.Cu at (153.3, 163.6)
- added R39: 4K7, digikey-footprints:0603, F.Cu at (160.5, 156.7)
- added R4: 560, digikey-footprints:0603, F.Cu at (270.2, 121.1)
- added R40: 4K7, digikey-footprints:0603, F.Cu at (150.4, 146.7)
- added R41: 4K7, digikey-footprints:0603, F.Cu at (150.4, 148.2)
- added R42: 4K7, digikey-footprints:0603, F.Cu at (143.1, 163.1)
- added R43: 4K7, digikey-footprints:0603, F.Cu at (155.9, 162.1)
- added R5: 560, digikey-footprints:0603, F.Cu at (267.0, 125.1)
- added R6: 330, digikey-footprints:0603, F.Cu at (227.9, 142.9)
- added R7: 330, digikey-footprints:0603, F.Cu at (221.3, 149.3)
- added R8: 10k, digikey-footprints:0603, F.Cu at (217.0, 155.2)
- added R9: 330, digikey-footprints:0603, F.Cu at (196.6, 155.2)
- added S1: KS-01Q-01, digikey-footprints:PushButton_Round_D12mm_THT_KS-01Q-01, F.Cu at (256.0, 156.6)
- added U10: AT42QT1070-SSUR, custom-footprints:AT42QT1070-SSUR, F.Cu at (185.5, 163.8)
- added U3: ATMEGA16A-AU, custom-footprints:QFP80P1200X1200X120-44N, F.Cu at (78.8, 56.7)
- added U4: ESP8266, Pin_Headers:Pin_Header_Straight_2x04_Pitch2.54mm, F.Cu at (227.5, 89.3)
- added U5: MC74HC125ADTR2G, custom-footprints:MC74HC125A_TSSOP−14, F.Cu at (242.8, 121.9)
- added U6: OV7670, Pin_Headers:Pin_Header_Straight_2x08_Pitch2.54mm, F.Cu at (101.0, 100.3)
- added U7: SIT2001BI-S2-33E-24.000000G, custom-footprints:SiT2001B_SOT23, F.Cu at (177.0, 89.4)
- added U8: PCA9306D_118, digikey-footprints:SOIC-8_W3.9mm, F.Cu at (241.3, 150.7)
- added U9: LCD_2x16_w_i2c, Pin_Headers:Pin_Header_Straight_1x04_Pitch2.54mm, F.Cu at (236.8, 148.8)
- added Y1: ABLS-12.000MHZ-B2-T, custom-footprints:ABLS2-10.000MHZ-D4Y-T, F.Cu at (260.7, 102.0)
- added Y2: ABLS2-10.000MHZ-D4Y-T, custom-footprints:ABLS2-10.000MHZ-D4Y-T, F.Cu at (202.9, 138.7)
- C1, C2: footprint Capacitors_SMD:C_0603_HandSoldering -> digikey-footprints:0603
- U2: value AZ1117CH-3_3TRG1 -> AZ1117CD-3.3TRG1DICT-ND; footprint digikey-footprints:SOT-223 -> custom-footprints:TO252-2
- moved U2 132.8 mm to (27.3, 33.1), turned to 0 degrees
- moved J1 114.9 mm to (21.7, 56.8)
- moved U1 28.2 mm to (163.1, 65.3)
Connections:
- C1 pad 1: /Input_Interface/VDD_5V0 -> /Display/VDD_5V0
- C2 pad 1: /Input_Interface/VDD_3V3 -> /Camera/VDD_3V3
- J1 pad 1: /Input_Interface/VDD_5V0 -> Net-(C5-Pad1)
- J1 pad 2: (no net) -> /Input_Interface/USB_DN
- J1 pad 3: (no net) -> /Input_Interface/USB_DP
- U1 pad 1: (no net) -> GND
- U1 pad 13: (no net) -> Net-(C6-Pad1)
- U1 pad 16: (no net) -> /Camera/VDD_3V3
- U1 pad 2: (no net) -> Net-(R2-Pad1)
- U1 pad 3: (no net) -> Net-(R1-Pad1)
- U1 pad 4: (no net) -> /Camera/VDD_3V3
- U1 pad 5: (no net) -> /Input_Interface/USB_DP
- U1 pad 6: (no net) -> /Input_Interface/USB_DN
- U1 pad 7: (no net) -> Net-(C3-Pad1)
- U1 pad 8: (no net) -> Net-(C4-Pad1)
- U2 pad 2: /Input_Interface/VDD_3V3 -> /Camera/VDD_3V3
- U2 pad 3: /Input_Interface/VDD_5V0 -> /Display/VDD_5V0
Routing:
- net Net-(C5-Pad1): track 0.00 -> 8.46 mm
- net /Input_Interface/USB_DP: track 0.00 -> 7.12 mm
- net /Input_Interface/USB_DN: track 0.00 -> 4.31 mm
- net GND: track 0.00 -> 1.85 mm, vias 0 -> 3
- added copper zone on B.Cu, net GND
- added copper zone on F.Cu, net GND
Other:
- board outline added: 100 x 100 mm

Commit message: feat: position components in layout
Parts:
- C3: value 22p -> 27p
- moved C9 261.2 mm to (40.5, 25.5)
- moved C4 256.7 mm to (35.4, 38.9), turned to 90 degrees
- moved C8 243.8 mm to (27.4, 40.9), turned to 90 degrees
- moved R5 242.3 mm to (47.5, 22.6)
- moved D4 239.3 mm to (51.8, 22.6), turned to 180 degrees
- moved C3 235.4 mm to (44.9, 38.9), turned to 90 degrees
- moved C6 232.7 mm to (39.4, 63.0), turned to 270 degrees
- moved R1 229.4 mm to (47.3, 57.1)
- moved Y1 228.0 mm to (40.2, 44.0), turned to 180 degrees
- moved C7 226.9 mm to (43.3, 63.0), turned to 270 degrees
- moved R2 225.8 mm to (47.3, 55.1)
- moved R12 221.8 mm to (22.1, 71.4)
- moved D2 217.0 mm to (60.2, 66.3), turned to 270 degrees
- moved S1 216.6 mm to (84.1, 24.8), turned to 270 degrees
- moved D3 216.0 mm to (63.7, 66.3), turned to 270 degrees
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Connections:
- J11 pad 1: /Camera/VDD_3V3 -> /Camera/SDA_3V3
- J11 pad 2: /Camera/SDA_3V3 -> GND
- J11 pad 3: GND -> /Camera/SCL_3V3
- J11 pad 4: /Camera/SCL_3V3 -> /Microcontroller/QT_CHN
- J11 pad 5: /Microcontroller/QT_CHN -> /Microcontroller/QT_RST
- J11 pad 6: /Microcontroller/QT_RST -> /Camera/VDD_3V3
- J12 pad 1: /Keypad/VDD_3V3 -> /Keypad/SDA_3V3
- J12 pad 2: /Keypad/SDA_3V3 -> /Keypad/QP_GND
- J12 pad 3: /Keypad/QP_GND -> /Keypad/SCL_3V3
- J12 pad 4: /Keypad/SCL_3V3 -> /Keypad/QT_CHN
- J12 pad 5: /Keypad/QT_CHN -> /Keypad/QT_RST
- J12 pad 6: /Keypad/QT_RST -> /Keypad/VDD_3V3
- J8 pad 9: /Memory/_SD_DET -> GND
Routing:
- net /Keypad/VDD_3V3: track 0.00 -> 51.4 mm
- net /Keypad/SDA_3V3: track 0.00 -> 47.5 mm, vias 0 -> 1
- net /Keypad/SCL_3V3: track 0.00 -> 40.9 mm, vias 0 -> 1
- net /Keypad/_QT_CHN_IN: track 0.00 -> 16.1 mm
- net /Keypad/_QT_RST_IN: track 0.00 -> 1.72 mm
- added copper zone on B.Cu, net /Keypad/QP_GND
- added copper zone on F.Cu, net /Keypad/QP_GND

Commit message: feat: update layout
Connections:
- J11 pad 1: /Camera/SDA_3V3 -> /Camera/SCL_3V3
- J11 pad 3: /Camera/SCL_3V3 -> /Camera/SDA_3V3
- J12 pad 1: /Keypad/SDA_3V3 -> /Keypad/SCL_3V3
- J12 pad 3: /Keypad/SCL_3V3 -> /Keypad/SDA_3V3
Routing:
- net Net-(K3-Pad1): track 0.00 -> 78.2 mm
- net Net-(K4-Pad1): track 0.00 -> 67.8 mm
- net Net-(K2-Pad1): track 0.00 -> 60.1 mm
- net Net-(K5-Pad1): track 0.00 -> 51.2 mm
- net Net-(K6-Pad1): track 0.00 -> 33.6 mm
- net Net-(K7-Pad1): track 0.00 -> 23.7 mm
- net /Keypad/_QT_RST_IN: track 1.72 -> 20.9 mm, vias 0 -> 2
- net Net-(K1-Pad1): track 0.00 -> 16.7 mm
- net /Keypad/SCL_3V3: track 40.9 -> 47.7 mm, vias 1 -> 0
- net Net-(R34-Pad1): track 0.00 -> 3.76 mm
- net /Keypad/SDA_3V3: track 47.5 -> 49.3 mm, vias 1 -> 0
- net /Keypad/_QT_CHN_IN: track 16.1 -> 14.5 mm, vias 0 -> 2
Changed lines of the file:
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@@
     (thickness 1.6)
     (drawings 5)
-    (tracks 54)
+    (tracks 101)
     (zones 0)
     (modules 111)
@@
   )
   (setup
-    (last_trace_width 0.3)
+    (last_trace_width 0.5)
     (user_trace_width 0.3)
     (user_trace_width 0.5)
@@
     )
     (pad 1 thru_hole rect (at 0 0 90) (size 1.7 1.7) (drill 1) (layers *.Cu *.Mask)
-      (net 31 /Camera/SDA_3V3))
+      (net 30 /Camera/SCL_3V3))
     (pad 2 thru_hole oval (at 0 2.54 90) (size 1.7 1.7) (drill 1) (layers *.Cu *.Mask)
       (net 1 GND))
     (pad 3 thru_hole oval (at 0 5.08 90) (size 1.7 1.7) (drill 1) (layers *.Cu *.Mask)
-      (net 30 /Camera/SCL_3V3))
+      (net 31 /Camera/SDA_3V3))
     (pad 4 thru_hole oval (at 0 7.62 90) (size 1.7 1.7) (drill 1) (layers *.Cu *.Mask)
       (net 41 /Microcontroller/QT_CHN))
@@
       (net 44 /Keypad/QT_CHN))
     (pad 3 thru_hole oval (at 0 5.08 90) (size 1.7 1.7) (drill 1) (layers *.Cu *.Mask)
-      (net 45 /Keypad/SCL_3V3))
+      (net 46 /Keypad/SDA_3V3))
     (pad 2 thru_hole oval (at 0 2.54 90) (size 1.7 1.7) (drill 1) (layers *.Cu *.Mask)
       (net 16 /Keypad/QP_GND))
     (pad 1 thru_hole rect (at 0 0 90) (size 1.7 1.7) (drill 1) (layers *.Cu *.Mask)
-      (net 46 /Keypad/SDA_3V3))
+      (net 45 /Keypad/SCL_3V3))
     (model ${KISYS3DMOD}/Pin_Headers.3dshapes/Pin_Header_Straight_1x06_Pitch2.54mm.wrl
       (at (xyz 0 0 0))
@@
   (segment (start 29.456 57.92) (end 29.456 56.859) (width 0.3) (layer F.Cu) (net 20) (status 20))
   (segment (start 28.829 58.547) (end 29.456 57.92) (width 0.3) (layer F.Cu) (net 20))
-  (via (at 114.4016 110.3884) (size 0.6) (drill 0.4) (layers F.Cu B.Cu) (net 45))
-  (segment (start 112.2488 111.0488) (end 113.7412 111.0488) (width 0.5) (layer F.Cu) (net 45))
-  (segment (start 113.7412 111.0488) (end 114.4016 110.3884) (width 0.5) (layer F.Cu) (net 45))
-  (segment (start 85.09 97.9424) (end 85.09 93.98) (width 0.5) (layer B.Cu) (net 45))
-  (segment (start 90.1192 102.9716) (end 85.09 97.9424) (width 0.5) (layer B.Cu) (net 45))
-  (segment (start 114.4016 110.3884) (end 106.9848 102.9716) (width 0.5) (layer B.Cu) (net 45))
-  (segment (start 106.9848 102.9716) (end 90.1192 102.9716) (width 0.5) (layer B.Cu) (net 45))
-  (via (at 114.5032 114.1984) (size 0.6) (drill 0.4) (layers F.Cu B.Cu) (net 46))
-  (segment (start 112.2488 114.8588) (end 113.8428 114.8588) (width 0.5) (layer F.Cu) (net 46))
-  (segment (start 113.8428 114.8588) (end 114.5032 114.1984) (width 0.5) (layer F.Cu) (net 46))
-  (segment (start 114.5032 114.1984) (end 105.664 105.3592) (width 0.5) (layer B.Cu) (net 46))
-  (segment (start 105.664 105.3592) (end 87.7824 105.3592) (width 0.5) (layer B.Cu) (net 46))
-  (segment (start 80.01 97.5868) (end 80.01 93.98) (width 0.5) (layer B.Cu) (net 46))
-  (segment (start 87.7824 105.3592) (end 80.01 97.5868) (width 0.5) (layer B.Cu) (net 46))
+  (segment (start 113.5338 111.0488) (end 114.4016 110.181) (width 0.3) (layer F.Cu) (net 45))
+  (segment (start 112.2488 111.0488) (end 113.5338 111.0488) (width 0.3) (layer F.Cu) (net 45))
+  (segment (start 114.4016 110.181) (end 114.4016 106.426) (width 0.3) (layer F.Cu) (net 45))
+  (segment (start 114.4016 106.426) (end 113.4872 105.5116) (width 0.3) (layer F.Cu) (net 45))
+  (segment (start 113.4872 105.5116) (end 100.8888 105.5116) (width 0.3) (layer F.Cu) (net 45))
+  (segment (start 100.8888 105.5116) (end 95.0976 99.7204) (width 0.3) (layer F.Cu) (net 45))
+  (segment (start 95.0976 99.7204) (end 82.4992 99.7204) (width 0.3) (layer F.Cu) (net 45))
+  (segment (start 80.01 97.2312) (end 80.01 93.98) (width 0.3) (layer F.Cu) (net 45))
+  (segment (start 82.4992 99.7204) (end 80.01 97.2312) (width 0.3) (layer F.Cu) (net 45))
+  (segment (start 113.5338 114.8588) (end 116.1288 112.2638) (width 0.3) (layer F.Cu) (net 46))
+  (segment (start 112.2488 114.8588) (end 113.5338 114.8588) (width 0.3) (layer F.Cu) (net 46))
+  (segment (start 116.1288 112.2638) (end 116.1288 105.4608) (width 0.3) (layer F.Cu) (net 46))
+  (segment (start 116.1288 105.4608) (end 115.1128 104.4448) (width 0.3) (layer F.Cu) (net 46))
+  (segment (start 115.1128 104.4448) (end 101.1936 104.4448) (width 0.3) (layer F.Cu) (net 46))
+  (segment (start 101.1936 104.4448) (end 95.6056 98.8568) (width 0.3) (layer F.Cu) (net 46))
+  (segment (start 95.6056 98.8568) (end 87.0204 98.8568) (width 0.3) (layer F.Cu) (net 46))
+  (segment (start 85.09 96.9264) (end 85.09 93.98) (width 0.3) (layer F.Cu) (net 46))
+  (segment (start 87.0204 98.8568) (end 85.09 96.9264) (width 0.3) (layer F.Cu) (net 46))
+  (segment (start 93.2884 106.8832) (end 92.4052 106) (width 0.5) (layer F.Cu) (net 53))
+  (segment (start 108.774 106.8832) (end 93.2884 106.8832) (width 0.5) (layer F.Cu) (net 53))
+  (segment (start 45.0592 118.0592) (end 40 113) (width 0.5) (layer F.Cu) (net 54))
+  (segment (start 98.0044 118.0592) (end 45.0592 118.0592) (width 0.5) (layer F.Cu) (net 54))
+  (segment (start 41.5856 106) (end 27.2288 106) (width 0.5) (layer F.Cu) (net 55))
+  (segment (start 101.0524 116.586) (end 52.1716 116.586) (width 0.5) (layer F.Cu) (net 55))
+  (segment (start 52.1716 116.586) (end 41.5856 106) (width 0.5) (layer F.Cu) (net 55))
+  (segment (start 54.132798 115.1636) (end 54.081998 115.1128) (width 0.5) (layer F.Cu) (net 56))
+  (segment (start 98.0044 115.1636) (end 54.132798 115.1636) (width 0.5) (layer F.Cu) (net 56))
+  (segment (start 54.081998 115.1128) (end 52.4764 115.1128) (width 0.5) (layer F.Cu) (net 56))
+  (segment (start 44.999999 102.999999) (end 40 98) (width 0.5) (layer F.Cu) (net 56))
+  (segment (start 44.999999 107.636399) (end 44.999999 102.999999) (width 0.5) (layer F.Cu) (net 56))
+  (segment (start 52.4764 115.1128) (end 44.999999 107.636399) (width 0.5) (layer F.Cu) (net 56))
+  (segment (start 60.7256 113.6904) (end 53.0352 106) (width 0.5) (layer F.Cu) (net 57))
+  (segment (start 101.0636 113.6904) (end 60.7256 113.6904) (width 0.5) (layer F.Cu) (net 57))
+  (segment (start 74.3908 112.776) (end 67.6148 106) (width 0.5) (layer F.Cu) (net 58))
+  (segment (start 96.5948 112.776) (end 74.3908 112.776) (width 0.5) (layer F.Cu) (net 58))
+  (segment (start 98.106 112.0648) (end 97.306 112.0648) (width 0.5) (layer F.Cu) (net 58))
+  (segment (start 97.306 112.0648) (end 96.5948 112.776) (width 0.5) (layer F.Cu) (net 58))
+  (segment (start 100.2016 110.3884) (end 100.1508 110.3376) (width 0.5) (layer F.Cu) (net 59))
+  (segment (start 101.0016 110.3884) (end 100.2016 110.3884) (width 0.5) (layer F.Cu) (net 59))
+  (segment (start 85.060799 110.999999) (end 80.0608 106) (width 0.5) (layer F.Cu) (net 59))
+  (segment (start 85.510801 111.450001) (end 85.060799 110.999999) (width 0.5) (layer F.Cu) (net 59))
+  (segment (start 95.021201 111.450001) (end 85.510801 111.450001) (width 0.5) (layer F.Cu) (net 59))
+  (segment (start 96.133602 110.3376) (end 95.021201 111.450001) (width 0.5) (layer F.Cu) (net 59))
+  (segment (start 100.1508 110.3376) (end 96.133602 110.3376) (width 0.5) (layer F.Cu) (net 59))
   (segment (start 113.826 97.1804) (end 115.5416 97.1804) (width 0.3) (layer F.Cu) (net 65) (status 30))
+  (segment (start 115.5416 97.8804) (end 115.57 97.9088) (width 0.3) (layer F.Cu) (net 65))
+  (segment (start 115.5416 97.1804) (end 115.5416 97.8804) (width 0.3) (layer F.Cu) (net 65))
+  (via (at 115.57 98.7044) (size 0.6) (drill 0.4) (layers F.Cu B.Cu) (net 65))
+  (segment (start 115.57 97.9088) (end 115.57 98.7044) (width 0.3) (layer F.Cu) (net 65))
+  (segment (start 116.169201 99.303601) (end 116.169201 110.784401) (width 0.3) (layer B.Cu) (net 65))
+  (segment (start 115.57 98.7044) (end 116.169201 99.303601) (width 0.3) (layer B.Cu) (net 65))
+  (segment (start 116.169201 110.784401) (end 116.169201 111.109999) (width 0.3) (layer B.Cu) (net 65))
+  (via (at 114.554 112.7252) (size 0.6) (drill 0.4) (layers F.Cu B.Cu) (net 65))
+  (segment (start 116.169201 111.109999) (end 114.554 112.7252) (width 0.3) (layer B.Cu) (net 65))
+  (segment (start 113.6904 113.5888) (end 112.2488 113.5888) (width 0.3) (layer F.Cu) (net 65))
+  (segment (start 114.554 112.7252) (end 113.6904 113.5888) (width 0.3) (layer F.Cu) (net 65))
   (segment (start 113.826 101.6508) (end 115.5304 101.6508) (width 0.3) (layer F.Cu) (net 67) (status 30))
-  (segment (start 113.826 102.2508) (end 115.7732 104.198) (width 0.3) (layer F.Cu) (net 67))
-  (segment (start 113.826 101.6508) (end 113.826 102.2508) (width 0.3) (layer F.Cu) (net 67))
-  (segment (start 115.7732 104.198) (end 115.7732 111.252) (width 0.3) (layer F.Cu) (net 67))
-  (segment (start 114.7064 112.3188) (end 112.2488 112.3188) (width 0.3) (layer F.Cu) (net 67))
-  (segment (start 115.7732 111.252) (end 114.7064 112.3188) (width 0.3) (layer F.Cu) (net 67))
+  (segment (start 115.5304 102.3508) (end 115.5192 102.362) (width 0.3) (layer F.Cu) (net 67))
+  (segment (start 115.5304 101.6508) (end 115.5304 102.3508) (width 0.3) (layer F.Cu) (net 67))
+  (via (at 115.5192 103.3272) (size 0.6) (drill 0.4) (layers F.Cu B.Cu) (net 67))
+  (segment (start 115.5192 102.362) (end 115.5192 103.3272) (width 0.3) (layer F.Cu) (net 67))
+  (segment (start 115.5192 103.3272) (end 115.5192 110.4392) (width 0.3) (layer B.Cu) (net 67))
+  (via (at 114.5032 111.4552) (size 0.6) (drill 0.4) (layers F.Cu B.Cu) (net 67))
+  (segment (start 115.5192 110.4392) (end 114.5032 111.4552) (width 0.3) (layer B.Cu) (net 67))
+  (segment (start 113.6396 112.3188) (end 112.2488 112.3188) (width 0.3) (layer F.Cu) (net 67))
+  (segment (start 114.5032 111.4552) (end 113.6396 112.3188) (width 0.3) (layer F.Cu) (net 67))
+  (segment (start 112.2488 108.958) (end 110.174 106.8832) (width 0.5) (layer F.Cu) (net 77))
+  (segment (start 112.2488 109.7788) (end 112.2488 108.958) (width 0.5) (layer F.Cu) (net 77))
   (zone (net 1) (net_name GND) (layer F.Cu) (hatch edge 0.508)
     (connect_pads (clearance 0.508))

Commit message: feat: layout updated
Parts:
- moved D6 18.7 mm to (48.8, 39.1), turned to 0 degrees
- moved R21 15.4 mm to (52.1, 39.1), turned to 0 degrees
- moved C4 4.81 mm to (37.1, 43.4), turned to 0 degrees
- moved C3 4.52 mm to (45.2, 43.4), turned to 180 degrees
- moved Y1 3.76 mm to (41.1, 47.6)
- moved K6 2.24 mm to (65.4, 106.8)
- moved K7 2.24 mm to (77.8, 107.3)
- moved K1 2.24 mm to (90.2, 106.1)
- moved C12 1.20 mm to (53.3, 43.4), turned to 0 degrees
- moved J5 1.17 mm to (60.7, 62.5)
- moved C11 1.09 mm to (61.5, 43.4), turned to 180 degrees
- moved R10 0.88 mm to (60.7, 28.3), turned to 270 degrees
- turned R25 to 180 degrees
Connections:
- net /Memory/MISO renamed /Microcontroller/MOSI
- net /Memory/SCK renamed /Microcontroller/SCK
- C19 pad 1: /Microcontroller/CS -> /Memory/VDD_3V3_IN
- C20 pad 2: /Microcontroller/CS -> /Memory/VDD_3V3_IN
- J7 pad 2: /Microcontroller/CS -> /Memory/VDD_3V3_IN
- J7 pad 4: /Microcontroller/CS -> /Memory/VDD_3V3_IN
- J8 pad 4: /Microcontroller/CS -> /Memory/VDD_3V3_IN
- R12 pad 2: /Microcontroller/CS -> /Memory/VDD_3V3_IN
- R25 pad 2: Net-(R25-Pad2) -> /Memory/VDD_3V3_IN
- U5 pad 12: Net-(R25-Pad2) -> /Microcontroller/CS
- U5 pad 14: /Microcontroller/CS -> /Memory/VDD_3V3_IN
Routing:
- net /Camera/VDD_3V3: track 0.00 -> 317.9 mm, vias 0 -> 7
- net /Display/VDD_5V0: track 0.00 -> 116.9 mm, vias 0 -> 4
- net /Camera/SCL_3V3: track 0.00 -> 103.3 mm, vias 0 -> 5
- net /Microcontroller/MOSI: track 0.00 -> 99.2 mm, vias 0 -> 5
- net /Camera/SDA_3V3: track 0.00 -> 96.0 mm, vias 0 -> 4
- net /Microcontroller/SCK: track 0.00 -> 91.9 mm, vias 0 -> 5
- net /Memory/_SD_DET: track 0.00 -> 88.5 mm, vias 0 -> 2
- net /Input_Interface/SPI_RST: track 0.00 -> 85.7 mm, vias 0 -> 4
- net /Microcontroller/MISO: track 0.00 -> 79.8 mm, vias 0 -> 5
- net /Microcontroller/CS: track 0.00 -> 72.9 mm, vias 0 -> 2
- net /Memory/VDD_3V3_IN: track 0.00 -> 41.9 mm, vias 0 -> 2
- net /Microcontroller/QT_RST: track 0.00 -> 38.1 mm, vias 0 -> 1
- net /Microcontroller/QT_CHN: track 0.00 -> 36.2 mm, vias 0 -> 1
- net /Microcontroller/SPI_RX: track 0.00 -> 32.8 mm, vias 0 -> 1
- net /Input_Interface/SPI_RX: track 0.00 -> 31.5 mm, vias 0 -> 1
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