File: Projects/CameraSystem/Schematics/CameraSystem.kicad_pcb (KiCad board)
At the start: 2 copper layers, 100 x 100 mm, 111 parts, among them J1 10118192-0001LF, J10 Conn_02x02_Odd_Even, J11 Conn_01x06, J12 Conn_01x06, J13 Conn_02x02_Odd_Even, J14 Conn_02x05_Odd_Even, J2 Conn_02x03_Odd_Even, J3 Conn_01x02, J4 Conn_01x03, J5 Conn_01x02, J6 Conn_02x02_Odd_Even, J7 Conn_02x02_Odd_Even, J8 DM3D-SF, J9 Conn_02x02_Odd_Even, K1 TouchPad, K2 TouchPad, K3 TouchPad, K4 TouchPad, K5 TouchPad, K6 TouchPad, K7 TouchPad, Q1 BC846B_215, Q2 BC846B_215, Q3 BC846B_215, Q4 BC846B_215, U1 CH340, U10 AT42QT1070-SSUR, U2 AZ1117CD-3.3TRG1DICT-ND, U3 ATMEGA16A-AU, U4 ESP8266, U5 MC74HC125ADTR2G, U6 OV7670, U7 SIT2001BI-S2-33E-24.000000G, U8 PCA9306D_118, U9 LCD_2x16_w_i2c, Y1 ABLS-12.000MHZ-B2-T, Y2 ABLS2-10.000MHZ-D4Y-T

Commit message: feat: update gerber files
Parts:
- added REF**: MountingHole_3mm, Mounting_Holes:MountingHole_3mm, F.Cu at (24.0, 87.4)
- added REF**: MountingHole_3mm, Mounting_Holes:MountingHole_3mm, F.Cu at (24.0, 95.4)
- added REF**: MountingHole_3mm, Mounting_Holes:MountingHole_3mm, F.Cu at (24.0, 116.0)
- added REF**: MountingHole_3mm, Mounting_Holes:MountingHole_3mm, F.Cu at (116.0, 116.0)
- added REF**: MountingHole_3mm, Mounting_Holes:MountingHole_3mm, F.Cu at (116.0, 95.4)
- added REF**: MountingHole_3mm, Mounting_Holes:MountingHole_3mm, F.Cu at (116.0, 87.4)
- added REF**: MountingHole_3mm, Mounting_Holes:MountingHole_3mm, F.Cu at (116.0, 24.0)
- added REF**: MountingHole_3mm, Mounting_Holes:MountingHole_3mm, F.Cu at (24.0, 24.0)
- K1, K2, K3, K4, K5, K6, K7: moved to B.Cu
- moved K7 2.64 mm to (77.6, 104.7)
- moved K4 2.49 mm to (39.4, 97.2)
- moved K6 1.64 mm to (65.4, 105.1)
- moved K2 1.22 mm to (37.8, 112.5)
- moved K5 0.94 mm to (52.7, 105.5)
- moved J1 0.70 mm to (22.4, 56.8)
- moved K3 0.50 mm to (27.3, 105.7)
- moved K1 0.44 mm to (90.2, 105.7)
Connections:
- net /Input_Interface/SPI_RX renamed /Microcontroller/SPI_TX
Routing:
- net Net-(K7-Pad1): track 21.5 -> 20.5 mm, vias 0 -> 1
- net Net-(K4-Pad1): track 65.8 -> 64.9 mm, vias 0 -> 1
- net /Input_Interface/USB_DP: track 19.5 -> 18.7 mm
- net /Input_Interface/USB_DN: track 14.7 -> 14.0 mm
- net Net-(K6-Pad1): track 34.0 -> 33.5 mm, vias 0 -> 1
- net Net-(K2-Pad1): track 58.5 -> 58.3 mm, vias 0 -> 1
- net Net-(K1-Pad1): vias 0 -> 1
- net Net-(K5-Pad1): track 46.7 -> 46.8 mm, vias 0 -> 1
- net Net-(K3-Pad1): vias 0 -> 1
Other:
- board text added: "3.3V"
- board text added: "A"
- board text added: "B"
- board text added: "C"
- board text added: "CAMVIEW V.1 V. Tolentino 16.10.18"
- board text added: "ISP"
- board text added: "MISO"
- board text added: "MOSI"
- board text added: "QPAD V.1 V. Tolentino 16.10.18"
- board text added: "RX"
- board text added: "SCK"
- board text added: "SCL"
- board text added: "SDA"
- board text added: "TX"
