File: Projects/CameraSystem/Schematics/Input_Interface.sch (KiCad schematic (older format))
At the start: 23 parts, among them J1 10118192-0001LF, U1 CH340, U2 AZ1117CD-3.3TRG1DICT-ND, Y1 12MHz

Commit message: feat: assign footprints
Parts:
- U2: footprint (none) -> custom-footprints:TO252-2
- Y1: value 12MHz -> ABLS-12.000MHZ-B2-T; footprint (none) -> custom-footprints:ABLS2-10.000MHZ-D4Y-T
Changed lines of the file:
@@
 P 2550 6350
 F 0 "Y1" H 2550 6500 50  0000 C CNN
-F 1 "12MHz" H 2550 6200 50  0000 C CNN
-F 2 "" H 2550 6350 50  0001 C CNN
+F 1 "ABLS-12.000MHZ-B2-T" H 2550 6200 50  0000 C CNN
+F 2 "custom-footprints:ABLS2-10.000MHZ-D4Y-T" H 2550 6350 50  0001 C CNN
 F 3 "" H 2550 6350 50  0001 C CNN
 	1    2550 6350
@@
 F 0 "U2" H 7825 2215 50  0000 C CNN
 F 1 "AZ1117CD-3.3TRG1DICT-ND" H 7825 2124 50  0000 C CNN
-F 2 "" H 7800 1900 50  0001 C CNN
+F 2 "custom-footprints:TO252-2" H 7800 1900 50  0001 C CNN
 F 3 "" H 7800 1900 50  0001 C CNN
 	1    7800 1900

Commit message: feat: position components in layout
Parts:
- C3: value 22p -> 27p
Changed lines of the file:
@@
 P 2150 6700
 F 0 "C3" H 2175 6800 50  0000 L CNN
-F 1 "22p" H 2175 6600 50  0000 L CNN
+F 1 "27p" H 2175 6600 50  0000 L CNN
 F 2 "digikey-footprints:0603" H 2188 6550 50  0001 C CNN
 F 3 "" H 2150 6700 50  0001 C CNN

Commit message: feat: layout updated
Parts:
- D1: footprint digikey-footprints:SOT-553 -> custom-footprints:TPD2E001DRLR_no_stencil
Connections:
- wire segments 80 -> 88
- no-connect marks 8 -> 7
Changed lines of the file:
@@
-$EndComp
-$Comp
-L CameraSystem-rescue:TPD2E001DRLR D?
-U 1 1 5BB52C47
-P 2900 2150
-AR Path="/5BB52C47" Ref="D?"  Part="1"
-AR Path="/5BB4C1AE/5BB52C47" Ref="D1"  Part="1"
-F 0 "D1" H 2590 2465 60  0000 L CNN
-F 1 "TPD2E001DRLR" H 3030 1700 60  0000 R CNN
-F 2 "digikey-footprints:SOT-553" H 3100 2350 60  0001 L CNN
-F 3 "http://www.ti.com/lit/ds/symlink/tpd2e001.pdf" H 3100 2450 60  0001 L CNN
-F 4 "296-21883-1-ND" H 3100 2550 60  0001 L CNN "Digi-Key_PN"
-F 5 "TPD2E001DRLR" H 3100 2650 60  0001 L CNN "MPN"
-F 6 "Circuit Protection" H 3100 2750 60  0001 L CNN "Category"
-F 7 "TVS - Diodes" H 3100 2850 60  0001 L CNN "Family"
-F 8 "http://www.ti.com/lit/ds/symlink/tpd2e001.pdf" H 3100 2950 60  0001 L CNN "DK_Datasheet_Link"
-F 9 "/product-detail/en/texas-instruments/TPD2E001DRLR/296-21883-1-ND/1629242" H 3100 3050 60  0001 L CNN "DK_Detail_Page"
-F 10 "TVS DIODE 5.5V SOT5" H 3100 3150 60  0001 L CNN "Description"
-F 11 "Texas Instruments" H 3100 3250 60  0001 L CNN "Manufacturer"
-F 12 "Active" H 3100 3350 60  0001 L CNN "Status"
-	1    2900 2150
-	1    0    0    -1
 $EndComp
 $Comp
@@
 	2050 2350 2050 2900
 Wire Wire Line
-	1550 2050 2500 2050
-Wire Wire Line
-	1550 2150 2400 2150
-Wire Wire Line
 	1550 2250 2050 2250
 Wire Wire Line
@@
 NoConn ~ 4200 5950
 NoConn ~ 4200 6050
-NoConn ~ 2800 2550
 Wire Wire Line
 	3950 1600 4750 1600
 Wire Wire Line
 	9700 1900 10300 1900
+Wire Wire Line
+	2400 2150 2250 2150
+Wire Wire Line
+	2250 2150 2250 2050
+Wire Wire Line
+	1550 2050 2250 2050
+Wire Wire Line
+	2500 2050 2300 2050
+Wire Wire Line
+	2300 2050 2300 2200
+Wire Wire Line
+	2300 2200 2150 2200
+Wire Wire Line
+	2150 2200 2150 2150
+Wire Wire Line
+	1550 2150 2150 2150
+$Comp
+L CameraSystem-rescue:TPD2E001DRLR D?
+U 1 1 5BB52C47
+P 2900 2150
+AR Path="/5BB52C47" Ref="D?"  Part="1"
+AR Path="/5BB4C1AE/5BB52C47" Ref="D1"  Part="1"
+F 0 "D1" H 2590 2465 60  0000 L CNN
+F 1 "TPD2E001DRLR" H 3030 1700 60  0000 R CNN
+F 2 "custom-footprints:TPD2E001DRLR_no_stencil" H 3100 2350 60  0001 L CNN
+F 3 "http://www.ti.com/lit/ds/symlink/tpd2e001.pdf" H 3100 2450 60  0001 L CNN
+F 4 "296-21883-1-ND" H 3100 2550 60  0001 L CNN "Digi-Key_PN"
+F 5 "TPD2E001DRLR" H 3100 2650 60  0001 L CNN "MPN"
+F 6 "Circuit Protection" H 3100 2750 60  0001 L CNN "Category"
+F 7 "TVS - Diodes" H 3100 2850 60  0001 L CNN "Family"
+F 8 "http://www.ti.com/lit/ds/symlink/tpd2e001.pdf" H 3100 2950 60  0001 L CNN "DK_Datasheet_Link"
+F 9 "/product-detail/en/texas-instruments/TPD2E001DRLR/296-21883-1-ND/1629242" H 3100 3050 60  0001 L CNN "DK_Detail_Page"
+F 10 "TVS DIODE 5.5V SOT5" H 3100 3150 60  0001 L CNN "Description"
+F 11 "Texas Instruments" H 3100 3250 60  0001 L CNN "Manufacturer"
+F 12 "Active" H 3100 3350 60  0001 L CNN "Status"
+	1    2900 2150
+	1    0    0    -1
+$EndComp
+Wire Wire Line
+	2800 2550 2400 2550
+Wire Wire Line
+	2400 2550 2400 2350
+Connection ~ 2400 2350
 $EndSCHEMATC

Commit message: feat: update gerber files
Connections:
- net labels added: U2U_SPI_RX, U2U_SPI_TX
- net labels removed: SPI_RX, SPI_TX
Changed lines of the file:
@@
 SPI_RST
 Text HLabel 1350 5450 0    60   Output ~ 0
-SPI_TX
+U2U_SPI_TX
 Text HLabel 1350 5550 0    60   Input ~ 0
-SPI_RX
+U2U_SPI_RX
 Wire Wire Line
 	1550 2350 2050 2350
@@
 	8250 5600 8350 5600
 Text Label 8350 5600 0    60   ~ 0
-SPI_TX
+U2U_SPI_TX
 Wire Wire Line
 	8900 5600 9000 5600
 Text Label 9000 5600 0    60   ~ 0
-SPI_RX
+U2U_SPI_RX
 Wire Wire Line
 	8550 4200 8650 4200

Commit message: CameraSystem: BOM updated
Parts:
- C4: value 22p -> 27p
Changed lines of the file:
@@
 P 2900 6700
 F 0 "C4" H 2925 6800 50  0000 L CNN
-F 1 "22p" H 2925 6600 50  0000 L CNN
+F 1 "27p" H 2925 6600 50  0000 L CNN
 F 2 "digikey-footprints:0603" H 2938 6550 50  0001 C CNN
 F 3 "" H 2900 6700 50  0001 C CNN
