File: Projects/CameraSystem/Schematics/Input_Interface.sch (KiCad schematic (older format))
At the start: 23 parts, among them J1 10118192-0001LF, U1 CH340, U2 AZ1117CD-3.3TRG1DICT-ND, Y1 ABLS-12.000MHZ-B2-T

Commit message: replace tvs diodes of camera system
Parts:
- removed D1: TPD2E001DRLR, custom-footprints:TPD2E001DRLR_no_stencil, symbol CameraSystem-rescue:TPD2E001DRLR
- added D? (x3): SMBJ5.0A, symbol cl-semiconductors:UD_TVS
Connections:
- net labels added: USB_SPI_RST, USB_SPI_RX, USB_SPI_TX
- net labels removed: SPI_RST, U2U_SPI_RX, U2U_SPI_TX
- wire segments 88 -> 87
Other:
- moved on the sheet: C7
Changed lines of the file:
@@
 Text Label 2100 5650 0    60   ~ 0
 VDD_3V3
-Text Label 1750 2150 0    60   ~ 0
+Text Label 2650 2150 0    60   ~ 0
 USB_DP
-Text Label 1750 2050 0    60   ~ 0
+Text Label 2650 2050 0    60   ~ 0
 USB_DN
 Text Label 2100 5750 0    60   ~ 0
@@
 Text Label 2100 5850 0    60   ~ 0
 USB_DN
-Text Label 5600 5350 0    60   ~ 0
+Text Label 5900 5350 0    60   ~ 0
 VDD_3V3
 $Comp
@@
 L Device:C C7
 U 1 1 5BB520D4
-P 5450 5600
-F 0 "C7" H 5475 5700 50  0000 L CNN
-F 1 "100n" H 5475 5500 50  0000 L CNN
-F 2 "digikey-footprints:0603" H 5488 5450 50  0001 C CNN
-F 3 "" H 5450 5600 50  0001 C CNN
-	1    5450 5600
+P 5750 5600
+F 0 "C7" H 5775 5700 50  0000 L CNN
+F 1 "100n" H 5775 5500 50  0000 L CNN
+F 2 "digikey-footprints:0603" H 5788 5450 50  0001 C CNN
+F 3 "" H 5750 5600 50  0001 C CNN
+	1    5750 5600
 	1    0    0    -1
 $EndComp
@@
 L power:GND #PWR0104
 U 1 1 5BB52260
-P 5450 5850
-F 0 "#PWR0104" H 5450 5600 50  0001 C CNN
-F 1 "GND" H 5450 5700 50  0000 C CNN
-F 2 "" H 5450 5850 50  0001 C CNN
-F 3 "" H 5450 5850 50  0001 C CNN
-	1    5450 5850
+P 5750 5850
+F 0 "#PWR0104" H 5750 5600 50  0001 C CNN
+F 1 "GND" H 5750 5700 50  0000 C CNN
+F 2 "" H 5750 5850 50  0001 C CNN
+F 3 "" H 5750 5850 50  0001 C CNN
+	1    5750 5850
 	1    0    0    -1
 $EndComp
@@
 Text Notes 4250 3600 0    197  ~ 39
 USB TO UART
-Text HLabel 4850 5650 2    60   Output ~ 0
-SPI_RST
+Text HLabel 4900 5650 2    60   Output ~ 0
+USB_SPI_RST
 Text HLabel 1350 5450 0    60   Output ~ 0
-U2U_SPI_TX
+USB_SPI_TX
 Text HLabel 1350 5550 0    60   Input ~ 0
-U2U_SPI_RX
+USB_SPI_RX
 Wire Wire Line
 	1550 2350 2050 2350
 Wire Wire Line
-	2050 2350 2050 2900
+	2050 2350 2050 2850
 Wire Wire Line
 	1550 2250 2050 2250
@@
 	3000 5850 2100 5850
 Wire Wire Line
-	4200 5350 5450 5350
+	4200 5350 5750 5350
 Wire Wire Line
 	2150 6950 2150 6850
@@
 Connection ~ 2150 6350
 Wire Wire Line
-	5450 5350 5450 5450
-Wire Wire Line
-	5450 5750 5450 5850
+	5750 5350 5750 5450
+Wire Wire Line
+	5750 5750 5750 5850
 Wire Wire Line
 	4400 5650 4200 5650
 Wire Wire Line
-	2400 2150 2400 2350
-Wire Wire Line
-	2400 2350 2500 2350
-Wire Wire Line
-	3100 2650 3100 2900
-Wire Wire Line
 	1550 1950 2400 1950
 Wire Wire Line
@@
 Wire Wire Line
 	2400 1600 3100 1600
-Wire Wire Line
-	3100 1750 3100 1600
 Connection ~ 3100 1600
 Wire Wire Line
@@
 	3450 2150 3450 2900
 Wire Wire Line
-	4700 5650 4850 5650
+	4700 5650 4900 5650
 $Comp
 L Device:R R5
@@
 Wire Wire Line
 	1900 3550 2000 3550
-Connection ~ 5450 5350
+Connection ~ 5750 5350
 $Comp
 L Device:CP C9
@@
 	3450 1600 3650 1600
 Wire Wire Line
-	5450 5350 5600 5350
+	5750 5350 5900 5350
 Wire Wire Line
 	9000 1900 9700 1900
@@
 	9700 1900 10300 1900
 Wire Wire Line
-	2400 2150 2250 2150
-Wire Wire Line
-	2250 2150 2250 2050
-Wire Wire Line
-	1550 2050 2250 2050
-Wire Wire Line
-	2500 2050 2300 2050
-Wire Wire Line
-	2300 2050 2300 2200
-Wire Wire Line
-	2300 2200 2150 2200
-Wire Wire Line
-	2150 2200 2150 2150
-Wire Wire Line
-	1550 2150 2150 2150
-$Comp
-L CameraSystem-rescue:TPD2E001DRLR D?
-U 1 1 5BB52C47
-P 2900 2150
-AR Path="/5BB52C47" Ref="D?"  Part="1"
-AR Path="/5BB4C1AE/5BB52C47" Ref="D1"  Part="1"
-F 0 "D1" H 2590 2465 60  0000 L CNN
-F 1 "TPD2E001DRLR" H 3030 1700 60  0000 R CNN
-F 2 "custom-footprints:TPD2E001DRLR_no_stencil" H 3100 2350 60  0001 L CNN
-F 3 "http://www.ti.com/lit/ds/symlink/tpd2e001.pdf" H 3100 2450 60  0001 L CNN
-F 4 "296-21883-1-ND" H 3100 2550 60  0001 L CNN "Digi-Key_PN"
-F 5 "TPD2E001DRLR" H 3100 2650 60  0001 L CNN "MPN"
-F 6 "Circuit Protection" H 3100 2750 60  0001 L CNN "Category"
-F 7 "TVS - Diodes" H 3100 2850 60  0001 L CNN "Family"
-F 8 "http://www.ti.com/lit/ds/symlink/tpd2e001.pdf" H 3100 2950 60  0001 L CNN "DK_Datasheet_Link"
-F 9 "/product-detail/en/texas-instruments/TPD2E001DRLR/296-21883-1-ND/1629242" H 3100 3050 60  0001 L CNN "DK_Detail_Page"
-F 10 "TVS DIODE 5.5V SOT5" H 3100 3150 60  0001 L CNN "Description"
-F 11 "Texas Instruments" H 3100 3250 60  0001 L CNN "Manufacturer"
-F 12 "Active" H 3100 3350 60  0001 L CNN "Status"
-	1    2900 2150
-	1    0    0    -1
-$EndComp
-Wire Wire Line
-	2800 2550 2400 2550
-Wire Wire Line
-	2400 2550 2400 2350
-Connection ~ 2400 2350
-Wire Wire Line
 	1450 3800 1450 3700
 Wire Wire Line
@@
 Wire Wire Line
 	1450 5550 1500 5550
+Wire Wire Line
+	1550 2050 2500 2050
+Wire Wire Line
+	1550 2150 2300 2150
+$Comp
+L cl-semiconductors:UD_TVS D?
+U 1 1 5C9E1EC0
+P 2300 2350
+F 0 "D?" V 2304 2438 50  0000 L CNN
+F 1 "SMBJ5.0A" V 2395 2438 50  0000 L CNN
+F 2 "" H 2300 2350 50  0001 C CNN
+F 3 "" H 2300 2350 50  0001 C CNN
+	1    2300 2350
+	0    1    1    0
+$EndComp
+$Comp
+L cl-semiconductors:UD_TVS D?
+U 1 1 5C9E1F5C
+P 2500 2500
+F 0 "D?" V 2504 2588 50  0000 L CNN
+F 1 "SMBJ5.0A" V 2595 2588 50  0000 L CNN
+F 2 "" H 2500 2500 50  0001 C CNN
+F 3 "" H 2500 2500 50  0001 C CNN
+	1    2500 2500
+	0    1    1    0
+$EndComp
+Wire Wire Line
+	2300 2850 2050 2850
+Wire Wire Line
+	2300 2150 2300 2250
+Connection ~ 2300 2150
+Wire Wire Line
+	2300 2150 2650 2150
+Wire Wire Line
+	2300 2550 2300 2850
+Connection ~ 2050 2850
+Wire Wire Line
+	2050 2850 2050 2900
+Wire Wire Line
+	2500 2050 2500 2400
+Connection ~ 2500 2050
+Wire Wire Line
+	2500 2050 2650 2050
+Wire Wire Line
+	2500 2700 2500 2850
+Wire Wire Line
+	2500 2850 2300 2850
+Connection ~ 2300 2850
+$Comp
+L cl-semiconductors:UD_TVS D?
+U 1 1 5C9F1686
+P 3100 2500
+F 0 "D?" V 3104 2588 50  0000 L CNN
+F 1 "SMBJ5.0A" V 3195 2588 50  0000 L CNN
+F 2 "" H 3100 2500 50  0001 C CNN
+F 3 "" H 3100 2500 50  0001 C CNN
+	1    3100 2500
+	0    1    1    0
+$EndComp
+Wire Wire Line
+	3100 1600 3100 2400
+Wire Wire Line
+	3100 2700 3100 2900
 $EndSCHEMATC

Commit message: replace tvs diodes of camera system
Parts:
- gave numbers to parts that had none: 3
Changed lines of the file:
@@
 	1550 2150 2300 2150
 $Comp
-L cl-semiconductors:UD_TVS D?
+L cl-semiconductors:UD_TVS D1
 U 1 1 5C9E1EC0
 P 2300 2350
-F 0 "D?" V 2304 2438 50  0000 L CNN
+F 0 "D1" V 2304 2438 50  0000 L CNN
 F 1 "SMBJ5.0A" V 2395 2438 50  0000 L CNN
 F 2 "" H 2300 2350 50  0001 C CNN
@@
 $EndComp
 $Comp
-L cl-semiconductors:UD_TVS D?
+L cl-semiconductors:UD_TVS D5
 U 1 1 5C9E1F5C
 P 2500 2500
-F 0 "D?" V 2504 2588 50  0000 L CNN
+F 0 "D5" V 2504 2588 50  0000 L CNN
 F 1 "SMBJ5.0A" V 2595 2588 50  0000 L CNN
 F 2 "" H 2500 2500 50  0001 C CNN
@@
 Connection ~ 2300 2850
 $Comp
-L cl-semiconductors:UD_TVS D?
+L cl-semiconductors:UD_TVS D7
 U 1 1 5C9F1686
 P 3100 2500
-F 0 "D?" V 3104 2588 50  0000 L CNN
+F 0 "D7" V 3104 2588 50  0000 L CNN
 F 1 "SMBJ5.0A" V 3195 2588 50  0000 L CNN
 F 2 "" H 3100 2500 50  0001 C CNN

Commit message: linux adaptation
Parts:
- removed D1, D5, D7: SMBJ5.0A, symbol cl-semiconductors:UD_TVS
- added D1, D5, D7: SMBJ5.0CA, symbol Device:D_TVS
- D2: value APG1608CGKC/T -> LED; footprint custom-footprints:LED_APG1608 -> LED_SMD:LED_1206_3216Metric
- D3: value APG1608SYKC/T -> LED; footprint custom-footprints:LED_APG1608 -> LED_SMD:LED_1206_3216Metric
- D4: value APG1608SURKC/T -> LED; footprint custom-footprints:LED_APG1608 -> LED_SMD:LED_1206_3216Metric
- U1: symbol cl-integrated_circuits:CH340 -> CameraSystem-rescue:CH340-cl-integrated_circuits
- U2: symbol cl-integrated_circuits:AZ1117CD-3.3TRG1DICT-ND -> CameraSystem-rescue:AZ1117CD-3.3TRG1DICT-ND-cl-integrated_circuits
Changed lines of the file:
@@
 VDD_5V0
 $Comp
-L cl-integrated_circuits:CH340 U1
+L CameraSystem-rescue:CH340-cl-integrated_circuits U1
 U 1 1 5BB4DB29
 P 3600 5650
+AR Path="/5BB4DB29" Ref="U1"  Part="1"
+AR Path="/5BB4C1AE/5BB4DB29" Ref="U1"  Part="1"
 F 0 "U1" H 3600 6150 50  0000 L BNN
 F 1 "CH340" H 3500 5050 50  0000 L BNN
@@
 $EndComp
 $Comp
-L Device:LED D4
-U 1 1 5BB7F63E
-P 9700 2600
-F 0 "D4" H 9700 2700 50  0000 C CNN
-F 1 "APG1608SURKC/T" H 9700 2450 50  0000 C CNN
-F 2 "custom-footprints:LED_APG1608" H 9700 2600 50  0001 C CNN
-F 3 "" H 9700 2600 50  0001 C CNN
-	1    9700 2600
-	0    -1   -1   0
-$EndComp
-$Comp
 L power:GND #PWR0107
 U 1 1 5BB7F6C9
@@
 	1    0    0    -1
 $EndComp
-$Comp
-L Device:LED D2
-U 1 1 5BB82C0F
-P 2200 4400
-F 0 "D2" H 2200 4500 50  0000 C CNN
-F 1 "APG1608CGKC/T" H 2200 4250 50  0000 C CNN
-F 2 "custom-footprints:LED_APG1608" H 2200 4400 50  0001 C CNN
-F 3 "" H 2200 4400 50  0001 C CNN
-	1    2200 4400
-	0    -1   -1   0
-$EndComp
 Wire Wire Line
 	2200 4250 2200 4100
@@
 	1    0    0    -1
 $EndComp
-$Comp
-L Device:LED D3
-U 1 1 5BB82CC8
-P 1450 4400
-F 0 "D3" H 1450 4500 50  0000 C CNN
-F 1 "APG1608SYKC/T" H 1450 4250 50  0000 C CNN
-F 2 "custom-footprints:LED_APG1608" H 1450 4400 50  0001 C CNN
-F 3 "" H 1450 4400 50  0001 C CNN
-	1    1450 4400
-	0    -1   -1   0
-$EndComp
 Wire Wire Line
 	1450 4250 1450 4100
@@
 Imax=750mA
 $Comp
-L cl-integrated_circuits:AZ1117CD-3.3TRG1DICT-ND U2
+L CameraSystem-rescue:AZ1117CD-3.3TRG1DICT-ND-cl-integrated_circuits U2
 U 1 1 5BBEC1C5
 P 7800 1900
@@
 Wire Wire Line
 	1550 2150 2300 2150
-$Comp
-L cl-semiconductors:UD_TVS D1
-U 1 1 5C9E1EC0
-P 2300 2350
-F 0 "D1" V 2304 2438 50  0000 L CNN
-F 1 "SMBJ5.0A" V 2395 2438 50  0000 L CNN
-F 2 "" H 2300 2350 50  0001 C CNN
-F 3 "" H 2300 2350 50  0001 C CNN
-	1    2300 2350
-	0    1    1    0
-$EndComp
-$Comp
-L cl-semiconductors:UD_TVS D5
-U 1 1 5C9E1F5C
-P 2500 2500
-F 0 "D5" V 2504 2588 50  0000 L CNN
-F 1 "SMBJ5.0A" V 2595 2588 50  0000 L CNN
-F 2 "" H 2500 2500 50  0001 C CNN
-F 3 "" H 2500 2500 50  0001 C CNN
-	1    2500 2500
-	0    1    1    0
-$EndComp
 Wire Wire Line
 	2300 2850 2050 2850
@@
 	2500 2850 2300 2850
 Connection ~ 2300 2850
-$Comp
-L cl-semiconductors:UD_TVS D7
-U 1 1 5C9F1686
-P 3100 2500
-F 0 "D7" V 3104 2588 50  0000 L CNN
-F 1 "SMBJ5.0A" V 3195 2588 50  0000 L CNN
-F 2 "" H 3100 2500 50  0001 C CNN
-F 3 "" H 3100 2500 50  0001 C CNN
-	1    3100 2500
+Wire Wire Line
+	3100 1600 3100 2400
+Wire Wire Line
+	3100 2700 3100 2900
+$Comp
+L Device:LED D4
+U 1 1 5CA51920
+P 9700 2600
+F 0 "D4" V 9738 2483 50  0000 R CNN
+F 1 "LED" V 9647 2483 50  0000 R CNN
+F 2 "LED_SMD:LED_1206_3216Metric" H 9700 2600 50  0001 C CNN
+F 3 "~" H 9700 2600 50  0001 C CNN
+	1    9700 2600
+	0    -1   -1   0
+$EndComp
+$Comp
+L Device:LED D2
+U 1 1 5CA51D03
+P 1450 4400
+F 0 "D2" V 1488 4283 50  0000 R CNN
+F 1 "LED" V 1397 4283 50  0000 R CNN
+F 2 "LED_SMD:LED_1206_3216Metric" H 1450 4400 50  0001 C CNN
+F 3 "~" H 1450 4400 50  0001 C CNN
+	1    1450 4400
+	0    -1   -1   0
+$EndComp
+$Comp
+L Device:LED D3
+U 1 1 5CA51D7D
+P 2200 4400
+F 0 "D3" V 2238 4283 50  0000 R CNN
+F 1 "LED" V 2147 4283 50  0000 R CNN
+F 2 "LED_SMD:LED_1206_3216Metric" H 2200 4400 50  0001 C CNN
+F 3 "~" H 2200 4400 50  0001 C CNN
+	1    2200 4400
+	0    -1   -1   0
+$EndComp
+$Comp
+L Device:D_TVS D1
+U 1 1 5CA3FD26
+P 2300 2400
+F 0 "D1" V 2254 2479 50  0000 L CNN
+F 1 "SMBJ5.0CA" V 2345 2479 50  0000 L CNN
+F 2 "" H 2300 2400 50  0001 C CNN
+F 3 "~" H 2300 2400 50  0001 C CNN
+	1    2300 2400
 	0    1    1    0
 $EndComp
-Wire Wire Line
-	3100 1600 3100 2400
-Wire Wire Line
-	3100 2700 3100 2900
+$Comp
+L Device:D_TVS D7
+U 1 1 5CA3FED6
+P 3100 2550
+F 0 "D7" V 3054 2629 50  0000 L CNN
+F 1 "SMBJ5.0CA" V 3145 2629 50  0000 L CNN
+F 2 "" H 3100 2550 50  0001 C CNN
+F 3 "~" H 3100 2550 50  0001 C CNN
+	1    3100 2550
+	0    1    1    0
+$EndComp
+$Comp
+L Device:D_TVS D5
+U 1 1 5CA3FF3A
+P 2500 2550
+F 0 "D5" V 2454 2629 50  0000 L CNN
+F 1 "SMBJ5.0CA" V 2545 2629 50  0000 L CNN
+F 2 "" H 2500 2550 50  0001 C CNN
+F 3 "~" H 2500 2550 50  0001 C CNN
+	1    2500 2550
+	0    1    1    0
+$EndComp
 $EndSCHEMATC

Commit message: camera was updated
Parts:
- C1: renamed from C3; footprint digikey-footprints:0603 -> Capacitor_SMD:C_0603_1608Metric_Pad1.05x0.95mm_HandSolder
- C2: renamed from C4; footprint digikey-footprints:0603 -> Capacitor_SMD:C_0603_1608Metric_Pad1.05x0.95mm_HandSolder
- C3: renamed from C5; footprint digikey-footprints:0603 -> Capacitor_SMD:C_0603_1608Metric_Pad1.05x0.95mm_HandSolder
- C4: renamed from C6; footprint digikey-footprints:0603 -> Capacitor_SMD:C_0603_1608Metric_Pad1.05x0.95mm_HandSolder
- C5: renamed from C7; footprint digikey-footprints:0603 -> Capacitor_SMD:C_0603_1608Metric_Pad1.05x0.95mm_HandSolder
- C7: renamed from C1; footprint digikey-footprints:0603 -> Capacitor_SMD:C_0603_1608Metric_Pad1.05x0.95mm_HandSolder
- C8: renamed from C2; footprint digikey-footprints:0603 -> Capacitor_SMD:C_0603_1608Metric_Pad1.05x0.95mm_HandSolder
- D1: renamed from D2; value LED -> BLUE_LED
- D2: renamed from D3; value LED -> YELLOW_LED
- D3: renamed from D1; footprint (none) -> custom-footprints:SMB_DO-214AA
- D4: renamed from D5; footprint (none) -> custom-footprints:SMB_DO-214AA
- D5: renamed from D7; footprint (none) -> custom-footprints:SMB_DO-214AA
- D6: renamed from D4; value LED -> GREEN_LED
- R1: renamed from R4; footprint digikey-footprints:0603 -> Resistor_SMD:R_0603_1608Metric_Pad1.05x0.95mm_HandSolder
- R2: renamed from R1; footprint digikey-footprints:0603 -> Resistor_SMD:R_0603_1608Metric_Pad1.05x0.95mm_HandSolder
- R3: renamed from R2; footprint digikey-footprints:0603 -> Resistor_SMD:R_0603_1608Metric_Pad1.05x0.95mm_HandSolder
- R4: renamed from R3; footprint digikey-footprints:0603 -> Resistor_SMD:R_0603_1608Metric_Pad1.05x0.95mm_HandSolder
- R5: footprint digikey-footprints:0603 -> Resistor_SMD:R_0603_1608Metric_Pad1.05x0.95mm_HandSolder
- renumbered C8 to C6
Other:
- note removed: "-PLC designed to support 450mA + 2mA (LCD) + 4x2.5mA (LEDs) = 462mA (max)"

Commit message: camera was updated
Parts:
- added D4: SS14, custom-footprints:SMA_DO-214AC, symbol Device:D_Schottky
- U2: footprint custom-footprints:TO252-2 -> Package_TO_SOT_SMD:TO-252-2_TabPin1
- renumbered D4 to D5, D5 to D6, D6 to D7
Connections:
- net at D2.1 (K), R3.1: now also D4.2 (A); no longer U1.2 (TXD)
- new net: D4.1 (K), U1.2 (TXD)
Changed lines of the file:
@@
 F 0 "U2" H 7825 2215 50  0000 C CNN
 F 1 "AZ1117CD-3.3TRG1DICT-ND" H 7825 2124 50  0000 C CNN
-F 2 "custom-footprints:TO252-2" H 7800 1900 50  0001 C CNN
+F 2 "Package_TO_SOT_SMD:TO-252-2_TabPin1" H 7800 1900 50  0001 C CNN
 F 3 "" H 7800 1900 50  0001 C CNN
 	1    7800 1900
@@
 Connection ~ 2200 5450
 Wire Wire Line
-	2200 5450 3000 5450
+	2200 5450 2300 5450
 Wire Wire Line
 	2200 4550 2200 5450
@@
 	3100 2700 3100 2900
 $Comp
-L Device:LED D6
+L Device:LED D7
 U 1 1 5CA51920
 P 9700 2600
-F 0 "D6" V 9738 2483 50  0000 R CNN
+F 0 "D7" V 9738 2483 50  0000 R CNN
 F 1 "GREEN_LED" V 9647 2483 50  0000 R CNN
 F 2 "LED_SMD:LED_1206_3216Metric" H 9700 2600 50  0001 C CNN
@@
 $EndComp
 $Comp
-L Device:D_TVS D5
+L Device:D_TVS D6
 U 1 1 5CA3FED6
 P 3100 2550
-F 0 "D5" V 3054 2629 50  0000 L CNN
+F 0 "D6" V 3054 2629 50  0000 L CNN
 F 1 "SMBJ5.0CA" V 3145 2629 50  0000 L CNN
 F 2 "custom-footprints:SMB_DO-214AA" H 3100 2550 50  0001 C CNN
@@
 $EndComp
 $Comp
-L Device:D_TVS D4
+L Device:D_TVS D5
 U 1 1 5CA3FF3A
 P 2500 2550
-F 0 "D4" V 2454 2629 50  0000 L CNN
+F 0 "D5" V 2454 2629 50  0000 L CNN
 F 1 "SMBJ5.0CA" V 2545 2629 50  0000 L CNN
 F 2 "custom-footprints:SMB_DO-214AA" H 2500 2550 50  0001 C CNN
@@
 	0    1    1    0
 $EndComp
+$Comp
+L Device:D_Schottky D4
+U 1 1 5CAE48C6
+P 2450 5450
+F 0 "D4" H 2450 5234 50  0000 C CNN
+F 1 "SS14" H 2450 5325 50  0000 C CNN
+F 2 "custom-footprints:SMA_DO-214AC" H 2450 5450 50  0001 C CNN
+F 3 "~" H 2450 5450 50  0001 C CNN
+	1    2450 5450
+	-1   0    0    1
+$EndComp
+Wire Wire Line
+	2600 5450 3000 5450
 $EndSCHEMATC

Commit message: SP specs updated
Parts:
- U2: footprint Package_TO_SOT_SMD:TO-252-2_TabPin1 -> Package_TO_SOT_SMD:TO-252-2
Changed lines of the file:
@@
 EESchema Schematic File Version 4
 LIBS:CameraSystem-cache
-EELAYER 29 0
+EELAYER 26 0
 EELAYER END
 $Descr A4 11693 8268
@@
 F 0 "U2" H 7825 2215 50  0000 C CNN
 F 1 "AZ1117CD-3.3TRG1DICT-ND" H 7825 2124 50  0000 C CNN
-F 2 "Package_TO_SOT_SMD:TO-252-2_TabPin1" H 7800 1900 50  0001 C CNN
+F 2 "Package_TO_SOT_SMD:TO-252-2" H 7800 1900 50  0001 C CNN
 F 3 "" H 7800 1900 50  0001 C CNN
 	1    7800 1900

Commit message: camera layout updated
Connections:
- net USB_VCC: now reaches C3.1, D6.1 (A1), F1.2, J1.1
Changed lines of the file:
@@
 Wire Wire Line
 	2600 5450 3000 5450
+Text Label 2550 1600 0    50   ~ 0
+USB_VCC
 $EndSCHEMATC
