File: Projects/Solar_Powered_Battery/Schematics/SolarPanelCharger/Buck_5V0.sch (KiCad schematic (older format))
At the start: 11 parts

Commit message: update solar panel schematic
Parts:
- removed Q?: BC847, Package_TO_SOT_SMD:SOT-23, symbol Transistor_BJT:BC847
- added R11: 3k3, Resistor_SMD:R_0603_1608Metric_Pad1.05x0.95mm_HandSolder, symbol Device:R
- C3: renamed from C?; footprint (none) -> Capacitor_THT:CP_Radial_D5.0mm_P2.50mm
- C4: renamed from C?; footprint (none) -> Capacitor_SMD:C_0603_1608Metric_Pad1.05x0.95mm_HandSolder
- C5: renamed from C?; value 5.6n -> 6n8; footprint (none) -> Capacitor_SMD:C_0603_1608Metric_Pad1.05x0.95mm_HandSolder
- D5: renamed from D?; footprint (none) -> custom-footprints:SMB_DO-214AA
- L1: renamed from L?; footprint (none) -> custom-footprints:CD54
- R12: renamed from R?; value 2k -> 3k3; footprint (none) -> Resistor_SMD:R_0603_1608Metric_Pad1.05x0.95mm_HandSolder
- R13: renamed from R?; value 6k2 -> 5k1; footprint (none) -> Resistor_SMD:R_0603_1608Metric_Pad1.05x0.95mm_HandSolder
- R14, R15: renamed from R?; footprint (none) -> Resistor_SMD:R_0603_1608Metric_Pad1.05x0.95mm_HandSolder
- U3: renamed from U?; footprint (none) -> Package_SO:SOP-8_3.76x4.96mm_P1.27mm
Connections:
- net GND: now also R11.2
- net at C5.1, R12.1, R13.2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: now also R11.1
Changed lines of the file:
@@
 EESchema Schematic File Version 4
+LIBS:SolarPanelCharger-cache
 EELAYER 29 0
 EELAYER END
 $Descr A4 11693 8268
 encoding utf-8
-Sheet 3 3
+Sheet 3 6
 Title ""
 Date ""
@@
 $EndDescr
 $Comp
-L cl-integrated_circuits:TD1583 U?
+L cl-integrated_circuits:TD1583 U3
 U 1 1 5CB23F24
 P 5200 3300
-F 0 "U?" H 5200 3715 50  0000 C CNN
+F 0 "U3" H 5200 3715 50  0000 C CNN
 F 1 "TD1583" H 5200 3624 50  0000 C CNN
-F 2 "" H 5200 3300 50  0001 C CNN
+F 2 "Package_SO:SOP-8_3.76x4.96mm_P1.27mm" H 5200 3300 50  0001 C CNN
 F 3 "" H 5200 3300 50  0001 C CNN
 	1    5200 3300
@@
 NoConn ~ 5500 3350
 $Comp
-L power:GND #PWR?
+L power:GND #PWR014
 U 1 1 5CB248A4
 P 4800 3550
-F 0 "#PWR?" H 4800 3300 50  0001 C CNN
+F 0 "#PWR014" H 4800 3300 50  0001 C CNN
 F 1 "GND" H 4805 3377 50  0000 C CNN
 F 2 "" H 4800 3550 50  0001 C CNN
@@
 BUCK_IN
 $Comp
-L Device:CP C?
+L Device:CP C3
 U 1 1 5CB251E1
 P 3600 3500
-F 0 "C?" H 3718 3591 50  0000 L CNN
+F 0 "C3" H 3718 3591 50  0000 L CNN
 F 1 "100u" H 3718 3500 50  0000 L CNN
-F 2 "" H 3638 3350 50  0001 C CNN
+F 2 "Capacitor_THT:CP_Radial_D5.0mm_P2.50mm" H 3638 3350 50  0001 C CNN
 F 3 "~" H 3600 3500 50  0001 C CNN
 F 4 "16V" H 3718 3409 50  0000 L CNN "Value"
@@
 	3600 3650 3600 3800
 $Comp
-L Device:R R?
+L Device:R R12
 U 1 1 5CB26C42
 P 5800 3750
-F 0 "R?" H 5870 3796 50  0000 L CNN
-F 1 "2k" H 5870 3705 50  0000 L CNN
-F 2 "" V 5730 3750 50  0001 C CNN
+F 0 "R12" H 5870 3796 50  0000 L CNN
+F 1 "3k3" H 5870 3705 50  0000 L CNN
+F 2 "Resistor_SMD:R_0603_1608Metric_Pad1.05x0.95mm_HandSolder" V 5730 3750 50  0001 C CNN
 F 3 "~" H 5800 3750 50  0001 C CNN
 	1    5800 3750
@@
 $EndComp
 $Comp
-L power:GND #PWR?
+L power:GND #PWR016
 U 1 1 5CB27061
 P 5800 4000
-F 0 "#PWR?" H 5800 3750 50  0001 C CNN
+F 0 "#PWR016" H 5800 3750 50  0001 C CNN
 F 1 "GND" H 5805 3827 50  0000 C CNN
 F 2 "" H 5800 4000 50  0001 C CNN
@@
 	5800 3600 5800 3450
 Wire Wire Line
-	5800 3450 5500 3450
-$Comp
-L Device:R R?
+	5800 3450 5600 3450
+$Comp
+L Device:R R13
 U 1 1 5CB277FC
 P 6200 3450
-F 0 "R?" V 6100 3600 50  0000 C CNN
-F 1 "6k2" V 6084 3450 50  0000 C CNN
-F 2 "" V 6130 3450 50  0001 C CNN
+F 0 "R13" V 6100 3600 50  0000 C CNN
+F 1 "5k1" V 6084 3450 50  0000 C CNN
+F 2 "Resistor_SMD:R_0603_1608Metric_Pad1.05x0.95mm_HandSolder" V 6130 3450 50  0001 C CNN
 F 3 "~" H 6200 3450 50  0001 C CNN
 	1    6200 3450
@@
 $EndComp
 $Comp
-L Device:C C?
+L Device:C C5
 U 1 1 5CB27FC5
 P 6200 3850
-F 0 "C?" V 6452 3850 50  0000 C CNN
-F 1 "5.6n" V 6361 3850 50  0000 C CNN
-F 2 "" H 6238 3700 50  0001 C CNN
+F 0 "C5" V 6452 3850 50  0000 C CNN
+F 1 "6n8" V 6361 3850 50  0000 C CNN
+F 2 "Capacitor_SMD:C_0603_1608Metric_Pad1.05x0.95mm_HandSolder" H 6238 3700 50  0001 C CNN
 F 3 "~" H 6200 3850 50  0001 C CNN
 	1    6200 3850
@@
 	6450 3450 6350 3450
 $Comp
-L Device:D_Schottky D?
+L Device:D_Schottky D5
 U 1 1 5CB29B04
 P 4600 3600
-F 0 "D?" V 4554 3679 50  0000 L CNN
+F 0 "D5" V 4554 3679 50  0000 L CNN
 F 1 "SS24" V 4645 3679 50  0000 L CNN
-F 2 "" H 4600 3600 50  0001 C CNN
+F 2 "custom-footprints:SMB_DO-214AA" H 4600 3600 50  0001 C CNN
 F 3 "~" H 4600 3600 50  0001 C CNN
 	1    4600 3600
@@
 	4600 3350 4900 3350
 $Comp
-L power:GND #PWR?
+L power:GND #PWR011
 U 1 1 5CB258ED
 P 3600 3800
-F 0 "#PWR?" H 3600 3550 50  0001 C CNN
+F 0 "#PWR011" H 3600 3550 50  0001 C CNN
 F 1 "GND" H 3605 3627 50  0000 C CNN
 F 2 "" H 3600 3800 50  0001 C CNN
@@
 $EndComp
 $Comp
-L power:GND #PWR?
+L power:GND #PWR013
 U 1 1 5CB2C227
 P 4600 3800
-F 0 "#PWR?" H 4600 3550 50  0001 C CNN
+F 0 "#PWR013" H 4600 3550 50  0001 C CNN
 F 1 "GND" H 4605 3627 50  0000 C CNN
 F 2 "" H 4600 3800 50  0001 C CNN
@@
 $EndComp
 $Comp
-L Device:L L?
+L Device:L L1
 U 1 1 5CB2C6F7
 P 4350 3350
-F 0 "L?" V 4631 3350 50  0000 C CNN
+F 0 "L1" V 4631 3350 50  0000 C CNN
 F 1 "15u" V 4540 3350 50  0000 C CNN
-F 2 "" H 4350 3350 50  0001 C CNN
+F 2 "custom-footprints:CD54" H 4350 3350 50  0001 C CNN
 F 3 "~" H 4350 3350 50  0001 C CNN
 F 4 "1A" V 4449 3350 50  0000 C CNN "Value"
@@
 Connection ~ 4600 3350
 $Comp
-L Device:C C?
+L Device:C C4
 U 1 1 5CB2D093
 P 4100 3600
-F 0 "C?" H 3985 3554 50  0000 R CNN
+F 0 "C4" H 3985 3554 50  0000 R CNN
 F 1 "22u" H 3985 3645 50  0000 R CNN
-F 2 "" H 4138 3450 50  0001 C CNN
+F 2 "Capacitor_SMD:C_0603_1608Metric_Pad1.05x0.95mm_HandSolder" H 4138 3450 50  0001 C CNN
 F 3 "~" H 4100 3600 50  0001 C CNN
 F 4 "10V" H 4100 3600 50  0001 C CNN "Value"
@@
 	4100 3350 4100 3450
 $Comp
-L power:GND #PWR?
+L power:GND #PWR012
 U 1 1 5CB2DD03
 P 4100 3800
-F 0 "#PWR?" H 4100 3550 50  0001 C CNN
+F 0 "#PWR012" H 4100 3550 50  0001 C CNN
 F 1 "GND" H 4105 3627 50  0000 C CNN
 F 2 "" H 4100 3800 50  0001 C CNN
@@
 BUCK_5V0
 $Comp
-L Device:R R?
+L Device:R R14
 U 1 1 5CB2E876
 P 6800 2950
-F 0 "R?" H 6730 2904 50  0000 R CNN
+F 0 "R14" H 6730 2904 50  0000 R CNN
 F 1 "10k" H 6730 2995 50  0000 R CNN
-F 2 "" V 6730 2950 50  0001 C CNN
+F 2 "Resistor_SMD:R_0603_1608Metric_Pad1.05x0.95mm_HandSolder" V 6730 2950 50  0001 C CNN
 F 3 "~" H 6800 2950 50  0001 C CNN
 	1    6800 2950
@@
 BUCK_5V0
 $Comp
-L Device:R R?
+L Device:R R15
 U 1 1 5CB30809
 P 6800 3550
-F 0 "R?" V 7007 3550 50  0000 C CNN
+F 0 "R15" V 7007 3550 50  0000 C CNN
 F 1 "33k" V 6916 3550 50  0000 C CNN
-F 2 "" V 6730 3550 50  0001 C CNN
+F 2 "Resistor_SMD:R_0603_1608Metric_Pad1.05x0.95mm_HandSolder" V 6730 3550 50  0001 C CNN
 F 3 "~" H 6800 3550 50  0001 C CNN
 	1    6800 3550
@@
 BUCK_IN
 $Comp
-L power:GND #PWR?
+L power:GND #PWR017
 U 1 1 5CB328C4
 P 6800 3900
-F 0 "#PWR?" H 6800 3650 50  0001 C CNN
+F 0 "#PWR017" H 6800 3650 50  0001 C CNN
 F 1 "GND" V 6805 3772 50  0000 R CNN
 F 2 "" H 6800 3900 50  0001 C CNN
@@
 Text Label 6650 3250 0    50   ~ 0
 EN
-$Comp
-L Transistor_BJT:BC847 Q?
-U 1 1 5CB3392E
-P 7300 3600
-F 0 "Q?" H 7491 3646 50  0000 L CNN
-F 1 "BC847" H 7491 3555 50  0000 L CNN
-F 2 "Package_TO_SOT_SMD:SOT-23" H 7500 3525 50  0001 L CIN
-F 3 "http://www.infineon.com/dgdl/Infineon-BC847SERIES_BC848SERIES_BC849SERIES_BC850SERIES-DS-v01_01-en.pdf?fileId=db3a304314dca389011541d4630a1657" H 7300 3600 50  0001 L CNN
-	1    7300 3600
+Connection ~ 6800 3250
+Wire Wire Line
+	5500 3250 6800 3250
+$Comp
+L Device:R R11
+U 1 1 5CB1D7FB
+P 5600 3750
+F 0 "R11" H 5670 3796 50  0000 L CNN
+F 1 "3k3" H 5670 3705 50  0000 L CNN
+F 2 "Resistor_SMD:R_0603_1608Metric_Pad1.05x0.95mm_HandSolder" V 5530 3750 50  0001 C CNN
+F 3 "~" H 5600 3750 50  0001 C CNN
+	1    5600 3750
 	-1   0    0    -1
 $EndComp
-$Comp
-L power:GND #PWR?
-U 1 1 5CB382AA
-P 7200 3900
-F 0 "#PWR?" H 7200 3650 50  0001 C CNN
-F 1 "GND" H 7205 3727 50  0000 C CNN
-F 2 "" H 7200 3900 50  0001 C CNN
-F 3 "" H 7200 3900 50  0001 C CNN
-	1    7200 3900
-	1    0    0    -1
-$EndComp
-Wire Wire Line
-	7200 3900 7200 3800
-Wire Wire Line
-	7500 3600 7750 3600
-Text HLabel 7750 3600 2    50   Input ~ 0
-_EN
-Connection ~ 6800 3250
-Wire Wire Line
-	6800 3250 7200 3250
-Wire Wire Line
-	7200 3250 7200 3400
-Wire Wire Line
-	5500 3250 6800 3250
+Wire Wire Line
+	5600 3450 5600 3600
+Connection ~ 5600 3450
+Wire Wire Line
+	5600 3450 5500 3450
+$Comp
+L power:GND #PWR015
+U 1 1 5CB1E0E0
+P 5600 4000
+F 0 "#PWR015" H 5600 3750 50  0001 C CNN
+F 1 "GND" H 5605 3827 50  0000 C CNN
+F 2 "" H 5600 4000 50  0001 C CNN
+F 3 "" H 5600 4000 50  0001 C CNN
+	1    5600 4000
+	1    0    0    -1
+$EndComp
+Wire Wire Line
+	5600 4000 5600 3900
 $EndSCHEMATC
