File: Projects/Solar_Powered_Battery/Schematics/SolarPanelCharger/SolarPanelCharger.kicad_pcb (KiCad board)
At the start: 2 copper layers, 77 parts, among them J1 Conn_01x04_Female, J2 Conn_01x05_Female, J3 USB_B_Female, Q1 BC847, Q2 BC847, Q3 BC847, Q4 AO3401A, Q5 AO3401A, Q6 AO3400, Q7 AO3400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

Commit message: pcb updated
Parts:
- added D11: BLUE, LED_SMD:LED_1206_3216Metric_Pad1.42x1.75mm_HandSolder, F.Cu at (62.7, 32.5)
- added D12: WHITE, LED_SMD:LED_1206_3216Metric_Pad1.42x1.75mm_HandSolder, F.Cu at (62.6, 21.9)
- added R34: 1k, Resistor_SMD:R_0603_1608Metric_Pad1.05x0.95mm_HandSolder, F.Cu at (64.3, 25.2)
- added R35: 1k, Resistor_SMD:R_0603_1608Metric_Pad1.05x0.95mm_HandSolder, F.Cu at (64.3, 29.0)
- moved R13 107.4 mm to (40.4, 37.1)
- moved C5 105.2 mm to (40.4, 38.9), turned to 180 degrees
- moved R12 99.1 mm to (44.4, 38.9)
- moved C4 99.0 mm to (47.2, 29.9), turned to 90 degrees
- moved D5 98.3 mm to (37.4, 24.8), turned to 180 degrees
- moved R11 97.3 mm to (44.4, 40.8)
- moved C3 96.6 mm to (36.4, 30.3), turned to 180 degrees
- moved R14 95.8 mm to (47.3, 34.2), turned to 90 degrees
- moved R15 93.5 mm to (47.3, 38.0), turned to 270 degrees
- moved R28 91.9 mm to (73.1, 53.4), turned to 270 degrees
- moved U2 90.5 mm to (26.1, 53.8), turned to 180 degrees
- moved R5 88.9 mm to (30.8, 54.0), turned to 90 degrees
- moved R26 87.0 mm to (70.1, 50.5)
- moved C8 86.2 mm to (67.3, 51.4), turned to 270 degrees
- moved D8 85.7 mm to (68.4, 45.9), turned to 90 degrees
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Connections:
- C1 pad 1: /BAT -> /LOGIC_SUPPLY
- C2 pad 1: Net-(C2-Pad1) -> /LOGIC_SUPPLY
- C7 pad 1: /BAT -> /BOOST_5V0/BOOST_IN
- C9 pad 1: /BAT -> /BOOST_5V0/BOOST_IN
- D1 pad 1: Net-(C2-Pad1) -> /LOGIC_SUPPLY
- D2 pad 1: Net-(C2-Pad1) -> /LOGIC_SUPPLY
- D2 pad 2: /BAT -> /BOOST_5V0/BOOST_IN
- J2 pad 1: /BAT -> /BOOST_5V0/BOOST_IN
- J2 pad 2: /BAT -> /BOOST_5V0/BOOST_IN
- J3 pad 2: Net-(J3-Pad2) -> (no net)
- J3 pad 3: Net-(J3-Pad3) -> (no net)
- L2 pad 2: /BAT -> /BOOST_5V0/BOOST_IN
- R10 pad 1: Net-(C2-Pad1) -> /LOGIC_SUPPLY
- R5 pad 1: Net-(C2-Pad1) -> /LOGIC_SUPPLY
- R8 pad 1: Net-(C2-Pad1) -> /LOGIC_SUPPLY
- U1 pad 8: /BAT -> /LOGIC_SUPPLY
- U3 pad 1: Net-(U3-Pad1) -> (no net)
- U3 pad 6: Net-(U3-Pad6) -> (no net)
- U3 pad 8: Net-(U3-Pad8) -> (no net)
- U4 pad 5: /BAT -> /BOOST_5V0/BOOST_IN
- U5 pad 5: /BAT -> /BOOST_5V0/BOOST_IN
- U5 pad 6: Net-(U5-Pad6) -> (no net)
Routing:
- net /Buck_5V0/BUCK_5V0: track 0.00 -> 43.8 mm, vias 0 -> 2
- net /BOOST_5V0/BOOST_IN: track 0.00 -> 43.3 mm, vias 0 -> 3
- net /BatteryCharger/VCC: track 0.00 -> 36.2 mm, vias 0 -> 4
- net /LOGIC_SUPPLY: track 0.00 -> 36.1 mm, vias 0 -> 2
- net /Buck_5V0/BUCK_IN: track 0.00 -> 34.7 mm
- net Net-(C10-Pad2): track 0.00 -> 25.3 mm, vias 0 -> 3
- net Net-(C12-Pad1): track 0.00 -> 19.8 mm
- net Net-(C10-Pad1): track 0.00 -> 19.5 mm, vias 0 -> 2
- net /BatteryCharger/temp: track 0.00 -> 17.8 mm
- net Net-(C11-Pad2): track 0.00 -> 16.9 mm
- net /VREF_3V0: track 0.00 -> 10.6 mm
- net /_EN_BAT: track 0.00 -> 10.6 mm
- net Net-(R6-Pad2): track 0.00 -> 9.99 mm, vias 0 -> 2
- net Net-(D8-Pad2): track 0.00 -> 8.77 mm
- net Net-(C5-Pad1): track 0.00 -> 8.40 mm
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- added copper zone on B.Cu, net GND
- added copper zone on F.Cu, net GND
Other:
- board outline added: 60 x 44 mm

Commit message: pcb updated
Parts:
- removed D9: 7V5, custom-footprints:LL34
- added REF**: MountingHole_2.2mm_M2, MountingHole:MountingHole_2.2mm_M2, F.Cu at (23.0, 44.1)
- added REF**: MountingHole_2.2mm_M2, MountingHole:MountingHole_2.2mm_M2, F.Cu at (117.0, 44.0)
- added REF**: MountingHole_2.2mm_M2, MountingHole:MountingHole_2.2mm_M2, F.Cu at (116.9, 22.9)
- added REF**: MountingHole_2.2mm_M2, MountingHole:MountingHole_2.2mm_M2, F.Cu at (78.0, 28.0)
- moved D11 42.6 mm to (103.3, 45.2)
- moved R30 41.0 mm to (97.5, 24.5)
- moved Q7 40.9 mm to (97.4, 38.7)
- moved Q8 40.9 mm to (97.4, 31.2)
- moved Q9 40.9 mm to (97.4, 35.1)
- moved R32 40.9 mm to (93.7, 28.4)
- moved R33 40.9 mm to (93.4, 37.8)
- moved C11 40.9 mm to (93.5, 39.6)
- moved C12 40.9 mm to (101.1, 31.2)
- moved C13 40.9 mm to (101.1, 35.1)
- moved J3 40.9 mm to (110.6, 33.1)
- moved Q5 40.9 mm to (93.5, 35.0)
- moved R31 40.9 mm to (97.3, 41.7)
- moved R34 40.9 mm to (104.8, 31.2)
- moved R35 40.9 mm to (104.8, 35.0)
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Routing:
- net /EN_BAT: track 7.43 -> 83.3 mm, vias 0 -> 3
- net /_EN_BAT: track 10.6 -> 68.1 mm, vias 0 -> 2
- net /Buck_5V0/BUCK_5V0: track 43.8 -> 79.6 mm, vias 2 -> 0
- net /BOOST_5V0/BOOST_OUT: track 5.01 -> 26.8 mm, vias 0 -> 3
- net /BOOST_5V0/BOOST_IN: track 43.3 -> 60.7 mm, vias 3 -> 4
- net /Buck_5V0/EN: track 7.65 -> 17.3 mm, vias 0 -> 3
- net Net-(D11-Pad2): track 2.69 -> 9.30 mm
- net Net-(C11-Pad2): track 16.9 -> 23.3 mm
- net Net-(D12-Pad2): track 2.52 -> 8.52 mm
- net Net-(C10-Pad2): track 25.3 -> 30.6 mm
- net Net-(D5-Pad1): track 7.99 -> 12.3 mm
- net Net-(C5-Pad1): track 8.40 -> 12.2 mm
- net Net-(D3-Pad2): track 6.61 -> 9.08 mm
- net Net-(D4-Pad2): track 6.60 -> 9.01 mm
- net /Buck_5V0/BUCK_IN: track 34.7 -> 36.8 mm, vias 0 -> 1
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Other:
- board size 60 x 44 mm -> 100 x 27 mm

Commit message: pcb updated
Routing:
- net /BOOST_5V0/BOOST_OUT: track 26.8 -> 8.65 mm, vias 3 -> 7
- net /Buck_5V0/BUCK_5V0: track 79.6 -> 77.4 mm
- net GND: vias 34 -> 39
- added copper zone on B.Cu, net /BOOST_5V0/BOOST_OUT
- added copper zone on F.Cu, net /BOOST_5V0/BOOST_OUT
- added copper zone on F.Cu, net /Buck_5V0/BUCK_5V0
Other:
- board text added: "BAT"
- board text added: "SP"
- board text added: "Solar Charger V1.0 V.Tolentino"
Changed lines of the file:
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@@
   (general
     (thickness 1.6)
-    (drawings 4)
-    (tracks 421)
+    (drawings 7)
+    (tracks 426)
     (zones 0)
     (modules 84)
@@
   )
   (setup
-    (last_trace_width 0.5)
+    (last_trace_width 0.25)
     (user_trace_width 0.5)
     (user_trace_width 1)
@@
     (visible_elements 7FFFFFFF)
     (pcbplotparams
-      (layerselection 0x010fc_ffffffff)
+      (layerselection 0x010f0_ffffffff)
       (usegerberextensions false)
       (usegerberattributes false)
@@
       (psnegative false)
       (psa4output false)
-      (plotreference true)
-      (plotvalue true)
+      (plotreference false)
+      (plotvalue false)
       (plotinvisibletext false)
       (padsonsilk false)
@@
       (outputformat 1)
       (mirror false)
-      (drillshape 1)
+      (drillshape 0)
       (scaleselection 1)
-      (outputdirectory ""))
+      (outputdirectory "Gerber/"))
   )
   (net 0 "")
@@
     (pad 1 np_thru_hole circle (at 0 0) (size 2.2 2.2) (drill 2.2) (layers *.Cu *.Mask))
   )
+  (gr_text "Solar Charger V1.0 V.Tolentino" (at 67.7672 21.844) (layer F.SilkS)
+    (effects (font (size 1.5 1.5) (thickness 0.3)))
+  )
+  (gr_text BAT (at 108.6612 44.8564) (layer F.SilkS)
+    (effects (font (size 1.5 1.5) (thickness 0.3)))
+  )
+  (gr_text SP (at 108.2548 22.606) (layer F.SilkS)
+    (effects (font (size 1.5 1.5) (thickness 0.3)))
+  )
   (gr_line (start 20 20) (end 20 47) (layer Edge.Cuts) (width 0.05))
   (gr_line (start 20 47) (end 120 47) (layer Edge.Cuts) (width 0.05))
@@
   (via (at 64.9732 42.5196) (size 0.8) (drill 0.4) (layers F.Cu B.Cu) (net 1))
   (via (at 63.8048 42.5196) (size 0.8) (drill 0.4) (layers F.Cu B.Cu) (net 1))
+  (via (at 54.1528 30.8864) (size 0.8) (drill 0.4) (layers F.Cu B.Cu) (net 1))
+  (via (at 54.1528 29.5148) (size 0.8) (drill 0.4) (layers F.Cu B.Cu) (net 1))
+  (via (at 54.2036 28.0924) (size 0.8) (drill 0.4) (layers F.Cu B.Cu) (net 1))
+  (via (at 54.4576 38.7096) (size 0.8) (drill 0.4) (layers F.Cu B.Cu) (net 1))
+  (via (at 60.0964 35.4584) (size 0.8) (drill 0.4) (layers F.Cu B.Cu) (net 1))
   (segment (start 36.2554 38.7604) (end 36.2554 33.9344) (width 1) (layer F.Cu) (net 2))
   (segment (start 36.2554 29.4482) (end 35.4076 28.6004) (width 1) (layer F.Cu) (net 2))
@@
   (segment (start 46.3966 23.6956) (end 46.4754 23.7744) (width 1) (layer F.Cu) (net 3))
   (segment (start 45.8216 23.6956) (end 46.3966 23.6956) (width 1) (layer F.Cu) (net 3))
-  (segment (start 58.5724 29.21) (end 58.5724 35.719299) (width 1) (layer F.Cu) (net 3))
-  (segment (start 53.1368 23.7744) (end 58.5724 29.21) (width 1) (layer F.Cu) (net 3))
   (segment (start 52.3862 26.0442) (end 52.3748 26.0328) (width 0.5) (layer F.Cu) (net 3))
   (segment (start 52.3862 26.6192) (end 52.3862 26.0442) (width 0.5) (layer F.Cu) (net 3))
@@
   (segment (start 46.4754 23.7744) (end 52.3748 23.7744) (width 1) (layer F.Cu) (net 3))
   (segment (start 52.3748 23.7744) (end 53.1368 23.7744) (width 1) (layer F.Cu) (net 3))
-  (segment (start 85.8203 23.7744) (end 53.1368 23.7744) (width 1) (layer F.Cu) (net 3))
   (segment (start 92.2244 30.1785) (end 85.8203 23.7744) (width 1) (layer F.Cu) (net 3))
   (segment (start 93.6244 30.1785) (end 92.2244 30.1785) (width 1) (layer F.Cu) (net 3))
+  (segment (start 58.5724 23.8252) (end 58.6232 23.7744) (width 1) (layer F.Cu) (net 3))
+  (segment (start 58.5724 35.719299) (end 58.5724 23.8252) (width 1) (layer F.Cu) (net 3))
+  (segment (start 85.8203 23.7744) (end 58.6232 23.7744) (width 1) (layer F.Cu) (net 3))
+  (segment (start 58.6232 23.7744) (end 53.1368 23.7744) (width 1) (layer F.Cu) (net 3))
   (segment (start 48.8048 28.3832) (end 48.8188 28.3692) (width 0.5) (layer F.Cu) (net 4))
   (segment (start 50.6196 28.3692) (end 50.6476 28.3972) (width 0.5) (layer F.Cu) (net 4))
@@
   (segment (start 78.0034 38.2874) (end 79.0194 37.2714) (width 1) (layer F.Cu) (net 6))
   (segment (start 78.0034 39.9314) (end 78.0034 38.2874) (width 1) (layer F.Cu) (net 6))
-  (segment (start 78.0034 39.9314) (end 76.9594 39.9314) (width 1) (layer F.Cu) (net 6))
-  (via (at 76.454 40.4368) (size 0.8) (drill 0.4) (layers F.Cu B.Cu) (net 6))
-  (segment (start 76.9594 39.9314) (end 76.454 40.4368) (width 1) (layer F.Cu) (net 6))
-  (segment (start 76.454 39.871115) (end 81.781115 34.544) (width 1) (layer B.Cu) (net 6))
-  (segment (start 76.454 40.4368) (end 76.454 39.871115) (width 1) (layer B.Cu) (net 6))
-  (via (at 90.0684 34.544) (size 0.8) (drill 0.4) (layers F.Cu B.Cu) (net 6))
-  (segment (start 81.781115 34.544) (end 90.0684 34.544) (width 1) (layer B.Cu) (net 6))
   (via (at 90.0684 34.544) (size 0.8) (drill 0.4) (layers F.Cu B.Cu) (net 6))
   (segment (start 93.113872 34.028511) (end 93.4974 34.028511) (width 1) (layer F.Cu) (net 6))
@@
   (segment (start 90.468399 34.144001) (end 92.998382 34.144001) (width 1) (layer F.Cu) (net 6))
   (segment (start 90.0684 34.544) (end 90.468399 34.144001) (width 1) (layer F.Cu) (net 6))
+  (via (at 90.0176 35.6108) (size 0.8) (drill 0.4) (layers F.Cu B.Cu) (net 6))
+  (via (at 88.7984 35.6108) (size 0.8) (drill 0.4) (layers F.Cu B.Cu) (net 6))
+  (via (at 88.8492 33.528) (size 0.8) (drill 0.4) (layers F.Cu B.Cu) (net 6))
+  (via (at 76.5048 39.3192) (size 0.8) (drill 0.4) (layers F.Cu B.Cu) (net 6))
+  (via (at 90.0684 34.544) (size 0.8) (drill 0.4) (layers F.Cu B.Cu) (net 6))
+  (via (at 76.454 40.4368) (size 0.8) (drill 0.4) (layers F.Cu B.Cu) (net 6))
   (segment (start 94.5879 32.192) (end 94.5744 32.1785) (width 1) (layer F.Cu) (net 7))
   (segment (start 96.3709 32.192) (end 94.5879 32.192) (width 1) (layer F.Cu) (net 7))
@@
     (polygon
       (pts
-        (xy 20.0152 20.0152) (xy 119.9896 20.0152) (xy 119.9896 46.99) (xy 20.0152 46.99)
+        (xy 20.0152 20.0152) (xy 47.1424 20.0152) (xy 47.1424 24.5364) (xy 53.6956 24.5364) (xy 57.9628 31.4452)
+        (xy 59.3852 31.4452) (xy 59.3852 26.8732) (xy 61.468 24.5364) (xy 83.312 24.5364) (xy 91.2876 32.004)
+        (xy 94.3356 32.004) (xy 94.3356 20.0152) (xy 119.9896 20.0152) (xy 119.9896 46.99) (xy 20.0152 46.99)
       )
     )
@@
       )
     )
+  )
+  (zone (net 3) (net_name /Buck_5V0/BUCK_5V0) (layer F.Cu) (hatch edge 0.508)
+    (connect_pads (clearance 0.254))
+    (min_thickness 0.254)
+    (fill yes (arc_segments 16) (thermal_gap 0.508) (thermal_bridge_width 0.508))
+    (polygon
+      (pts
+        (xy 47.3964 24.2824) (xy 47.3964 20.0152) (xy 94.0308 20.0152) (xy 94.0308 31.6484) (xy 91.3384 31.6484)
+        (xy 83.5152 24.2824) (xy 61.3156 24.2824) (xy 59.0804 26.5684) (xy 59.0804 31.0896) (xy 58.0644 31.0896)
+        (xy 53.9496 24.2824)
+      )
+    )
+  )
+  (zone (net 6) (net_name /BOOST_5V0/BOOST_OUT) (layer B.Cu) (hatch edge 0.508)
+    (priority 1)
+    (connect_pads (clearance 0.254))
+    (min_thickness 0.254)
+    (fill yes (arc_segments 16) (thermal_gap 0.508) (thermal_bridge_width 0.508))
+    (polygon
+      (pts
+        (xy 75.6412 41.402) (xy 75.6412 33.9344) (xy 76.454 33.02) (xy 89.7636 33.02) (xy 91.2876 34.3408)
+        (xy 91.2876 35.4584) (xy 91.2876 36.83) (xy 90.0684 38.1) (xy 88.4936 38.1) (xy 87.2236 37.0332)
+        (xy 85.2932 35.4584) (xy 82.0928 35.4076) (xy 77.4192 40.0812) (xy 77.4192 41.4528) (xy 75.6412 41.4528)
+      )
+    )
+  )
+  (zone (net 6) (net_name /BOOST_5V0/BOOST_OUT) (layer F.Cu) (hatch edge 0.508)
+    (priority 1)
+    (connect_pads (clearance 0.254))
+    (min_thickness 0.254)
+    (fill yes (arc_segments 16) (thermal_gap 0.508) (thermal_bridge_width 0.508))
+    (polygon
+      (pts
+        (xy 75.946 40.386) (xy 75.946 38.6588) (xy 77.2668 38.6588) (xy 77.2668 39.4208) (xy 78.5368 39.4208)
+        (xy 78.5368 40.5384) (xy 77.2668 40.5384) (xy 77.2668 40.9448) (xy 75.946 40.9448)
+      )
+    )
+  )
+  (zone (net 6) (net_name /BOOST_5V0/BOOST_OUT) (layer F.Cu) (hatch edge 0.508)
+    (priority 1)
+    (connect_pads (clearance 0.254))
+    (min_thickness 0.254)
+    (fill yes (arc_segments 16) (thermal_gap 0.508) (thermal_bridge_width 0.508))
+    (polygon
+      (pts
+        (xy 90.4748 33.6296) (xy 89.7636 33.02) (xy 88.1888 33.02) (xy 88.1888 35.9664) (xy 88.7984 36.3728)
+        (xy 90.17 36.3728) (xy 90.7288 35.8648) (xy 91.7956 34.6456)
+      )
+    )
