File: Projects/Watering_System/Schematic/WateringSystem.sch (KiCad schematic (older format))
At the start: 20 parts

Commit message: add gerber files for watering project
Parts:
- removed J?: Conn_02x04_Counter_Clockwise, symbol Connector_Generic:Conn_02x04_Counter_Clockwise
- removed R?: 10k, symbol Device:R
- removed SW?: SW_Push, symbol Switch:SW_Push
- added D2: YELLOW, LED_SMD:LED_1206_3216Metric_Pad1.42x1.75mm_HandSolder, symbol Device:LED
- added D3: RED, LED_SMD:LED_1206_3216Metric_Pad1.42x1.75mm_HandSolder, symbol Device:LED
- added J2: Conn_02x04_Odd_Even, Connector_PinHeader_2.54mm:PinHeader_2x04_P2.54mm_Vertical, symbol Connector_Generic:Conn_02x04_Odd_Even
- added J4: WATER_SENSOR, Connector_PinHeader_2.54mm:PinHeader_1x04_P2.54mm_Vertical, symbol Connector:Conn_01x04_Female
- added R2, R4: 560, Resistor_SMD:R_0603_1608Metric_Pad1.05x0.95mm_HandSolder, symbol Device:R
- added R5, R6: ??, Resistor_SMD:R_0603_1608Metric_Pad1.05x0.95mm_HandSolder, symbol Device:R
- A1: footprint Module:Arduino_Nano -> Module:Arduino_Nano_WithMountingHoles
- C1, C2: renamed from C?; footprint (none) -> Capacitor_SMD:C_0603_1608Metric_Pad1.05x0.95mm_HandSolder
- C3: renamed from C?; value C -> 100n; footprint (none) -> Capacitor_SMD:C_0603_1608Metric_Pad1.05x0.95mm_HandSolder
- D1: renamed from D?; value D_Schottky -> SS14; footprint (none) -> custom-footprints:SMA_DO-214AC
- J1: renamed from J?; value Conn_01x04_Female -> MOTOR_INTERFACE; footprint (none) -> Connector_PinHeader_2.54mm:PinHeader_1x04_P2.54mm_Vertical
- J3: renamed from J?; value Conn_01x03_Male -> FLASH_WIFI; footprint (none) -> Connector_PinHeader_2.54mm:PinHeader_1x03_P2.54mm_Vertical
- Q1: renamed from Q?; value Q_NMOS_GSD -> AO3400A; footprint (none) -> Package_TO_SOT_SMD:SOT-23
- R1: renamed from 47k; value R -> 47k; footprint (none) -> Resistor_SMD:R_0603_1608Metric_Pad1.05x0.95mm_HandSolder
- R10, R7: renamed from R?; value 0 -> 4k7; footprint (none) -> Resistor_SMD:R_0603_1608Metric_Pad1.05x0.95mm_HandSolder
- R11, R12, R8: renamed from R?; footprint (none) -> Resistor_SMD:R_0603_1608Metric_Pad1.05x0.95mm_HandSolder
- R3: renamed from R?; value R -> 100; footprint (none) -> Resistor_SMD:R_0603_1608Metric_Pad1.05x0.95mm_HandSolder
- U1: renamed from U?; footprint (none) -> Connector_PinHeader_2.54mm:PinHeader_2x04_P2.54mm_Vertical
- U2: renamed from U?; footprint (none) -> Connector_PinHeader_2.54mm:PinHeader_1x04_P2.54mm_Vertical
Connections:
- net labels added: GPIO0_WIFI, LR_LEVEL, MOTOR_GND, M_FILTERED_PWM, RED_LED, RST_WIFI, SR_LEVEL, YELLOW_LED
- net labels removed: MOTOR_N, _RS_EMPTY
- wire segments 86 -> 115
- no-connect marks 1 -> 15
Other:
- note added: "homemade water sensors"
- moved on the sheet: R10, R7, U2

Commit message: update bom
Parts:
- added C?: 2u2, Capacitor_SMD:C_0603_1608Metric_Pad1.05x0.95mm_HandSolder, symbol Device:C
- added C?: 470p, Capacitor_SMD:C_0603_1608Metric_Pad1.05x0.95mm_HandSolder, symbol Device:C
- added U?: MIC5219-3.3YM5, Package_TO_SOT_SMD:SOT-23-5, symbol Regulator_Linear:MIC5219-3.3YM5
Connections:
- net 3V3: now also C?.1, U?.5 (OUT); no longer A1.17 (3V3)
- net 5V0: now also U?.1 (IN), U?.3 (EN)
- net GND: now also C?.2, C?.2, U?.2 (GND)
- new net: C?.1, U?.4 (BP)
- no-connect marks 15 -> 16
Changed lines of the file:
@@
 EESchema Schematic File Version 4
 LIBS:WateringSystem-cache
-EELAYER 26 0
+EELAYER 29 0
 EELAYER END
 $Descr A4 11693 8268
@@
 Text Label 5950 2700 0    50   ~ 0
 5V0
-Wire Wire Line
-	5700 3200 5700 2700
-Wire Wire Line
-	5700 2700 5600 2700
-Text Label 5600 2700 0    50   ~ 0
-3V3
 Wire Wire Line
 	1200 3700 1400 3700
@@
 Text Label 8750 5650 0    50   ~ 0
 GPIO0_WIFI
+$Comp
+L Regulator_Linear:MIC5219-3.3YM5 U?
+U 1 1 5CEABBD1
+P 2250 6500
+F 0 "U?" H 2250 6842 50  0000 C CNN
+F 1 "MIC5219-3.3YM5" H 2250 6751 50  0000 C CNN
+F 2 "Package_TO_SOT_SMD:SOT-23-5" H 2250 6825 50  0001 C CNN
+F 3 "http://ww1.microchip.com/downloads/en/DeviceDoc/MIC5219-500mA-Peak-Output-LDO-Regulator-DS20006021A.pdf" H 2250 6500 50  0001 C CNN
+	1    2250 6500
+	1    0    0    -1
+$EndComp
+NoConn ~ 5700 3200
+$Comp
+L power:GND #PWR?
+U 1 1 5CEBC8EB
+P 2250 7350
+F 0 "#PWR?" H 2250 7100 50  0001 C CNN
+F 1 "GND" H 2255 7177 50  0000 C CNN
+F 2 "" H 2250 7350 50  0001 C CNN
+F 3 "" H 2250 7350 50  0001 C CNN
+	1    2250 7350
+	1    0    0    -1
+$EndComp
+Wire Wire Line
+	2250 6800 2250 7250
+Wire Wire Line
+	1950 6400 1750 6400
+Wire Wire Line
+	2550 6400 3050 6400
+Text Label 1250 6400 0    50   ~ 0
+5V0
+Text Label 3250 6400 0    50   ~ 0
+3V3
+Wire Wire Line
+	1950 6500 1750 6500
+Wire Wire Line
+	1750 6500 1750 6400
+Connection ~ 1750 6400
+Wire Wire Line
+	1750 6400 1250 6400
+$Comp
+L Device:C C?
+U 1 1 5CECCB8D
+P 3050 6900
+F 0 "C?" H 3165 6946 50  0000 L CNN
+F 1 "2u2" H 3165 6855 50  0000 L CNN
+F 2 "Capacitor_SMD:C_0603_1608Metric_Pad1.05x0.95mm_HandSolder" H 3088 6750 50  0001 C CNN
+F 3 "~" H 3050 6900 50  0001 C CNN
+	1    3050 6900
+	1    0    0    -1
+$EndComp
+$Comp
+L Device:C C?
+U 1 1 5CECD573
+P 2700 6900
+F 0 "C?" H 2815 6946 50  0000 L CNN
+F 1 "470p" H 2815 6855 50  0000 L CNN
+F 2 "Capacitor_SMD:C_0603_1608Metric_Pad1.05x0.95mm_HandSolder" H 2738 6750 50  0001 C CNN
+F 3 "~" H 2700 6900 50  0001 C CNN
+	1    2700 6900
+	1    0    0    -1
+$EndComp
+Wire Wire Line
+	2550 6500 2700 6500
+Wire Wire Line
+	2700 6500 2700 6750
+Wire Wire Line
+	2700 7050 2700 7250
+Wire Wire Line
+	2700 7250 2250 7250
+Connection ~ 2250 7250
+Wire Wire Line
+	2250 7250 2250 7350
+Wire Wire Line
+	3050 7050 3050 7250
+Wire Wire Line
+	3050 7250 2700 7250
+Connection ~ 2700 7250
+Wire Wire Line
+	3050 6750 3050 6400
+Connection ~ 3050 6400
+Wire Wire Line
+	3050 6400 3250 6400
 $EndSCHEMATC
